File: hellen88bmw.kicad_pcb (KiCad board)
At the start: 2 copper layers, 160 x 118 mm, 116 parts, among them J1 Conn_01x05, J10 Conn_01x12, J11 Conn_01x12, J12 Conn_01x12, J13 Conn_01x12, J2 Conn_01x05, J3 Micro_SD_Card, J4 Conn_01x05, J5 Conn_01x12, J6 Conn_01x12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

Commit message: Up 88bmw update
Routing:
- removed copper zone on B.Cu, net GND
Changed lines of the file:
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@@
-    )
-  )
-  (zone (net 89) (net_name "GND") (layer "F.Cu") (hatch edge 0.508)
-    (connect_pads (clearance 0.508))
-    (min_thickness 0.254)
-    (fill yes (thermal_gap 0.508) (thermal_bridge_width 0.508))
-    (polygon
-      (pts
-        (xy 234.95 51.435)
-        (xy 218.44 51.374312)
-        (xy 218.44 64.77)
-        (xy 212.09 64.77)
-        (xy 212.09 100.33)
-        (xy 218.44 100.33)
-        (xy 218.44 114.3)
-        (xy 213.36 114.3)
-        (xy 213.36 153.67)
-        (xy 230.505 153.67)
-        (xy 230.505 114.3)
-        (xy 234.95 114.3)
-        (xy 234.95 158.115)
-        (xy 230.505 158.115)
-        (xy 230.505 158.097361)
-        (xy 74.93 157.48)
-        (xy 74.93 40.005)
-        (xy 234.95 40.005)
-      )
     )
   )
@@
       )
     )
-  )
-  (zone (net 89) (net_name "GND") (layer "B.Cu") (hatch edge 0.508)
-    (connect_pads yes (clearance 0.508))
-    (min_thickness 0.254)
-    (fill yes (thermal_gap 0.508) (thermal_bridge_width 0.508))
-    (polygon
-      (pts
-        (xy 234.95 42.545)
-        (xy 234.95 51.435)
-        (xy 218.44 51.435)
-        (xy 218.44 64.135)
-        (xy 213.36 64.135)
-        (xy 213.36 99.695)
-        (xy 229.87 99.695)
-        (xy 229.87 64.135)
-        (xy 234.95 64.135)
-        (xy 234.95 100.965)
-        (xy 218.44 100.965)
-        (xy 218.44 114.3)
-        (xy 213.36 114.3)
-        (xy 213.36 152.4)
-        (xy 230.505 152.4)
-        (xy 230.505 114.3)
-        (xy 234.95 114.3)
-        (xy 234.95 158.115)
-        (xy 74.93 158.115)
-        (xy 74.93 40.64)
-        (xy 232.41 40.005)
-      )
-    )

Commit message: Up 88bmw update
Parts:
- removed J1, J2: Conn_01x05, Connector_PinHeader_2.54mm:PinHeader_1x05_P2.54mm_Vertical
- removed U2: molex_48pin_MRE, rusefi_lib:Molex_48_MRE_with-extras
Routing:
- net GND: track 842.1 -> 635.7 mm, vias 19 -> 10
- net /12_MAIN_RELAY: track 218.1 -> 81.2 mm, vias 4 -> 2
- net /GND_SENS: track 209.6 -> 89.8 mm, vias 3 -> 0
- net /GP6: track 156.9 -> 37.9 mm, vias 3 -> 1
- net /J806_PB9: track 137.6 -> 38.7 mm
- net /J808_PC10: track 109.6 -> 13.0 mm
- net /GP5: track 135.4 -> 38.9 mm, vias 3 -> 1
- net /MAIN_RELAY: track 136.8 -> 41.7 mm, vias 2 -> 0
- net /MAF_AV4: track 194.3 -> 110.8 mm, vias 5 -> 0
- net /IGN_4: track 118.3 -> 39.9 mm, vias 2 -> 0
- net /J805_PC11: track 116.7 -> 43.9 mm
- net /CLT_AT1: track 78.6 -> 6.82 mm
- net /NEUTRAL_IN_AT3: track 86.9 -> 19.4 mm, vias 2 -> 0
- net /IDLE_LS2: track 85.9 -> 19.7 mm
- net /IGN_2: track 119.3 -> 55.6 mm, vias 1 -> 0
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