File: hellen88bmw.kicad_pcb (KiCad board)
At the start: 4 copper layers, 160 x 118 mm, 305 parts, among them J1 920-462A2021Y10101, J10 Conn_01x12, J11 Conn_01x12, J12 Conn_01x12, J13 Conn_01x12, J14 VRIN1, J15 VRIN2, J16 VROUT1, J17 XH-8A, J18 PJ-3250-5A, J19 MiniFit, J2 UB-20PMFP-LC7002, J20 ETB, J21 ETB, J3 Micro_SD_Card, J4 Conn_01x05, J5 Conn_01x12, J6 Conn_01x12, J7 Conn_01x12, J8 Conn_01x12, J9 Conn_01x12, M1 Module-power12-0.2, M10 Module-ign8-0.1, M11 Module-mcu144-0.5, M12 Module-knock-0.1, M2 Module-can-0.1, M3 Module-wbo-0.2, M4 Module-can-0.1, M5 Module-power5-0.2, M6 Module-vr-0.1, M7 Module-input-0.1, M8 Module-knock-0.1, M9 Module-output-0.2, P1 P, P2 P, P3 P, P4 P, P5 P, P6 P, Q1 NGD8201AN, Q2 NGD8201AN, Q3 NGD8201AN, Q4 NGD8201AN, Q5 NGD8201AN, Q6 NGD8201AN, Q7 NGD8201AN, Q8 NGD8201AN, SW1 RESET, SW2 RESET, U1 MPXA6115A, U2 MPX4_MAP, U3 LIS2DW12TR, U4 LPS25HB, U5 MCP6002-xSN, U6 L6205PD

Commit message: update 28/08/2021
Parts:
- removed MMCU17, MMCU33, MMCU34, MMCU36: MMCU, Connector_PinHeader_1.00mm:PinHeader_1x01_P1.00mm_Vertical
- removed VIN21, VIN24, VIN25: Pad, Connector_PinHeader_1.00mm:PinHeader_1x01_P1.00mm_Vertical
- removed VIN5: VIN5, Connector_PinHeader_1.00mm:PinHeader_1x01_P1.00mm_Vertical
- removed VIN6: VIN6, Connector_PinHeader_1.00mm:PinHeader_1x01_P1.00mm_Vertical
- removed VIN7: VIN7, Connector_PinHeader_1.00mm:PinHeader_1x01_P1.00mm_Vertical
- added D10: 1N4148WS, Diode_SMD:D_SOD-323, F.Cu at (36.2, 86.2)
- added JP14: Jumper_2_Open, rusefi_lib:SM0805_jumper, F.Cu at (37.3, 83.3)
- added R27: 470k, Resistor_SMD:R_0402_1005Metric, F.Cu at (42.7, 89.0)
- added R34: 470k, Resistor_SMD:R_0402_1005Metric, F.Cu at (42.7, 85.0)
- added R35: 470k, Resistor_SMD:R_0402_1005Metric, F.Cu at (39.8, 85.8)
- added R36: 470k, Resistor_SMD:R_0402_1005Metric, F.Cu at (35.6, 88.7)
- added R37: 470k, Resistor_SMD:R_0402_1005Metric, F.Cu at (42.7, 87.0)
- added R38: 470k, Resistor_SMD:R_0402_1005Metric, F.Cu at (41.9, 83.0)
- added R39: 470k, Resistor_SMD:R_0402_1005Metric, F.Cu at (45.6, 85.0)
- added R40: 470k, Resistor_SMD:R_0402_1005Metric, F.Cu at (44.8, 83.0)
- added R41: 470k, Resistor_SMD:R_0402_1005Metric, F.Cu at (39.8, 87.8)
- VIN3: value Pad -> VIN8
- moved JP1 1.00 mm to (85.0, 55.0)
- moved JP29 1.00 mm to (87.8, 55.0)
- moved cr4 0.75 mm to (82.5, 53.0)
Connections:
- net /A3 renamed /TPS3
- J20 pad 3: /IN_TPS -> /IN_TPS3
- J20 pad 4: Net-(J20-Pad4) -> /IN_TPS2
- J21 pad 2: /IN_TPS -> /IN_PPS2
- J21 pad 3: Net-(J20-Pad4) -> /IN_PPS1
- M11 pad S11: Net-(M11-PadS11) -> /SENS4
- M11 pad S24: Net-(M11-PadS24) -> /TPS2
- M11 pad S8: Net-(M11-PadS8) -> /SENS1
- M11 pad S9: Net-(M11-PadS9) -> /SENS2
- M7 pad N23: Net-(M7-PadN23) -> /SENS4
- M7 pad N25: Net-(M7-PadN25) -> /SENS2
- M7 pad N26: Net-(M7-PadN26) -> /SENS1
- M7 pad S17: Net-(J20-Pad4) -> /IN_TPS2
- M7 pad S18: Net-(M7-PadS18) -> /IN_PPS2
- M7 pad S20: Net-(M7-PadS20) -> /IN_TPS3
- M7 pad S24: Net-(M7-PadS24) -> /IN_PPS1
- PP1 pad 14: GND -> Net-(JP14-Pad1)
- R1 pad 1: /IN_TPS -> /IN_TPS2
- R2 pad 1: Net-(J20-Pad4) -> /IN_PPS1
- VIN3 pad 1: Net-(M7-PadS18) -> Net-(M7-PadS21)
Routing:
- net /IN_PPS1: track 0.00 -> 193.0 mm, vias 0 -> 1
- net Net-(J20-Pad4): track 189.3 -> 0.00 mm, vias 1 -> 0
- net /OUT_MAIN: track 142.2 -> 192.7 mm, vias 2 -> 4
- net /MAIN_RELAY: track 50.5 -> 0.00 mm, vias 2 -> 0
- net GND: track 266.3 -> 309.9 mm, vias 192 -> 241
- net /SENS1: track 0.00 -> 13.0 mm
- net /SENS2: track 0.00 -> 12.1 mm
- net Net-(M7-PadN26): track 10.4 -> 0.00 mm
- net Net-(M7-PadN25): track 9.92 -> 0.00 mm
- net Net-(M7-PadS20): track 4.58 -> 0.00 mm
- net /IN_TPS3: track 0.00 -> 4.58 mm
- net /COIL_8: track 101.3 -> 105.8 mm
- net Net-(M7-PadS21): track 6.11 -> 10.6 mm
- net Net-(M7-PadS18): track 4.53 -> 0.00 mm
- net Net-(M7-PadS24): track 3.70 -> 0.00 mm
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