File: hellen88bmw.kicad_sch (KiCad schematic)
At the start: 310 parts, among them J1 920-462A2021Y10101, J10 Conn_01x12, J11 Conn_01x12, J12 Conn_01x12, J13 Conn_01x12, J14 VRIN1, J15 VRIN2, J16 VROUT1, J17 XH-8A, J18 PJ-3250-5A, J19 MiniFit, J2 UB-20PMFP-LC7002, J20 ETB_6p, J21 ETB_4p, J3 Micro_SD_Card, J4 Conn_01x05, J5 Conn_01x12, J6 Conn_01x12, J7 Conn_01x12, J8 Conn_01x12, J9 Conn_01x12, M1 Module-power12-0.2, M10 Module-ign8-0.1, M11 Module-mcu-0.4, M12 Module-knock-0.1, M2 Module-can-0.1, M3 Module-wbo-0.2, M4 Module-can-0.1, M5 Module-power5-0.2, M6 Module-vr-0.1, M7 Module-input-0.1, M8 Module-knock-0.1, M9 Module-output-0.2, P1 P, P2 P, P3 P, P4 P, P5 P, P6 P, Q1 NGD8201AN, Q2 NGD8201AN, Q3 NGD8201AN, Q4 NGD8201AN, Q5 NGD8201AN, Q6 NGD8201AN, Q7 NGD8201AN, Q8 NGD8201AN, SW1 BOOT0, SW2 RESET, U1 MPXA6115A, U2 MPX4_MAP, U3 LIS2DW12TR, U4 LPS25HB, U5 MCP6002-xSN, U6 L6205PD

Commit message: fix 14/08/2021
Parts:
- J2: LCSC NA -> DNP
- M11: value Module-mcu-0.4 -> Module-mcu-0.5; footprint hellen-one-mcu-0.4:mcu -> hellen-one-mcu-0.5:mcu; symbol hellen-one-mcu-000.4:Module-mcu-0.4 -> hellen-one-mcu-000.5:Module-mcu-0.5
- SW1: value BOOT0 -> RESET
Changed lines of the file:
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@@
     (in_bom yes) (on_board yes)
     (property "Reference" "SW1" (id 0) (at 635 180.34 0))
-    (property "Value" "BOOT0" (id 1) (at 635 182.88 0))
+    (property "Value" "RESET" (id 1) (at 635 182.88 0))
     (property "Footprint" "Button_Switch_SMD:SW_SPST_B3U-1000P-B" (id 2) (at 635 186.69 0)
       (effects (font (size 1.27 1.27)) hide)
@@
       (effects (font (size 1.27 1.27)) hide)
     )
+    (property "Comment" "" (id 5) (at 635 186.69 0)
+      (effects (font (size 1.27 1.27)) hide)
+    )
     (pin "1")
     (pin "2")
@@
       (effects (font (size 1.27 1.27)) hide)
     )
-    (property "LCSC" "NA" (id 4) (at 510.54 26.67 0)
+    (property "LCSC" "DNP" (id 4) (at 510.54 26.67 0)
       (effects (font (size 1.27 1.27)) hide)
     )
@@
     (pin "9")
   )
-  (symbol (lib_id "hellen-one-mcu-000.4:Module-mcu-0.4") (at 561.34 151.13 0) (unit 4)
+  (symbol (lib_id "hellen-one-mcu-000.5:Module-mcu-0.5") (at 561.34 151.13 0) (unit 4)
     (in_bom yes) (on_board yes)
     (property "Reference" "M11" (id 0) (at 563.88 149.86 0))
-    (property "Value" "Module-mcu-0.4" (id 1) (at 579.12 177.8 0))
-    (property "Footprint" "hellen-one-mcu-0.4:mcu" (id 2) (at 561.34 151.13 0)
+    (property "Value" "Module-mcu-0.5" (id 1) (at 579.12 177.8 0))
+    (property "Footprint" "hellen-one-mcu-0.5:mcu" (id 2) (at 561.34 151.13 0)
       (effects (font (size 1.27 1.27)) hide)
     )
@@
     (pin "W8")
   )
-  (symbol (lib_id "hellen-one-mcu-000.4:Module-mcu-0.4") (at 426.72 303.53 0) (mirror y) (unit 3)
+  (symbol (lib_id "hellen-one-mcu-000.5:Module-mcu-0.5") (at 426.72 303.53 0) (mirror y) (unit 3)
     (in_bom yes) (on_board yes)
     (property "Reference" "M11" (id 0) (at 425.45 302.26 0))
-    (property "Value" "Module-mcu-0.4" (id 1) (at 419.1 401.32 0))
-    (property "Footprint" "hellen-one-mcu-0.4:mcu" (id 2) (at 426.72 303.53 0)
+    (property "Value" "Module-mcu-0.5" (id 1) (at 419.1 401.32 0))
+    (property "Footprint" "hellen-one-mcu-0.5:mcu" (id 2) (at 426.72 303.53 0)
       (effects (font (size 1.27 1.27)) hide)
     )
@@
     (pin "W40")
   )
-  (symbol (lib_id "hellen-one-mcu-000.4:Module-mcu-0.4") (at 433.07 163.83 0) (unit 2)
+  (symbol (lib_id "hellen-one-mcu-000.5:Module-mcu-0.5") (at 433.07 163.83 0) (unit 2)
     (in_bom yes) (on_board yes)
     (property "Reference" "M11" (id 0) (at 440.69 162.56 0))
-    (property "Value" "Module-mcu-0.4" (id 1) (at 440.69 274.32 0))
-    (property "Footprint" "hellen-one-mcu-0.4:mcu" (id 2) (at 433.07 163.83 0)
+    (property "Value" "Module-mcu-0.5" (id 1) (at 440.69 274.32 0))
+    (property "Footprint" "hellen-one-mcu-0.5:mcu" (id 2) (at 433.07 163.83 0)
       (effects (font (size 1.27 1.27)) hide)
     )
@@
     (pin "W8")
   )
-  (symbol (lib_id "hellen-one-mcu-000.4:Module-mcu-0.4") (at 427.99 163.83 0) (mirror y) (unit 1)
+  (symbol (lib_id "hellen-one-mcu-000.5:Module-mcu-0.5") (at 427.99 163.83 0) (mirror y) (unit 1)
     (in_bom yes) (on_board yes)
     (property "Reference" "M11" (id 0) (at 420.37 162.56 0))
-    (property "Value" "Module-mcu-0.4" (id 1) (at 420.37 279.4 0))
-    (property "Footprint" "hellen-one-mcu-0.4:mcu" (id 2) (at 427.99 163.83 0)
+    (property "Value" "Module-mcu-0.5" (id 1) (at 420.37 279.4 0))
+    (property "Footprint" "hellen-one-mcu-0.5:mcu" (id 2) (at 427.99 163.83 0)
       (effects (font (size 1.27 1.27)) hide)
     )
@@
     )
     (path "/dac81d09-2272-472d-95eb-e6a2022d643a"
-      (reference "M11") (unit 1) (value "Module-mcu-0.4") (footprint "hellen-one-mcu-0.4:mcu")
+      (reference "M11") (unit 1) (value "Module-mcu-0.5") (footprint "hellen-one-mcu-0.5:mcu")
     )
     (path "/619fe453-b8d5-43d8-92ff-5dae7989bbfb"
-      (reference "M11") (unit 2) (value "Module-mcu-0.4") (footprint "hellen-one-mcu-0.4:mcu")
+      (reference "M11") (unit 2) (value "Module-mcu-0.5") (footprint "hellen-one-mcu-0.5:mcu")
     )
     (path "/42ac1216-7000-4a29-88d1-3cafdf3bfb7c"
-      (reference "M11") (unit 3) (value "Module-mcu-0.4") (footprint "hellen-one-mcu-0.4:mcu")
+      (reference "M11") (unit 3) (value "Module-mcu-0.5") (footprint "hellen-one-mcu-0.5:mcu")
     )
     (path "/4bb09719-8233-4eff-b783-fe7b9cfa32e1"
-      (reference "M11") (unit 4) (value "Module-mcu-0.4") (footprint "hellen-one-mcu-0.4:mcu")
+      (reference "M11") (unit 4) (value "Module-mcu-0.5") (footprint "hellen-one-mcu-0.5:mcu")
     )
     (path "/252b4f77-58b4-4ba1-a925-b260d38b7d08"
@@
     )
     (path "/6b6d9cce-9449-465a-86d0-676d54a1bd13"
-      (reference "SW1") (unit 1) (value "BOOT0") (footprint "Button_Switch_SMD:SW_SPST_B3U-1000P-B")
+      (reference "SW1") (unit 1) (value "RESET") (footprint "Button_Switch_SMD:SW_SPST_B3U-1000P-B")
     )
     (path "/c7277d80-f3af-46ed-b785-f515ad596404"

Commit message: fix 2 14/08/2021
Parts:
- added G1: Conn_01x01, footprints:LOGO, symbol Connector_Generic:Conn_01x01
- added G2: Conn_01x01, rusefi_lib:LOGO, symbol Connector_Generic:Conn_01x01
- renumbered *ref1 to PP1
Changed lines of the file:
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@@
     (pin "1")
   )
+  (symbol (lib_id "Connector_Generic:Conn_01x01") (at 581.66 558.038 90) (unit 1)
+    (in_bom yes) (on_board yes) (fields_autoplaced)
+    (property "Reference" "G1" (id 0) (at 584.2 558.7999 90)
+      (effects (font (size 1.27 1.27)) (justify right))
+    )
+    (property "Value" "Conn_01x01" (id 1) (at 584.2 561.3399 90)
+      (effects (font (size 1.27 1.27)) (justify right))
+    )
+    (property "Footprint" "footprints:LOGO" (id 2) (at 581.66 558.038 0)
+      (effects (font (size 1.27 1.27)) hide)
+    )
+    (property "Datasheet" "~" (id 3) (at 581.66 558.038 0)
+      (effects (font (size 1.27 1.27)) hide)
+    )
+    (pin "1")
+  )
+  (symbol (lib_id "Connector_Generic:Conn_01x01") (at 598.678 558.038 90) (unit 1)
+    (in_bom yes) (on_board yes) (fields_autoplaced)
+    (property "Reference" "G2" (id 0) (at 601.218 558.7999 90)
+      (effects (font (size 1.27 1.27)) (justify right))
+    )
+    (property "Value" "Conn_01x01" (id 1) (at 601.218 561.3399 90)
+      (effects (font (size 1.27 1.27)) (justify right))
+    )
+    (property "Footprint" "rusefi_lib:LOGO" (id 2) (at 598.678 558.038 0)
+      (effects (font (size 1.27 1.27)) hide)
+    )
+    (property "Datasheet" "~" (id 3) (at 598.678 558.038 0)
+      (effects (font (size 1.27 1.27)) hide)
+    )
+    (pin "1")
+  )
   (symbol (lib_id "Connector_Generic:Conn_01x01") (at 605.79 369.57 0) (unit 1)
     (in_bom yes) (on_board yes)
@@
   (symbol (lib_id "motronic_88pin_STS:Motronic_88pin") (at 33.02 148.59 90) (mirror x) (unit 2)
     (in_bom yes) (on_board yes)
-    (property "Reference" "*ref1" (id 0) (at 18.669 182.5498 0))
+    (property "Reference" "PP1" (id 0) (at 18.669 182.5498 0))
     (property "Value" "Motronic_88pin" (id 1) (at 20.9804 182.5498 0))
     (property "Footprint" "rusefi_lib_private:88pin_STS" (id 2) (at 21.59 183.515 0)
@@
   (symbol (lib_id "motronic_88pin_STS:Motronic_88pin") (at 33.02 71.12 90) (mirror x) (unit 1)
     (in_bom yes) (on_board yes)
-    (property "Reference" "*ref1" (id 0) (at 18.669 105.0798 0))
+    (property "Reference" "PP1" (id 0) (at 18.669 105.0798 0))
     (property "Value" "Motronic_88pin" (id 1) (at 20.9804 105.0798 0))
     (property "Footprint" "rusefi_lib_private:88pin_STS" (id 2) (at 21.59 106.045 0)
@@
   (symbol (lib_id "motronic_88pin_STS:Motronic_88pin") (at 33.02 222.25 90) (mirror x) (unit 3)
     (in_bom yes) (on_board yes)
-    (property "Reference" "*ref1" (id 0) (at 18.669 287.401 0))
+    (property "Reference" "PP1" (id 0) (at 18.669 287.401 0))
     (property "Value" "Motronic_88pin" (id 1) (at 20.9804 287.401 0))
     (property "Footprint" "rusefi_lib_private:88pin_STS" (id 2) (at 21.59 257.175 0)
@@
       (reference "#PWR0171") (unit 1) (value "V5A") (footprint "")
     )
-    (path "/00000000-0000-0000-0000-00005f7b99ce"
-      (reference "*ref1") (unit 1) (value "Motronic_88pin") (footprint "rusefi_lib_private:88pin_STS")
-    )
-    (path "/00000000-0000-0000-0000-00005f844f8b"
-      (reference "*ref1") (unit 2) (value "Motronic_88pin") (footprint "rusefi_lib_private:88pin_STS")
-    )
-    (path "/00000000-0000-0000-0000-00005f83acfe"
-      (reference "*ref1") (unit 3) (value "Motronic_88pin") (footprint "rusefi_lib_private:88pin_STS")
-    )
     (path "/00000000-0000-0000-0000-00006009e992"
       (reference "C1") (unit 1) (value "100nF") (footprint "Capacitor_SMD:C_0402_1005Metric")
@@
       (reference "D33") (unit 1) (value "1N4148WS") (footprint "Diode_SMD:D_SOD-323")
     )
+    (path "/16efd94d-045d-4f40-92e4-a8538f713373"
+      (reference "G1") (unit 1) (value "Conn_01x01") (footprint "footprints:LOGO")
+    )
+    (path "/9fd786cd-127c-4de7-a85c-e114caa86ada"
+      (reference "G2") (unit 1) (value "Conn_01x01") (footprint "rusefi_lib:LOGO")
+    )
     (path "/00000000-0000-0000-0000-000060dbb771"
       (reference "H1") (unit 1) (value "MountingHole") (footprint "MountingHole:MountingHole_4.3mm_M4_DIN965")
@@
       (reference "P6") (unit 1) (value "P") (footprint "Connector_Pin:Pin_D1.0mm_L10.0mm")
     )
+    (path "/00000000-0000-0000-0000-00005f7b99ce"
+      (reference "PP1") (unit 1) (value "Motronic_88pin") (footprint "rusefi_lib_private:88pin_STS")
+    )
+    (path "/00000000-0000-0000-0000-00005f844f8b"
+      (reference "PP1") (unit 2) (value "Motronic_88pin") (footprint "rusefi_lib_private:88pin_STS")
+    )
+    (path "/00000000-0000-0000-0000-00005f83acfe"
+      (reference "PP1") (unit 3) (value "Motronic_88pin") (footprint "rusefi_lib_private:88pin_STS")
+    )
     (path "/00000000-0000-0000-0000-00005fc69d39"

Commit message: 15/08/2021
Parts:
- M11: value Module-mcu-0.5 -> Module-mcu144-0.5
Changed lines of the file:
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@@
     (in_bom yes) (on_board yes)
     (property "Reference" "M11" (id 0) (at 563.88 149.86 0))
-    (property "Value" "Module-mcu-0.5" (id 1) (at 579.12 177.8 0))
+    (property "Value" "Module-mcu144-0.5" (id 1) (at 579.12 177.8 0))
     (property "Footprint" "hellen-one-mcu-0.5:mcu" (id 2) (at 561.34 151.13 0)
       (effects (font (size 1.27 1.27)) hide)
@@
     (in_bom yes) (on_board yes)
     (property "Reference" "M11" (id 0) (at 425.45 302.26 0))
-    (property "Value" "Module-mcu-0.5" (id 1) (at 419.1 401.32 0))
+    (property "Value" "Module-mcu144-0.5" (id 1) (at 419.1 401.32 0))
     (property "Footprint" "hellen-one-mcu-0.5:mcu" (id 2) (at 426.72 303.53 0)
       (effects (font (size 1.27 1.27)) hide)
@@
     (in_bom yes) (on_board yes)
     (property "Reference" "M11" (id 0) (at 440.69 162.56 0))
-    (property "Value" "Module-mcu-0.5" (id 1) (at 440.69 274.32 0))
+    (property "Value" "Module-mcu144-0.5" (id 1) (at 440.69 274.32 0))
     (property "Footprint" "hellen-one-mcu-0.5:mcu" (id 2) (at 433.07 163.83 0)
       (effects (font (size 1.27 1.27)) hide)
@@
     (in_bom yes) (on_board yes)
     (property "Reference" "M11" (id 0) (at 420.37 162.56 0))
-    (property "Value" "Module-mcu-0.5" (id 1) (at 420.37 279.4 0))
+    (property "Value" "Module-mcu144-0.5" (id 1) (at 420.37 279.4 0))
     (property "Footprint" "hellen-one-mcu-0.5:mcu" (id 2) (at 427.99 163.83 0)
       (effects (font (size 1.27 1.27)) hide)
@@
     )
     (path "/dac81d09-2272-472d-95eb-e6a2022d643a"
-      (reference "M11") (unit 1) (value "Module-mcu-0.5") (footprint "hellen-one-mcu-0.5:mcu")
+      (reference "M11") (unit 1) (value "Module-mcu144-0.5") (footprint "hellen-one-mcu-0.5:mcu")
     )
     (path "/619fe453-b8d5-43d8-92ff-5dae7989bbfb"
-      (reference "M11") (unit 2) (value "Module-mcu-0.5") (footprint "hellen-one-mcu-0.5:mcu")
+      (reference "M11") (unit 2) (value "Module-mcu144-0.5") (footprint "hellen-one-mcu-0.5:mcu")
     )
     (path "/42ac1216-7000-4a29-88d1-3cafdf3bfb7c"
-      (reference "M11") (unit 3) (value "Module-mcu-0.5") (footprint "hellen-one-mcu-0.5:mcu")
+      (reference "M11") (unit 3) (value "Module-mcu144-0.5") (footprint "hellen-one-mcu-0.5:mcu")
     )
     (path "/4bb09719-8233-4eff-b783-fe7b9cfa32e1"
-      (reference "M11") (unit 4) (value "Module-mcu-0.5") (footprint "hellen-one-mcu-0.5:mcu")
+      (reference "M11") (unit 4) (value "Module-mcu144-0.5") (footprint "hellen-one-mcu-0.5:mcu")
     )
     (path "/252b4f77-58b4-4ba1-a925-b260d38b7d08"

Commit message: BOM fix
Parts:
- J20: value ETB_6p -> ETB; LCSC (none) -> C343639
- J21: value ETB_4p -> ETB; LCSC (none) -> C343639
Changed lines of the file:
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@@
       (effects (font (size 1.27 1.27)) (justify left))
     )
-    (property "Value" "ETB_4p" (id 1) (at 441.198 537.4639 0)
+    (property "Value" "ETB" (id 1) (at 441.198 537.4639 0)
       (effects (font (size 1.27 1.27)) (justify left))
     )
@@
     )
     (property "Datasheet" "~" (id 3) (at 438.658 534.924 0)
+      (effects (font (size 1.27 1.27)) hide)
+    )
+    (property "LCSC" "C343639" (id 4) (at 438.658 534.924 0)
       (effects (font (size 1.27 1.27)) hide)
     )
@@
       (effects (font (size 1.27 1.27)) (justify left))
     )
-    (property "Value" "ETB_6p" (id 1) (at 415.29 534.6699 0)
+    (property "Value" "ETB" (id 1) (at 415.29 534.6699 0)
       (effects (font (size 1.27 1.27)) (justify left))
     )
@@
     )
     (property "Datasheet" "~" (id 3) (at 412.75 532.13 0)
+      (effects (font (size 1.27 1.27)) hide)
+    )
+    (property "LCSC" "C343639" (id 4) (at 412.75 532.13 0)
       (effects (font (size 1.27 1.27)) hide)
     )
@@
     )
     (path "/ec8636fb-8f33-480a-80a4-fe4e5c9ee953"
-      (reference "J20") (unit 1) (value "ETB_6p") (footprint "Connector_PinHeader_2.54mm:PinHeader_1x06_P2.54mm_Vertical")
+      (reference "J20") (unit 1) (value "ETB") (footprint "Connector_PinHeader_2.54mm:PinHeader_1x06_P2.54mm_Vertical")
     )
     (path "/ce96e045-4eec-49f9-87cd-8ae99dfc13c8"
-      (reference "J21") (unit 1) (value "ETB_4p") (footprint "Connector_PinHeader_2.54mm:PinHeader_1x04_P2.54mm_Vertical")
+      (reference "J21") (unit 1) (value "ETB") (footprint "Connector_PinHeader_2.54mm:PinHeader_1x04_P2.54mm_Vertical")
     )
     (path "/00000000-0000-0000-0000-00005f7c5b0c"

Commit message: BOM fix 17/08/2021
Parts:
- C10: LCSC C295934 -> C115688
- R25, R26: LCSC C384349 -> C138017
Changed lines of the file:
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@@
       (effects (font (size 1.27 1.27)) hide)
     )
-    (property "LCSC" "C384349" (id 4) (at 67.31 269.24 0)
+    (property "LCSC" "C138017" (id 4) (at 67.31 269.24 0)
       (effects (font (size 1.27 1.27)) hide)
     )
@@
       (effects (font (size 1.27 1.27)) hide)
     )
-    (property "LCSC" "C384349" (id 4) (at 72.39 269.24 0)
+    (property "LCSC" "C138017" (id 4) (at 72.39 269.24 0)
       (effects (font (size 1.27 1.27)) hide)
     )
@@
       (effects (font (size 1.27 1.27)) hide)
     )
-    (property "LCSC" "C295934" (id 4) (at 276.86 570.23 0)
-      (effects (font (size 1.27 1.27)) hide)
-    )
+    (property "LCSC" "C115688" (id 4) (at 276.86 570.23 0)
+      (effects (font (size 1.27 1.27)) hide)
+    )

Commit message: fix schematic and board
Parts:
- removed D3, D8: LED-WHITE-0603, LED_SMD:LED_0603_1608Metric, symbol Device:LED
- removed RN1: 470, Resistor_SMD:R_Array_Concave_4x0603, symbol Device:R_Pack04
- added C22: 100nF, Capacitor_SMD:C_0402_1005Metric, symbol Device:C
- added MMCU16: MMCU, Connector_PinHeader_1.00mm:PinHeader_1x01_P1.00mm_Vertical, symbol Connector_Generic:Conn_01x01
- RN2: value 470 -> 1k; LCSC C25510 -> C20197
Connections:
- net +3V3: now also C22.1
- net COIL_1: no longer D22.2 (A)
- net COIL_2: no longer D21.2 (A)
- net COIL_3: no longer D20.2 (A)
- net COIL_4: no longer D18.2 (A)
- net COIL_5: no longer D16.2 (A)
- net COIL_6: no longer D17.2 (A)
- net COIL_7: no longer D19.2 (A)
- net COIL_8: no longer D23.2 (A)
- net GND: now also C22.2
- net OUT_IGN1: now also D23.2 (A)
- net OUT_IGN2: now also D19.2 (A)
- net OUT_IGN3: now also D22.2 (A)
- net OUT_IGN4: now also D18.2 (A)
- net OUT_IGN5: now also D21.2 (A)
- net OUT_IGN6: now also D17.2 (A)
- net OUT_IGN7: now also D20.2 (A)
- net OUT_IGN8: now also D16.2 (A)
- net V12_PERM: now also JP26.2 (B); no longer M11.S6 (IN_D4)
- net V12_RAW: no longer JP26.2 (B)
- net at D7.1 (K): now also RN4.8 (R1.2)
- new net: M11.S6 (IN_D4), MMCU16.1 (Pin_1)
- no-connect marks 147 -> 144
Other:
- moved on the sheet: D16, D17, D18, D19, D20, D21, D22, D23, D7, RN5, RN6

Commit message: Issues 61,60,59,57,55,54,17,6,13,8,16,12
Parts:
- removed D1, D10, D13, D2: LED-BLUE-0603, LED_SMD:LED_0603_1608Metric, symbol Device:LED
- removed JP14, JP44: Jumper_2_Open, rusefi_lib:SM0805_jumper, symbol Jumper:Jumper_2_Open
- removed MMCU19, MMCU39: MMCU, Connector_PinHeader_1.00mm:PinHeader_1x01_P1.00mm_Vertical, symbol Connector_Generic:Conn_01x01
- removed R27: DNP, Resistor_SMD:R_0402_1005Metric, symbol Device:R
- removed RN2: 1k, Resistor_SMD:R_Array_Concave_4x0603, symbol Device:R_Pack04
- removed VOUT11, VOUT20, VOUT3, VOUT7: Pad, Connector_PinHeader_1.00mm:PinHeader_1x01_P1.00mm_Vertical, symbol hellen-one-common:Pad
- removed cr24, cr9: cr, Connector_PinHeader_1.00mm:PinHeader_1x01_P1.00mm_Vertical, symbol Connector_Generic:Conn_01x01
- added D1, D2, D3, D8: 1N4148WS, Diode_SMD:D_SOD-323, symbol Diode:1N4148WS
- added JP36, JP48, JP6: Jumper_2_Open, rusefi_lib:SM0805_jumper, symbol Jumper:Jumper_2_Open
- added R31: 1k6, Resistor_SMD:R_0402_1005Metric, symbol Device:R
- added R32, R33: 5k1, Resistor_SMD:R_0402_1005Metric, symbol Device:R
- JP20, JP21, JP54: LCSC C17477 -> DNP
- R1, R2: value 2k2 -> 470k; LCSC C114762 -> (none)
- R3: value 2k2 -> 750R; LCSC C114762 -> (none)
Connections:
- net GND_SENS is gone; now on net GND: C1.2, C2.2, J4.1 (Pin_1), U1.3 (GND), U2.2 (GND)
- net +12V: now also D2.1 (K), D3.1 (K), D8.1 (K)
- net +3V3: no longer R1.1
- net BOOT0: no longer R2.1
- net CLT: no longer JP78.2 (B), M7.S15 (IN_CLT), R25.2
- net GND: now also PP1.14, PP1.44, R1.2, R2.2, R31.2, R32.2, R33.2
- net IAT: no longer JP77.2 (B), M7.S16 (IN_IAT), R26.2
- net IN_TPS: now also R1.1
- net MAIN_RELAY: now also M11.E8 (OUT_IO1); no longer JP27.2 (B)
- net OUT_INJ7: now also JP6.1 (A)
- net OUT_MAIN: now also JP27.2 (B); no longer M11.E8 (OUT_IO1)
- net V12_RAW: now also D1.1 (K)
- net at PP1.36: now also JP36.1 (A)
- net at PP1.48: now also JP48.1 (A)
- net EVAP: now reaches M9.W38 (LOW3_DUAL)
- net EVAP: now also M11.E7 (OUT_IO5)
- net at D5.1 (K): now also R31.1
- net at D6.1 (K): now also R3.1
- net AC_COMPR: now reaches M9.W34 (LOW4_DUAL)
- net AC_COMPR: now also M11.E21 (OUT_IO7)
- net OUT_AC_COMPR: now reaches M9.W4 (OUT_LOW4_DUAL)
- net OUT_AC_COMPR: now also JP48.2 (B)
- net at J20.4 (Pin_4), J21.3 (Pin_3), M7.S17 (IN_AUX1): now also R2.1
- net OUT_EVAP: now reaches M9.S7 (OUT_LOW3_DUAL)
- net OUT_EVAP: now also D8.2 (A), JP36.2 (B)
- net at D4.1 (K): now also D2.2 (A), R33.1; no longer R3.1
- net at D12.1 (K): now also D1.2 (A), R32.1; no longer RN4.7 (R2.2)
- new net: D3.2 (A), JP6.2 (B)
- new net IN_CLT: JP78.2 (B), M7.S15 (IN_CLT), R25.2
- new net IN_IAT: JP77.2 (B), M7.S16 (IN_IAT), R26.2
- no-connect marks 144 -> 145
Other:
- moved on the sheet: D12, D4, D5, D6, R3, TP1, TP2, TP3, TP4, VIN21

Commit message: update 28/08/2021
Parts:
- removed MMCU17, MMCU33, MMCU34, MMCU36: MMCU, Connector_PinHeader_1.00mm:PinHeader_1x01_P1.00mm_Vertical, symbol Connector_Generic:Conn_01x01
- removed VIN21, VIN24, VIN25, VIN3: Pad, Connector_PinHeader_1.00mm:PinHeader_1x01_P1.00mm_Vertical, symbol hellen-one-common:Pad
- removed VIN5: VIN5, Connector_PinHeader_1.00mm:PinHeader_1x01_P1.00mm_Vertical, symbol Connector_Generic:Conn_01x01
- removed VIN6: VIN6, Connector_PinHeader_1.00mm:PinHeader_1x01_P1.00mm_Vertical, symbol Connector_Generic:Conn_01x01
- removed VIN7: VIN7, Connector_PinHeader_1.00mm:PinHeader_1x01_P1.00mm_Vertical, symbol Connector_Generic:Conn_01x01
- added D10: 1N4148WS, Diode_SMD:D_SOD-323, symbol Diode:1N4148WS
- added JP14: Jumper_2_Open, rusefi_lib:SM0805_jumper, symbol Jumper:Jumper_2_Open
- added R27, R34, R35, R36, R37, R38, R39, R40, R41: 470k, Resistor_SMD:R_0402_1005Metric, symbol Device:R
- added VIN3: VIN8, Connector_PinHeader_1.00mm:PinHeader_1x01_P1.00mm_Vertical, symbol Connector_Generic:Conn_01x01
Connections:
- net +12V: now also D10.1 (K)
- net GND: now also R27.2, R34.2, R35.2, R36.2, R37.2, R38.2, R39.2, R40.2, R41.2; no longer PP1.14
- net IN_MAF: now also JP14.2 (B)
- net IN_TPS: now also R27.1; no longer J20.3 (Pin_3), J21.2 (Pin_2), R1.1
- net OUT_IDLE: now also D10.2 (A)
- net TPS2: now also M11.S24 (IN_AUX1)
- net IN_TPS3: now reaches M7.S20 (IN_AUX3)
- net IN_TPS3: now also J20.3 (Pin_3), R34.1
- net at M7.S21 (IN_AUX4): now also R36.1, VIN3.1 (Pin_1)
- net at M7.S2 (IN_SENS2), VIN9.1 (Pin_1): now also R39.1
- net SENS4: now reaches M7.N23 (SENS4)
- net SENS4: now also M11.S11 (IN_SENS4)
- net SENS2: now reaches M11.S9 (IN_SENS2)
- net SENS2: now also M7.N25 (SENS2)
- net at M7.S1 (IN_SENS1), VIN8.1 (Pin_1): now also R37.1
- net IN_PPS1: now reaches J21.3 (Pin_3), R2.1
- net IN_PPS1: now also M7.S24 (IN_PPS); no longer J20.4 (Pin_4), M7.S17 (IN_AUX1)
- net IN_PPS2: now reaches M7.S18 (IN_AUX2)
- net IN_PPS2: now also J21.2 (Pin_2), R35.1
- net at M7.S25 (IN_O2S2), VIN1.1 (Pin_1): now also R40.1
- net at M7.S4 (IN_SENS4), VIN10.1 (Pin_1): now also R41.1
- net at M7.S9 (IN_O2S), VIN18.1 (Pin_1): now also R38.1
- net SENS1: now reaches M11.S8 (IN_SENS1)
- net SENS1: now also M7.N26 (SENS1)
- net A3 renamed TPS3
- new net: JP14.1 (A), PP1.14
- new net IN_TPS2: J20.4 (Pin_4), M7.S17 (IN_AUX1), R1.1
Other:
- moved on the sheet: R1, R2, VIN1, VIN10, VIN18, VIN22, VIN8, VIN9
