File: hellen88bmw.kicad_sch (KiCad schematic)
At the start: 306 parts, among them J1 920-462A2021Y10101, J10 Conn_01x12, J11 Conn_01x12, J12 Conn_01x12, J13 Conn_01x12, J14 VRIN1, J15 VRIN2, J16 VROUT1, J17 XH-8A, J18 PJ-3250-5A, J19 MiniFit, J2 UB-20PMFP-LC7002, J20 ETB, J21 ETB, J3 Micro_SD_Card, J4 Conn_01x05, J5 Conn_01x12, J6 Conn_01x12, J7 Conn_01x12, J8 Conn_01x12, J9 Conn_01x12, M1 Module-power12-0.2, M10 Module-ign8-0.1, M11 Module-mcu144-0.5, M12 Module-knock-0.1, M2 Module-can-0.1, M3 Module-wbo-0.2, M4 Module-can-0.1, M5 Module-power5-0.2, M6 Module-vr-0.1, M7 Module-input-0.1, M8 Module-knock-0.1, M9 Module-output-0.2, P1 P, P2 P, P3 P, P4 P, P5 P, P6 P, Q1 NGD8201AN, Q2 NGD8201AN, Q3 NGD8201AN, Q4 NGD8201AN, Q5 NGD8201AN, Q6 NGD8201AN, Q7 NGD8201AN, Q8 NGD8201AN, SW1 RESET, SW2 RESET, U1 MPXA6115A, U2 MPX4_MAP, U3 LIS2DW12TR, U4 LPS25HB, U5 MCP6002-xSN, U6 L6205PD

Commit message: update 29/08/2021
Parts:
- removed D14: LED-BLUE-0603, LED_SMD:LED_0603_1608Metric, symbol Device:LED
- removed RN4: 470, Resistor_SMD:R_Array_Concave_4x0603, symbol Device:R_Pack04
- added D13, D14, D34, D35, D36, D37, D38, D39, D40, D41, D42, D43: 1N4148WS, Diode_SMD:D_SOD-323, symbol Diode:1N4148WS
- added D44: B5819W, Diode_SMD:D_SOD-123, symbol Diode:1N4148WS
- added R42: 4.7k, Resistor_SMD:R_0402_1005Metric, symbol Device:R
- added R43: 5k1, Resistor_SMD:R_0402_1005Metric, symbol Device:R
- added cr9: cr, Connector_PinHeader_1.00mm:PinHeader_1x01_P1.00mm_Vertical, symbol Connector_Generic:Conn_01x01
- D10, D3, D8: value 1N4148WS -> B5819W; footprint Diode_SMD:D_SOD-323 -> Diode_SMD:D_SOD-123; LCSC C2128 -> C8598
- RN3: value 470 -> 20k; LCSC C25510 -> C12004
- RN7, RN8: value 470 -> 4.7k; LCSC C25510 -> C1980
Connections:
- net +12V: now also RN3.1 (R1.1), RN3.2 (R2.1), RN3.3 (R3.1), RN3.4 (R4.1), RN7.1 (R1.1), RN7.2 (R2.1), RN7.3 (R3.1), RN7.4 (R4.1), RN8.1 (R1.1), RN8.2 (R2.1), RN8.3 (R3.1), RN8.4 (R4.1), D44.1 (K)
- net +5V: now also R42.1
- net GND: now also JP46.1 (A), PP1.46, R43.2, cr9.1 (Pin_1); no longer PP1.44, PP1.45, RN3.1 (R1.1), RN3.2 (R2.1), RN3.3 (R3.1), RN3.4 (R4.1), RN7.1 (R1.1), RN7.2 (R2.1), RN7.3 (R3.1), RN7.4 (R4.1), RN8.1 (R1.1), RN8.2 (R2.1), RN8.3 (R3.1), RN8.4 (R4.1)
- net INJ1: no longer D24.2 (A)
- net INJ2: no longer D28.2 (A)
- net INJ3: no longer D25.2 (A)
- net INJ4: no longer D29.2 (A)
- net INJ5: no longer D26.2 (A)
- net INJ6: no longer D30.2 (A)
- net INJ7: no longer D27.2 (A)
- net INJ8: no longer D31.2 (A)
- net IN_CRANK: now also D7.1 (K), D42.2 (A); no longer D7.2 (A)
- net MAIN_RELAY: now also D43.1 (K)
- net OUT_INJ1: now also D24.1 (K), D13.2 (A)
- net OUT_INJ2: now also D28.1 (K), D14.2 (A)
- net OUT_INJ3: now also D25.1 (K), D34.2 (A)
- net OUT_INJ4: now also D29.1 (K), D35.2 (A)
- net OUT_INJ5: now also D26.1 (K), D36.2 (A)
- net OUT_INJ6: now also D30.1 (K), D37.2 (A)
- net OUT_INJ7: now also D27.1 (K), D38.2 (A)
- net OUT_INJ8: now also D31.1 (K), D39.2 (A)
- net OUT_PUMP: now also D15.1 (K), D40.2 (A); no longer D15.2 (A)
- net PUMP: now also D9.1 (K), D41.2 (A); no longer D9.2 (A)
- net at PP1.2, cr4.1 (Pin_1): now also D44.2 (A)
- net at RN7.5 (R4.2): now also D24.2 (A), D13.1 (K); no longer D24.1 (K)
- net at RN7.6 (R3.2): now also D28.2 (A), D14.1 (K); no longer D28.1 (K)
- net at RN3.5 (R4.2): now also D15.2 (A), D40.1 (K); no longer D9.1 (K)
- net at RN3.8 (R1.2): now also D9.2 (A), D41.1 (K)
- net at RN8.5 (R4.2): now also D26.2 (A), D36.1 (K); no longer D26.1 (K)
- net at RN8.6 (R3.2): now also D30.2 (A), D37.1 (K); no longer D30.1 (K)
- net at RN7.7 (R2.2): now also D25.2 (A), D34.1 (K); no longer D25.1 (K)
- net at RN8.7 (R2.2): now also D27.2 (A), D38.1 (K); no longer D27.1 (K)
- net at RN8.8 (R1.2): now also D31.2 (A), D39.1 (K); no longer D31.1 (K)
- net at D11.1 (K): now also D43.2 (A), R43.1
- net at RN7.8 (R1.2): now also D29.2 (A), D35.1 (K); no longer D29.1 (K)
- new net: PP1.44, PP1.45
- new net: D42.1 (K), D7.2 (A), R42.2
- no-connect marks 145 -> 144
Other:
- moved on the sheet: D11, D15, D24, D25, D28, D29, D7, D9, RN3, RN7, cr4

Commit message: update 31/08/2021
Parts:
- removed MMCU21: MMCU, Connector_PinHeader_1.00mm:PinHeader_1x01_P1.00mm_Vertical, symbol Connector_Generic:Conn_01x01
- removed R27, R34, R35, R36, R37, R38, R39, R40, R41: 470k, Resistor_SMD:R_0402_1005Metric, symbol Device:R
- removed VIN11: VIN11, Connector_PinHeader_1.00mm:PinHeader_1x01_P1.00mm_Vertical, symbol Connector_Generic:Conn_01x01
- removed VIN12: VIN12, Connector_PinHeader_1.00mm:PinHeader_1x01_P1.00mm_Vertical, symbol Connector_Generic:Conn_01x01
- removed VIN13: VIN13, Connector_PinHeader_1.00mm:PinHeader_1x01_P1.00mm_Vertical, symbol Connector_Generic:Conn_01x01
- removed VIN14: VIN14, Connector_PinHeader_1.00mm:PinHeader_1x01_P1.00mm_Vertical, symbol Connector_Generic:Conn_01x01
- removed VIN15: VIN15, Connector_PinHeader_1.00mm:PinHeader_1x01_P1.00mm_Vertical, symbol Connector_Generic:Conn_01x01
- added Q10, Q9: ZXMS6005SGTA, Package_TO_SOT_SMD:SOT-223, symbol ZXMS6005SGTA:ZXMS6005SGTA
- added R27, R34: 2k7, Resistor_SMD:R_0402_1005Metric, symbol hellen-one-common:Res
- added VOUT3, VOUT7: Pad, Connector_PinHeader_1.00mm:PinHeader_1x01_P1.00mm_Vertical, symbol hellen-one-common:Pad
- R1, R2: value 470k -> 10k; LCSC (none) -> C60489
Connections:
- net GND: now also PP1.44, PP1.45, R1.1, R2.1, Q10.3 (S_1), Q10.4 (S_2), Q9.3 (S_1), Q9.4 (S_2); no longer JP46.1 (A), PP1.46, R1.2, R2.2, cr9.1 (Pin_1)
- net GNDA: now also M7.J10 (PULL_AUX1), M7.J19 (PULL_TPS), M7.J20 (PULL_O2S), M7.J23 (PULL_SENS4), M7.J25 (PULL_SENS2), M7.J26 (PULL_SENS1), M7.J5 (PULL_PPS), M7.J7 (PULL_AUX4), M7.J9 (PULL_AUX2)
- net IDLE: now also R2.2, Q9.1 (IN); no longer M9.W21 (LOW1)
- net IN_CLT: now also R34.2
- net IN_IAT: now also R27.2
- net IN_PPS1: no longer R2.1
- net IN_TPS2: no longer R1.1
- net OUT_IDLE: now also Q9.2 (D); no longer M9.S8 (OUT_LOW1)
- net V5A: now also R27.1, R34.1; no longer M7.J10 (PULL_AUX1), M7.J19 (PULL_TPS), M7.J20 (PULL_O2S), M7.J5 (PULL_PPS), M7.J7 (PULL_AUX4), M7.J9 (PULL_AUX2)
- net at D44.2 (A), PP1.2, cr4.1 (Pin_1): now also Q10.2 (D)
- net ICV: now reaches M11.E28 (OUT_PWM8)
- net ICV: now also R1.2, Q10.1 (IN)
- new net: JP46.1 (A), PP1.46, cr9.1 (Pin_1)
- new net: M9.W21 (LOW1), VOUT7.1 (Pin_1)
- new net: M9.S8 (OUT_LOW1), VOUT3.1 (Pin_1)
- no-connect marks 144 -> 146
Other:
- moved on the sheet: D10, D44, JP2, cr4

Commit message: lib update 31/08/2021 2
Connections:
- net V12_RAW: no longer JP2.1 (A)
- net at JP56.1 (A), PP1.56: now also JP2.1 (A)
Changed lines of the file:
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@@
 (kicad_sch (version 20210621) (generator eeschema)
   (paper "A1")
+  (junction (at 39.624 222.25) (diameter 0.9144) (color 0 0 0 0))
   (junction (at 39.878 191.77) (diameter 0.9144) (color 0 0 0 0))
-  (junction (at 52.07 222.25) (diameter 0.9144) (color 0 0 0 0))
   (junction (at 54.61 86.36) (diameter 0.9144) (color 0 0 0 0))
   (junction (at 67.31 278.13) (diameter 0.9144) (color 0 0 0 0))
@@
     (stroke (width 0) (type solid) (color 0 0 0 0))
   )
+  (wire (pts (xy 39.624 222.25) (xy 33.02 222.25))
+    (stroke (width 0) (type solid) (color 0 0 0 0))
+  )
+  (wire (pts (xy 39.624 226.06) (xy 39.624 222.25))
+    (stroke (width 0) (type solid) (color 0 0 0 0))
+  )
+  (wire (pts (xy 39.624 226.06) (xy 57.15 226.06))
+    (stroke (width 0) (type solid) (color 0 0 0 0))
+  )
   (wire (pts (xy 39.878 187.452) (xy 39.878 191.77))
     (stroke (width 0) (type solid) (color 0 0 0 0))
@@
     (stroke (width 0) (type solid) (color 0 0 0 0))
   )
-  (wire (pts (xy 40.64 222.25) (xy 33.02 222.25))
+  (wire (pts (xy 40.64 222.25) (xy 39.624 222.25))
     (stroke (width 0) (type solid) (color 0 0 0 0))
   )
@@
     (stroke (width 0) (type solid) (color 0 0 0 0))
   )
-  (wire (pts (xy 52.07 226.06) (xy 52.07 222.25))
-    (stroke (width 0) (type solid) (color 0 0 0 0))
-  )
   (wire (pts (xy 54.61 86.36) (xy 73.66 86.36))
     (stroke (width 0) (type solid) (color 0 0 0 0))
@@
     (stroke (width 0) (type solid) (color 0 0 0 0))
   )
-  (wire (pts (xy 57.15 226.06) (xy 52.07 226.06))
-    (stroke (width 0) (type solid) (color 0 0 0 0))
-  )

Commit message: lib update 31/08/2021 2
Parts:
- removed D41: 1N4148WS, Diode_SMD:D_SOD-323, symbol Diode:1N4148WS
- removed D9: LED-BLUE-0603, LED_SMD:LED_0603_1608Metric, symbol Device:LED
- removed R16: 4k7, Resistor_SMD:R_0402_1005Metric, symbol Device:R
- removed RN3: 20k, Resistor_SMD:R_Array_Concave_4x0603, symbol Device:R_Pack04
- R15: value 4k7 -> 20k; LCSC C163826 -> C25765
- R27, R34: LCSC (none) -> C138017
- R3: LCSC (none) -> C25132
- R31: LCSC (none) -> C25931
- R32, R33, R43: LCSC (none) -> C25941
- R42: LCSC (none) -> C25940
- RN5, RN6: value 470 -> 1k; LCSC C25510 -> C240722
Connections:
- net +12V: now also R15.1
- net +3V3: no longer R15.1
- net LPS_SDA: no longer R15.2
- net OUT_ICV: now reaches D44.2 (A), PP1.2, Q10.2 (D), cr4.1 (Pin_1)
- net at D15.2 (A), D40.1 (K): now also R15.2
Other:
- company: (none) -> andreika @ rusEFI.com
- title: (none) -> Hellen88bmw
- moved on the sheet: D15, D40, D42, D7, D8, R42, VIN1, VIN10, VIN18, VIN3, VIN8, VIN9

Commit message: pcb board
Parts:
- removed J10, J11, J12, J13: Conn_01x12, Connector_PinHeader_2.54mm:PinHeader_1x12_P2.54mm_Vertical, symbol Connector_Generic:Conn_01x12
- added G3: Conn_01x01, rusefi_lib:LOGO, symbol Connector_Generic:Conn_01x01
- added G4: Conn_01x01, footprints:LOGO, symbol Connector_Generic:Conn_01x01
- C1, C18, C2, C20, C22, C3, C4, C5, C6: LCSC C105882 -> C307331
- C11, C13, C14, C16, C17, C19, C21, C7, C8, C9: LCSC C87152 -> C96446
- C15: LCSC C106258 -> C16772
- D10, D3, D44, D8: value B5819W -> B5819W
- J2: value UB-20PMFP-LC7002 -> DNP
- JP20, JP21, JP54, JP6: value Jumper_2_Open -> DNP
- Q10, Q9: LCSC С174042 -> C174042
Connections:
- no-connect marks 146 -> 102
Other:
- note added: "1 | Fuel pump 2 | ICV 3 | Inj 5 4 | Inj 6 5 | Inj 4 6 | GND 7 | VVT Solenoid | Inj7 8 | 9 | X 10 | X 11 | NC 12 | NC 13 | NC 14 | GND | MAF gnd 15 | GND 16 | IN CRANK+ 17 | IN CAM 18 | NC 19 | NC 20 | USB_D+ 21 | USB_D- 22 | COIL 7 23 | COIL 4 24 | COIL 6 25 | COIL 5 26 | V12_PERM 27 | OUT_MAIN 28 | GND 29 | OUT IDLE 30 | NC 31 | INJ 3 32 | INJ 2 33 | INJ 1 34 | GND 35 | INJ 8 36 | EVAP 37 | 38 |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"
- note removed: "1 | Fuel pump 2 | NC 3 | Inj 5 4 | Inj 6 5 | Inj 4 6 | GND 7 | VVT Solenoid | Inj7 8 | NC 9 | X 10 | X 11 | NC 12 | NC 13 | NC 14 | GND | MAF gnd 15 | GND 16 | IN CRANK+ 17 | IN CAM 18 | NC 19 | NC 20 | USB_D+ 21 | USB_D- 22 | COIL 7 23 | COIL 4 24 | COIL 6 25 | COIL 5 26 | 12v+ 27 | DME Relay 28 | GND 29 | OUT IDLE 30 | NC 31 | INJ 3 32 | INJ 2 33 | INJ 1 34 | GND 35 | INJ 8 36 | NC 37 | NC 38 |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"
- moved on the sheet: J4, J5, J6, J7, J8, J9

Commit message: Sch refactoring
Parts:
- removed C22, C5: 100nF, Capacitor_SMD:C_0402_1005Metric, symbol Device:C
- removed D10, D44: B5819W, Diode_SMD:D_SOD-123, symbol Diode:1N4148WS
- removed J3: Micro_SD_Card, rusefi_lib_private:693072010801, symbol Connector:Micro_SD_Card
- removed Q10, Q9: ZXMS6005SGTA, Package_TO_SOT_SMD:SOT-223, symbol ZXMS6005SGTA:ZXMS6005SGTA
- removed U3: LIS2DW12TR, kicad6:LGA12R50P4X4_200X200X70, symbol LIS2DW12TR:LIS2DW12TR
- added C?: 100n, hellen-one-common:C0603, symbol hellen-one-common:Cap
- added D10, D44: B5819W, Diode_SMD:D_SOD-123, symbol hellen-one-common:1N4148WS
- added J?: Conn_01x06, Connector_PinHeader_2.54mm:PinHeader_1x06_P2.54mm_Vertical, symbol Connector_Generic:Conn_01x06
- added M?: Module-sd-0.1, hellen-one-sd-0.1:sd, symbol hellen-one-sd-0.1:Module-sd-0.1
- added Q10, Q9: AUIPS2041L, Package_TO_SOT_SMD:SOT-223, symbol Power_Management:AUIPS2041L
- added U3: LIS2DW12TR, hellen-one-common:LGA-12_2x2mm_P0.5mm, symbol hellen-one-common:LIS2DW12TR
Connections:
- net +12V: now also D10.1 (K), D44.1 (K)
- net +3V3: now also C?.2, J?.1 (Pin_1), M?.V1 (V33), U3.10 (Vdd_IO), U3.9 (Vdd)
- net GND: now also C?.1, J?.6 (Pin_6), M?.G (GND), M?.V2 (GND), M?.V3 (GND), Q10.3 (S), Q9.3 (S), U3.6 (GND), U3.7 (RES), U3.8 (GND)
- net ICV: now also Q10.1 (IN)
- net IDLE: now also Q9.1 (IN)
- net IN_CRANK+: no longer M6.E2 (IN_VR1+)
- net IN_CRANK-: no longer M6.E1 (IN_VR1-)
- net IN_KNOCK1_RAW: no longer KNOCK_RAW1.1 (Pin_1), M8.W1 (IN_KNOCK)
- net IN_KNOCK2_RAW: no longer KNOCK_RAW2.1 (Pin_1), M12.W1 (IN_KNOCK)
- net OUT_ICV: now also D44.2 (A), Q10.2 (D)
- net OUT_IDLE: now also D10.2 (A), Q9.2 (D)
- net SD_CLK: now also M?.V6 (SD_SCK)
- net SD_CS: now also J?.2 (Pin_2), M?.V4 (SD_CS)
- net SD_MISO: now also J?.5 (Pin_5), M?.V7 (SD_MISO)
- net SD_MOSI: now also J?.3 (Pin_3), M?.V5 (SD_MOSI)
- net SPI_CS: now also U3.2 (~CS)
- net SPI_MISO: now also U3.3 (SA0/SDO)
- net SPI_MOSI: now also U3.4 (SDA/SDI)
- net SPI_SCK: now also U3.1 (SCL/SPC)
- new net: KNOCK_RAW2.1 (Pin_1), M12.W1 (IN_KNOCK)
- new net: KNOCK_RAW1.1 (Pin_1), M8.W1 (IN_KNOCK)
- new net SD_SCK: J?.4 (Pin_4)
- no-connect marks 102 -> 101
Other:
- note added: "Accelerometer"
- note added: "Baro"
- note added: "Internal pullups"
- moved on the sheet: C1, C2, C3, C4, C6, C7, C8, D1, D11, D12, D13, D14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

Commit message: Sch refactoring
Parts:
- removed R25, R26: 2k7, Resistor_SMD:R_0402_1005Metric, symbol Device:R
- P10: renamed from VOUT1; footprint Connector_PinHeader_1.00mm:PinHeader_1x01_P1.00mm_Vertical -> hellen-one-common:PAD-TH
- P11: renamed from VOUT2; footprint Connector_PinHeader_1.00mm:PinHeader_1x01_P1.00mm_Vertical -> hellen-one-common:PAD-TH
- P12: renamed from VOUT17; footprint Connector_PinHeader_1.00mm:PinHeader_1x01_P1.00mm_Vertical -> hellen-one-common:PAD-TH
- P13: renamed from VOUT16; footprint Connector_PinHeader_1.00mm:PinHeader_1x01_P1.00mm_Vertical -> hellen-one-common:PAD-TH
- P14: renamed from VOUT18; footprint Connector_PinHeader_1.00mm:PinHeader_1x01_P1.00mm_Vertical -> hellen-one-common:PAD-TH
- P15: renamed from VIN19; footprint Connector_PinHeader_1.00mm:PinHeader_1x01_P1.00mm_Vertical -> hellen-one-common:PAD-TH
- P16: renamed from VIN20; footprint Connector_PinHeader_1.00mm:PinHeader_1x01_P1.00mm_Vertical -> hellen-one-common:PAD-TH
- P17: renamed from VIN4; footprint Connector_PinHeader_1.00mm:PinHeader_1x01_P1.00mm_Vertical -> hellen-one-common:PAD-TH
- P18: renamed from VIN18; footprint Connector_PinHeader_1.00mm:PinHeader_1x01_P1.00mm_Vertical -> hellen-one-common:PAD-TH
- P19: renamed from VIN1; footprint Connector_PinHeader_1.00mm:PinHeader_1x01_P1.00mm_Vertical -> hellen-one-common:PAD-TH
- P20: renamed from VIN2; footprint Connector_PinHeader_1.00mm:PinHeader_1x01_P1.00mm_Vertical -> hellen-one-common:PAD-TH
- P21: renamed from VOUT24; footprint Connector_PinHeader_1.00mm:PinHeader_1x01_P1.00mm_Vertical -> hellen-one-common:PAD-TH
- P22: renamed from VOUT25; footprint Connector_PinHeader_1.00mm:PinHeader_1x01_P1.00mm_Vertical -> hellen-one-common:PAD-TH
- P23: renamed from VOUT13; footprint Connector_PinHeader_1.00mm:PinHeader_1x01_P1.00mm_Vertical -> hellen-one-common:PAD-TH
- P24: renamed from VOUT12; footprint Connector_PinHeader_1.00mm:PinHeader_1x01_P1.00mm_Vertical -> hellen-one-common:PAD-TH
- P25: renamed from VOUT26; footprint Connector_PinHeader_1.00mm:PinHeader_1x01_P1.00mm_Vertical -> hellen-one-common:PAD-TH
- P26: renamed from VOUT27; footprint Connector_PinHeader_1.00mm:PinHeader_1x01_P1.00mm_Vertical -> hellen-one-common:PAD-TH
- P27: renamed from VOUT28; footprint Connector_PinHeader_1.00mm:PinHeader_1x01_P1.00mm_Vertical -> hellen-one-common:PAD-TH
- P28: renamed from VOUT8; footprint Connector_PinHeader_1.00mm:PinHeader_1x01_P1.00mm_Vertical -> hellen-one-common:PAD-TH
- P29: renamed from VOUT7; footprint Connector_PinHeader_1.00mm:PinHeader_1x01_P1.00mm_Vertical -> hellen-one-common:PAD-TH
- P30: renamed from VOUT10; footprint Connector_PinHeader_1.00mm:PinHeader_1x01_P1.00mm_Vertical -> hellen-one-common:PAD-TH
- P31: renamed from VOUT29; footprint Connector_PinHeader_1.00mm:PinHeader_1x01_P1.00mm_Vertical -> hellen-one-common:PAD-TH
- P32: renamed from VOUT9; footprint Connector_PinHeader_1.00mm:PinHeader_1x01_P1.00mm_Vertical -> hellen-one-common:PAD-TH
- P7: renamed from VOUT3; footprint Connector_PinHeader_1.00mm:PinHeader_1x01_P1.00mm_Vertical -> hellen-one-common:PAD-TH
- P8: renamed from VOUT19; footprint Connector_PinHeader_1.00mm:PinHeader_1x01_P1.00mm_Vertical -> hellen-one-common:PAD-TH
- P9: renamed from VOUT21; footprint Connector_PinHeader_1.00mm:PinHeader_1x01_P1.00mm_Vertical -> hellen-one-common:PAD-TH
- gave numbers to parts that had none: 3
- renumbered PP1 to *ref1
Connections:
- net V5A is gone; now on net +5VA: M11.S33 (V5A), M12.E1 (V5A), M7.E5 (V5A), M7.J1 (PULL_V5A), M7.J17 (PULL_CAM), M7.J18 (PULL_VSS), M7.J21 (PULL_CRANK), M7.N1 (V5A), M8.E1 (V5A), R27.1, R34.1
- net GND: no longer M3.J_GND1 (PULL_DOWN1), M3.J_GND2 (PULL_DOWN2)
- net IN_CRANK+: now also M6.E2 (IN_VR1+)
- net IN_CRANK-: now also M6.E1 (IN_VR1-)
- net IN_KNOCK1_RAW: now also KNOCK_RAW1.1 (Pin_1), M8.W1 (IN_KNOCK)
- net IN_KNOCK2_RAW: now also KNOCK_RAW2.1 (Pin_1), M12.W1 (IN_KNOCK)
- net at M3.J1 (SEL1): now also M3.J_GND1 (PULL_DOWN1)
- net 5V_SENS2 renamed +5VA
- net V12_RAW renamed +12V_RAW
Other:
- note added: "#0"
- note added: "Analog inputs (sensors)"
- note added: "Bus types"
- note added: "Discrete inputs"
- note added: "General purpose bus"
- note added: "Ignition"
- note added: "Injection"
- note added: "LEDs"
- note added: "Ouputs"
- note added: "VVT_AV7"
- moved on the sheet: *ref1A, *ref1B, *ref1C, C1, C10, C11, C12, C13, C14, C15, C16, C17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

Commit message: Sch refactoring
Parts:
- removed JP22, JP23, JP24, JP25, JP49, JP50, JP51, JP52: Jumper_2_Open, rusefi_lib:SM0805_jumper, symbol Jumper:Jumper_2_Open
- removed P10, P11, P12, P13, P14, P20, P7, P8, P9: Pad, hellen-one-common:PAD-TH, symbol hellen-one-common:Pad
- removed R4: 1k, Resistor_SMD:R_0402_1005Metric, symbol Device:R
- removed VIN22: VIN5, Connector_PinHeader_1.00mm:PinHeader_1x01_P1.00mm_Vertical, symbol Connector_Generic:Conn_01x01
- removed VIN3: VIN8, Connector_PinHeader_1.00mm:PinHeader_1x01_P1.00mm_Vertical, symbol Connector_Generic:Conn_01x01
- added F1, F2, F3, F4, F5, F6, F7, F8: 10A, hellen-one-common:36911600000, symbol hellen-one-common:Fuse-Pad-Pad
- added R16, R25, R4: 680k, hellen-one-common:R0603, symbol hellen-one-common:Res
- added R26, R35: DNP, hellen-one-common:R0603, symbol hellen-one-common:Res
- added VIN1: VIN8, Connector_PinHeader_1.00mm:PinHeader_1x01_P1.00mm_Vertical, symbol Connector_Generic:Conn_01x01
- added VOUT1, VOUT10, VOUT11, VOUT2, VOUT3, VOUT7, VOUT8, VOUT9: VOUT4, Connector_PinHeader_1.00mm:PinHeader_1x01_P1.00mm_Vertical, symbol Connector_Generic:Conn_01x01
- R27, R34: value 2k7 -> 2.7k; footprint Resistor_SMD:R_0402_1005Metric -> hellen-one-common:R0603; Comment 0 -> (none); LCSC C138017 -> C13167
- renumbered *ref1 to PP1
Connections:
- net +5V: no longer J20.1 (Pin_1), J20.2 (Pin_2), J21.1 (Pin_1)
- net +5VA: now also J20.1 (Pin_1), J20.2 (Pin_2), J21.1 (Pin_1), M7.J7 (PULL_AUX4), R27.2, R34.2; no longer R27.1, R34.1
- net COIL_1: now also F6.2
- net COIL_2: now also F7.2
- net COIL_3: now also F8.2
- net COIL_4: now also F2.2
- net COIL_5: now also F4.2
- net COIL_6: now also F3.2
- net COIL_7: now also F1.2
- net COIL_8: now also F5.2
- net GNDA: now also R16.1, R25.1, R26.1, R35.1, R4.1; no longer M7.J10 (PULL_AUX1), M7.J24 (PULL_SENS3), M7.J7 (PULL_AUX4), M7.J8 (PULL_AUX3), M7.J9 (PULL_AUX2)
- net IN_CLT: now also R34.1; no longer R34.2
- net IN_IAT: now also R27.1; no longer R27.2
- net IN_KNOCK2: now also R26.2
- net IN_MAF: now also R35.2
- net IN_PPS2: now also R25.2
- net IN_TPS2: now also R4.2
- net IN_TPS3: now also R16.2
- net at PP1.22: now also F1.1
- net at PP1.23: now also F2.1
- net at PP1.24: now also F3.1
- net at PP1.25: now also F4.1
- net at PP1.49: now also F5.1
- net at PP1.50: now also F6.1
- net at PP1.51: now also F7.1
- net at PP1.52: now also F8.1
- net at M7.S19 (IN_MAP3): now also U1.4 (Vout)
- net at M9.S12 (OUT_LOW8_PULLUP): now also VOUT8.1 (Pin_1)
- net at M7.S21 (IN_AUX4): now also VIN1.1 (Pin_1)
- net at M9.S13 (OUT_LOW12): now also VOUT11.1 (Pin_1)
- net at M9.S10 (OUT_LOW11): now also VOUT10.1 (Pin_1)
- net at M9.S14 (OUT_LOW9): now also VOUT9.1 (Pin_1)
- net at M9.S8 (OUT_LOW1): now also VOUT1.1 (Pin_1)
- net at M9.W1 (OUT_LOW2): now also VOUT2.1 (Pin_1)
- net at M9.W3 (OUT_LOW6_DIODE): now also VOUT3.1 (Pin_1)
- net at M9.W9 (OUT_LOW7_PULLUP): now also VOUT7.1 (Pin_1)
- net AUX4: now reaches M7.N7 (AUX4)
- net AUX4: now also M11.S27 (IN_AUX4)
- removed net BARO: M11.S27 (IN_AUX4), U1.4 (Vout)
- no-connect marks 101 -> 105
Other:
- moved on the sheet: C1, U1
