File: hellen88bmw.kicad_sch (KiCad schematic)
At the start: 303 parts, among them J1 USB_B_Mini, J14 VRIN1, J15 VRIN2, J16 VROUT1, J17 XH-8A, J18 AudioJack_THR, J19 MiniFit, J2 Conn_01x05, J20 ETB, J21 PPS, J4 Conn_01x05, M1 Module-power12-0.2, M10 Module-ign8-0.1, M11 Module-mcu144-0.5, M12 Module-knock-0.1, M13 Module-sd-0.1, M2 Module-can-0.1, M3 Module-wbo-0.3, M4 Module-can-0.1, M5 Module-power5-0.2, M6 Module-vr-0.1, M7 Module-input-0.1, M8 Module-knock-0.1, M9 Module-output-0.2, P1 P, P2 P, P3 P, P4 P, P5 P, P6 P, Q1 NGD8201AN, Q10 AUIPS2041LTR, Q2 NGD8201AN, Q3 NGD8201AN, Q4 NGD8201AN, Q5 NGD8201AN, Q6 NGD8201AN, Q7 NGD8201AN, Q8 NGD8201AN, Q9 AUIPS2041LTR, SW1 Button_SPST, SW2 Button_SPST, U1 MPXA6115A, U2 MPX4_MAP, U3 LIS2DW12TR, U4 LPS25HB, U5 MCP6002-xSN, U6 L6205PD

Commit message: Some fixes
#34, #46, #43, #45, #23, #33, #28, #3,  #27, #49, #48, #47, #44, #26
Parts:
- removed M10: Module-ign8-0.1, hellen-one-ign8-0.1:ign8, symbol hellen-one-ign8-0.1:Module-ign8-0.1
- removed M11: Module-mcu144-0.5, hellen-one-mcu-0.5:mcu, symbol hellen-one-mcu-000.5:Module-mcu-0.5
- removed M9: Module-output-0.2, hellen-one-output-0.2:output, symbol hellen-one-output-0.2:Module-output-0.2
- removed VOUT3: VOUT4, Connector_PinHeader_1.00mm:PinHeader_1x01_P1.00mm_Vertical, symbol Connector_Generic:Conn_01x01
- removed cr5: cr, Connector_PinHeader_1.00mm:PinHeader_1x01_P1.00mm_Vertical, symbol Connector_Generic:Conn_01x01
- added C22, C23: 1u, hellen-one-common:C0603, symbol hellen-one-common:Cap
- added JP8: Jumper_2_Open, hellen-one-common:PAD-0805-PAD, symbol hellen-one-common:Jumper-Pad-Pad
- added M10: Module-ign8-0.2, hellen-one-ign8-0.2:ign8, symbol hellen-one-ign8-0.2:Module-ign8-0.2
- added M11: Module-mcu-0.6, hellen-one-mcu-0.6:mcu, symbol hellen-one-mcu-0.6:Module-mcu-0.6
- added M9: Module-output-0.3, hellen-one-output-0.3:output, symbol hellen-one-output-0.3:Module-output-0.3
- added U7: TLS115_SOIC, hellen-one-common:PG-DSO-8-43, symbol hellen-one-common:TLS115
- added U8: TLS115_SON, Package_SON:HVSON-8-1EP_3x3mm_P0.65mm_EP1.6x2.4mm, symbol hellen-one-common:TLS115
- C11, C13, C14, C16, C17, C19, C21, C7, C8, C9: value 10uF -> 10u
- renumbered VOUT1 to VOUT3
Connections:
- net +12V_RAW: now also M9.S11 (V12_RAW)
- net +3V3: now also M11.N16 (V33)
- net +5V: now also M11.S1 (V5), M9.W14 (V5), U7.5 (ADJ), U8.5 (ADJ)
- net +5VA: now also M11.S33 (V5A); no longer J20.1 (Pin_1), J20.2 (Pin_2), J21.1 (Pin_1), JP59.2
- net +ETB: now also M11.E14 (OUT_PWM2)
- net -ETB: now also M11.E15 (OUT_PWM3)
- net 12V_prot: now also C22.2, M9.W5 (V12P), U7.7 (EN), U7.8 (IN), U8.7 (EN), U8.8 (IN)
- net A1: now also M11.S30 (IN_O2S2)
- net A2: now also M11.S22 (IN_MAP3)
- net A4: now also M11.S23 (IN_RES3)
- net AC_COMPR: now also M11.E21 (OUT_IO7), M9.W34 (LOW4_DUAL)
- net AFR: now also M11.S16 (IN_O2S)
- net AUX4: now also M11.S27 (IN_AUX4)
- net BOOT0: now also M11.N28 (BOOT0)
- net CAM: now also M11.S15 (IN_CAM)
- net CAN_RX: now also M11.N2 (CAN_RX)
- net CAN_TX: now also M11.N3 (CAN_TX)
- net CAN_VIO: now also M11.N1 (CAN_VIO)
- net CLT: now also M11.S18 (IN_CLT)
- net CRANK: now also M11.S13 (IN_CRANK)
- net ETB_EN: now also M11.E27 (OUT_PWM1)
- net EVAP: now also M11.E7 (OUT_IO5), M9.W38 (LOW3_DUAL)
- net FUEL_CONSUM: now also M11.E18 (OUT_PWM6), M9.W22 (PP2)
- net GND: now also C22.1, C23.1, M10.G (GND), M11.S2 (GND), M11.S32 (GNDA), M9.G (GND), M9.S3 (GND), U7.3 (GND), U7.9 (GND), U8.3 (GND), U8.9 (GND)
- net IAT: now also M11.S19 (IN_IAT)
- net ICV: now also M11.E28 (OUT_PWM8)
- net IDLE: now also M11.E17 (OUT_PWM5)
- net IGN1: now also M10.V8 (IGN1), M11.W1 (OUT_IGN1)
- net IGN2: now also M10.V7 (IGN2), M11.W2 (OUT_IGN2)
- net IGN3: now also M10.V6 (IGN3), M11.W3 (OUT_IGN3)
- net IGN4: now also M10.V5 (IGN4), M11.W4 (OUT_IGN4)
- net IGN5: now also M10.V4 (IGN5), M11.W5 (OUT_IGN5)
- net IGN6: now also M10.V3 (IGN6), M11.W6 (OUT_IGN6)
- net IGN7: now also M10.V2 (IGN7), M11.W7 (OUT_IGN7)
- net IGN8: now also M10.V1 (IGN8), M11.W8 (OUT_IGN8)
- net IGN_V33: now also M10.V10 (V33), M11.W10 (IGN_V33)
- net IGN_V5: now also M10.V9 (VCC), M11.W9 (IGN_V5)
- net INJ1: now also M11.E25 (OUT_INJ1), M9.W24 (INJ1)
- net INJ2: now also M11.E26 (OUT_INJ2), M9.W23 (INJ2)
- net INJ3: now also M11.E29 (OUT_INJ3), M9.W20 (INJ3)
- net INJ4: now also M11.E30 (OUT_INJ4), M9.W19 (INJ4)
- net INJ5: now also M11.E31 (OUT_INJ5), M9.W18 (INJ5)
- net INJ6: now also M11.E32 (OUT_INJ6), M9.W17 (INJ6)
- net INJ7: now also M11.E33 (OUT_INJ7), M9.W16 (INJ7)
- net INJ8: now also M11.E34 (OUT_INJ8), M9.W15 (INJ8)
- net INK1: now also M11.S12 (IN_KNOCK)
- net INK2: now also M11.S10 (IN_SENS3)
- net IN_CRANK+: now also JP43.2; no longer JP16.2
- net IN_CRANK-: now also JP16.2; no longer JP43.2
- net LPS_SCL: now also M11.N19 (I2C_SCL)
- net LPS_SDA: now also M11.N18 (I2C_SDA)
- net MAF: now also M11.S20 (IN_MAP1)
- net MAIN_RELAY: now also M11.E8 (OUT_IO1), M9.W40 (LOW5_MAIN); no longer D11.2 (A), D43.1 (K)
- net MAP2: now also M11.S21 (IN_MAP2)
- net NRESET: now also M11.N24 (nReset)
- net OUT_AC_COMPR: now also M9.W4 (OUT_LOW4_DUAL)
- net OUT_EVAP: now also M9.S7 (OUT_LOW3_DUAL)
- net OUT_FUEL_CONSUM: now also M9.S6 (OUT_PP2)
- net OUT_IGN1: now also M10.S8 (OUT_IGN1)
- net OUT_IGN2: now also M10.S7 (OUT_IGN2)
- net OUT_IGN3: now also M10.S6 (OUT_IGN3)
- net OUT_IGN4: now also M10.S5 (OUT_IGN4)
- net OUT_IGN5: now also M10.S4 (OUT_IGN5)
- net OUT_IGN6: now also M10.S3 (OUT_IGN6)
- net OUT_IGN7: now also M10.S2 (OUT_IGN7)
- net OUT_IGN8: now also M10.S1 (OUT_IGN8)
- net OUT_INJ1: now also M9.S18 (OUT_INJ1)
- net OUT_INJ2: now also M9.S16 (OUT_INJ2)
- net OUT_INJ3: now also M9.S17 (OUT_INJ3)
- net OUT_INJ4: now also M9.W7 (OUT_INJ4)
- net OUT_INJ5: now also M9.W10 (OUT_INJ5)
- net OUT_INJ6: now also M9.S15 (OUT_INJ6)
- net OUT_INJ7: now also M9.W12 (OUT_INJ7)
- net OUT_INJ8: now also M9.W11 (OUT_INJ8)
- net OUT_TACH: now also M9.W6 (OUT_PP1)
- net PPS1: now also M11.S29 (IN_PPS)
- net PPS2: now also M11.S25 (IN_AUX2)
- net PUMP: now also M11.E6 (OUT_IO3), M9.W26 (LOW10)
- net RES1: now also M11.S28 (IN_RES1)
- net RES2: now also M11.S31 (IN_RES2)
- net SD_CLK: now also M11.N9 (SPI3_SCK)
- net SD_CS: now also M11.N8 (SPI3_CS)
- net SD_MISO: now also M11.N10 (SPI3_MISO)
- net SD_MOSI: now also M11.N11 (SPI3_MOSI)
- net SENS1: now also M11.S8 (IN_SENS1)
- net SENS2: now also M11.S9 (IN_SENS2)
- net SENS4: now also M11.S11 (IN_SENS4)
- net SPI_CS: now also M11.N23 (SPI2_CS)
- net SPI_MISO: now also M11.N21 (SPI2_MISO)
- net SPI_MOSI: now also M11.N22 (SPI2_MOSI)
- net SPI_SCK: now also M11.N20 (SPI2_SCK)
- net TACH: now also M11.E19 (OUT_PWM7), M9.W28 (PP1)
- net TPS: now also M11.S17 (IN_TPS)
- net TPS2: now also M11.S24 (IN_AUX1)
- net TPS3: now also M11.S26 (IN_AUX3)
- net USBM: now also M11.N31 (USB1M)
- net USBP: now also M11.N30 (USB1P)
- net VBAT: now also M11.N17 (VBAT)
- net VBUS: now also M11.N29 (VBUS)
- net VIGN: now also M11.S7 (VIGN)
- net VSS: now also M11.S14 (IN_VSS)
- net at PP1.8: now also JP8.1
- net at MMCU22.1 (Pin_1): now also M11.S3 (IN_D1)
- net at MMCU15.1 (Pin_1): now also M11.E12 (OUT_IO2)
- net at VOUT24.1 (Pin_1): now also M9.W21 (LOW1)
- net at MMCU7.1 (Pin_1): now also M11.N27 (SWO)
- net at VOUT5.1 (Pin_1): now also M9.S9 (OUT_HIGH2)
- net at VOUT9.1 (Pin_1): now also M9.S14 (OUT_LOW9)
- net at MMCU11.1 (Pin_1): now also M11.E3 (SPI1_MOSI)
- net at MMCU27.1 (Pin_1): now also M11.N15 (IO4)
- net at MMCU28.1 (Pin_1): now also M11.E9 (OUT_IO6)
- net at VOUT3.1 (Pin_1): now also M9.W3 (OUT_LOW6_DIODE)
- net at VOUT25.1 (Pin_1): now also M9.W29 (LOW2)
- net at MMCU9.1 (Pin_1): now also M11.E1 (SPI1_SCK)
- net at MMCU1.1 (Pin_1): now also M11.N5 (UART8_RX)
- net at VOUT22.1 (Pin_1): now also M9.S1 (OUT_SOLENOID_A1)
- net at VOUT10.1 (Pin_1): now also M9.S10 (OUT_LOW11)
- net at VOUT8.1 (Pin_1): now also M9.S12 (OUT_LOW8_PULLUP)
- net at VOUT11.1 (Pin_1): now also M9.S13 (OUT_LOW12)
- net at VOUT23.1 (Pin_1): now also M9.S2 (OUT_SOLENOID_A2)
- net at VOUT14.1 (Pin_1): now also M9.S4 (OUT_SOLENOID_B1)
- net at VOUT15.1 (Pin_1): now also M9.S5 (OUT_SOLENOID_B2)
- net at VOUT2.1 (Pin_1): now also M9.W1 (OUT_LOW2)
- net at VOUT4.1 (Pin_1): now also M9.W8 (OUT_HIGH1)
- net at VOUT7.1 (Pin_1): now also M9.W9 (OUT_LOW7_PULLUP)
- net at MMCU23.1 (Pin_1): now also M11.S4 (IN_D2)
- net at MMCU35.1 (Pin_1): now also M11.S5 (IN_D3)
- net at MMCU16.1 (Pin_1): now also M11.S6 (IN_D4)
- net at MMCU24.1 (Pin_1): now also M11.N12 (IO1)
- net at MMCU25.1 (Pin_1): now also M11.N13 (IO2)
- net at MMCU26.1 (Pin_1): now also M11.N14 (IO3)
- net at MMCU10.1 (Pin_1): now also M11.E2 (SPI1_MISO)
- net at MMCU14.1 (Pin_1): now also M11.E16 (OUT_PWM4)
- net at VOUT27.1 (Pin_1): now also M9.W39 (LOW7_HIGH1)
- net at MMCU4.1 (Pin_1): now also M11.N6 (UART2_TX)
- net at MMCU40.1 (Pin_1): now also M11.E20 (OUT_IO11)
- net at MMCU2.1 (Pin_1): now also M11.N4 (UART8_TX)
- net at MMCU18.1 (Pin_1): now also M11.E10 (OUT_IO10)
- net at MMCU30.1 (Pin_1): now also M11.E11 (OUT_IO9)
- net at MMCU31.1 (Pin_1): now also M11.E13 (OUT_IO12)
- net at MMCU29.1 (Pin_1): now also M11.E22 (OUT_IO8)
- net at MMCU38.1 (Pin_1): now also M11.E23 (OUT_IO4)
- net at MMCU32.1 (Pin_1): now also M11.E24 (OUT_IO13)
- net at MMCU8.1 (Pin_1): now also M11.N32 (USB1ID)
- net at MMCU12.1 (Pin_1): now also M11.E4 (SPI1_CS1)
- net at VOUT17.1 (Pin_1): now also M9.W36 (LOW12)
- net at VOUT12.1 (Pin_1): now also M9.W37 (LOW8_HIGH2)
- net at VOUT26.1 (Pin_1): now also M9.W25 (LOW6_DIODE)
- net at VOUT13.1 (Pin_1): now also M9.W27 (LOW9)
- net at VOUT21.1 (Pin_1): now also M9.W30 (SOLENOID_B2)
- net at VOUT20.1 (Pin_1): now also M9.W31 (SOLENOID_B1)
- net at VOUT19.1 (Pin_1): now also M9.W32 (SOLENOID_A2)
- net at VOUT18.1 (Pin_1): now also M9.W33 (SOLENOID_A1)
- net at VOUT16.1 (Pin_1): now also M9.W35 (LOW11)
- net at MMCU5.1 (Pin_1): now also M11.N25 (SWCLK)
- net at MMCU3.1 (Pin_1): now also M11.N7 (UART2_RX)
- net at MMCU6.1 (Pin_1): now also M11.N26 (SWDIO)
- net at MMCU13.1 (Pin_1): now also M11.E5 (SPI1_CS2)
- net OUT_MAIN renamed OUT_MAIN_RELAY
- net OUT_MAIN_RELAY: now also D11.2 (A), D43.1 (K), M9.W13 (OUT_LOW5_MAIN)
- net OUT_PUMP renamed OUT_FUEL_PUMP_RELAY
- net OUT_FUEL_PUMP_RELAY: now also M9.W2 (OUT_LOW10)
- new net +5VP: C23.2, J20.1 (Pin_1), J20.2 (Pin_2), J21.1 (Pin_1), JP59.2, U7.1 (OUT), U8.1 (OUT)
- new net OUT_CHECK_ENGINE: JP8.2, M9.S8 (OUT_LOW1)
- no-connect marks 39 -> 41
Other:
- note added: "C540240"
- note added: "C540241"
- note added: "C540242"
- note added: "C540243"
- note added: "ETB Drive-by-wire motor connector"
- note added: "Electronic Throttle Body/ETB"
- note added: "Protected 5V analog power supply"
- note added: "SOIC-8"
- note added: "TSON-10"
- note removed: "ETB driver"
- moved on the sheet: C10, C11, C12, C13, C14, C15, C16, C17, C18, C19, C20, C21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

Commit message: MCU144
Parts:
- M11: value Module-mcu-0.6 -> Module-mcu144-0.6
Changed lines of the file:
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@@
     (in_bom yes) (on_board yes)
     (property "Reference" "M11" (id 0) (at 577.85 111.76 0))
-    (property "Value" "Module-mcu-0.6" (id 1) (at 577.85 114.3 0))
+    (property "Value" "Module-mcu144-0.6" (id 1) (at 577.85 114.3 0))
     (property "Footprint" "hellen-one-mcu-0.6:mcu" (id 2) (at 568.96 115.57 0)
       (effects (font (size 1.27 1.27)) hide)
@@
       (effects (font (size 1.27 1.27)) (justify right))
     )
-    (property "Value" "Module-mcu-0.6" (id 1) (at 551.18 114.3 0)
+    (property "Value" "Module-mcu144-0.6" (id 1) (at 546.1 114.3 0)
       (effects (font (size 1.27 1.27)) (justify right))
     )
@@
       (effects (font (size 1.27 1.27)) (justify left))
     )
-    (property "Value" "Module-mcu-0.6" (id 1) (at 570.23 299.7199 0)
+    (property "Value" "Module-mcu144-0.6" (id 1) (at 570.23 299.7199 0)
       (effects (font (size 1.27 1.27)) (justify left))
     )
@@
     (in_bom yes) (on_board yes) (fields_autoplaced)
     (property "Reference" "M11" (id 0) (at 614.68 257.81 0))
-    (property "Value" "Module-mcu-0.6" (id 1) (at 614.68 260.35 0))
+    (property "Value" "Module-mcu144-0.6" (id 1) (at 614.68 260.35 0))
     (property "Footprint" "hellen-one-mcu-0.6:mcu" (id 2) (at 596.9 262.89 0)
       (effects (font (size 1.27 1.27)) hide)
@@
     )
     (path "/4a5ba710-59da-4d33-bf5b-90903381be28"
-      (reference "M11") (unit 1) (value "Module-mcu-0.6") (footprint "hellen-one-mcu-0.6:mcu")
+      (reference "M11") (unit 1) (value "Module-mcu144-0.6") (footprint "hellen-one-mcu-0.6:mcu")
     )
     (path "/4f4b9c60-b508-4905-9e7b-bc30ea466838"
-      (reference "M11") (unit 2) (value "Module-mcu-0.6") (footprint "hellen-one-mcu-0.6:mcu")
+      (reference "M11") (unit 2) (value "Module-mcu144-0.6") (footprint "hellen-one-mcu-0.6:mcu")
     )
     (path "/5bea29f7-9491-4d90-9d24-601079515983"
-      (reference "M11") (unit 3) (value "Module-mcu-0.6") (footprint "hellen-one-mcu-0.6:mcu")
+      (reference "M11") (unit 3) (value "Module-mcu144-0.6") (footprint "hellen-one-mcu-0.6:mcu")
     )
     (path "/7fdc726d-9583-46f7-87d4-ecc994f408ad"
-      (reference "M11") (unit 4) (value "Module-mcu-0.6") (footprint "hellen-one-mcu-0.6:mcu")
+      (reference "M11") (unit 4) (value "Module-mcu144-0.6") (footprint "hellen-one-mcu-0.6:mcu")
     )
     (path "/252b4f77-58b4-4ba1-a925-b260d38b7d08"
