File: kicad/hellen88bmw.kicad_pcb (KiCad board)
At the start: 2 copper layers, 160 x 118 mm, 239 parts, among them J1 920-462A2021Y10101, J10 Conn_01x12, J11 Conn_01x12, J12 Conn_01x12, J13 Conn_01x12, J14 VRIN1, J15 VRIN2, J16 VROUT1, J2 UB-20PMFP-LC7002, J3 Micro_SD_Card, J4 Conn_01x05, J5 Conn_01x12, J6 Conn_01x12, J7 Conn_01x12, J8 Conn_01x12, J9 Conn_01x12, M1 Module-power12-0.1, M10 Module-ign8-0.1, M11 Module-mcu-0.1, M2 Module-can-0.1, M3 Module-wbo-0.1, M4 Module-can-0.1, M5 Module-power5-0.1, M6 Module-vr-0.1, M7 Module-input-0.1, M8 Module-knock-0.1, M9 Module-output-0.1, Q1 NGD8201AN, Q2 NGD8201AN, Q3 NGD8201AN, Q4 NGD8201AN, Q5 NGD8201AN, Q6 NGD8201AN, Q7 NGD8201AN, Q8 NGD8201AN, SW1 BOOT0, SW2 RESET, U1 MPXA6115A, U2 MPX4_MAP

Commit message: Up 88
Parts:
- added J17: SD, Connector_PinHeader_2.54mm:PinHeader_1x06_P2.54mm_Vertical, F.Cu at (95.2, 93.9)
- added OUT_IGN1: OUT_IGN1, Connector_PinHeader_1.00mm:PinHeader_1x01_P1.00mm_Vertical, F.Cu at (196.5, 118.8)
- added OUT_IGN2: OUT_IGN2, Connector_PinHeader_1.00mm:PinHeader_1x01_P1.00mm_Vertical, F.Cu at (195.0, 116.8)
- added OUT_IGN3: OUT_IGN3, Connector_PinHeader_1.00mm:PinHeader_1x01_P1.00mm_Vertical, F.Cu at (193.5, 118.8)
- added OUT_IGN4: OUT_IGN4, Connector_PinHeader_1.00mm:PinHeader_1x01_P1.00mm_Vertical, F.Cu at (192.0, 116.8)
- added OUT_IGN5: OUT_IGN5, Connector_PinHeader_1.00mm:PinHeader_1x01_P1.00mm_Vertical, F.Cu at (190.5, 118.8)
- added OUT_IGN6: OUT_IGN6, Connector_PinHeader_1.00mm:PinHeader_1x01_P1.00mm_Vertical, F.Cu at (189.2, 116.8)
- added OUT_IGN7: OUT_IGN7, Connector_PinHeader_1.00mm:PinHeader_1x01_P1.00mm_Vertical, F.Cu at (187.8, 118.8)
- added OUT_IGN8: OUT_IGN8, Connector_PinHeader_1.00mm:PinHeader_1x01_P1.00mm_Vertical, F.Cu at (186.5, 116.8)
- added OUT_INJ1: OUT_INJ1, Connector_PinHeader_1.00mm:PinHeader_1x01_P1.00mm_Vertical, F.Cu at (273.0, 122.0)
- added OUT_INJ2: OUT_INJ2, Connector_PinHeader_1.00mm:PinHeader_1x01_P1.00mm_Vertical, F.Cu at (272.8, 117.8)
- added OUT_INJ3: OUT_INJ3, Connector_PinHeader_1.00mm:PinHeader_1x01_P1.00mm_Vertical, F.Cu at (273.2, 130.5)
- added OUT_INJ4: OUT_INJ4, Connector_PinHeader_1.00mm:PinHeader_1x01_P1.00mm_Vertical, F.Cu at (273.0, 114.5)
- added OUT_INJ5: OUT_INJ5, Connector_PinHeader_1.00mm:PinHeader_1x01_P1.00mm_Vertical, F.Cu at (273.0, 106.5)
- added OUT_INJ6: OUT_INJ6, Connector_PinHeader_1.00mm:PinHeader_1x01_P1.00mm_Vertical, F.Cu at (273.0, 110.5)
- added OUT_INJ7: OUT_INJ7, Connector_PinHeader_1.00mm:PinHeader_1x01_P1.00mm_Vertical, F.Cu at (273.0, 126.2)
- added OUT_INJ8: OUT_INJ8, Connector_PinHeader_1.00mm:PinHeader_1x01_P1.00mm_Vertical, F.Cu at (272.5, 102.5)
- moved SW2 147.3 mm to (37.5, 178.0)
- moved SW1 131.2 mm to (17.1, 172.0)
- moved MMCU11 37.8 mm to (-40.7, 138.1)
- moved MMCU8 37.8 mm to (-37.4, 138.1)
- moved C3 37.8 mm to (-20.6, 92.8)
- moved D1 37.8 mm to (22.6, 68.5)
- moved D12 37.8 mm to (8.73, 82.4)
- moved D14 37.8 mm to (25.0, 61.1)
- moved D16 37.8 mm to (12.9, 75.0)
- moved D17 37.8 mm to (-65.2, 117.1)
- moved D18 37.8 mm to (-39.4, 132.2)
- moved D19 37.8 mm to (-0.03, 90.5)
- moved D2 37.8 mm to (-8.44, 101.2)
- moved D21 37.8 mm to (-35.4, 126.3)
- moved D22 37.8 mm to (29.1, 61.1)
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Connections:
- JP85 pad 2: /CAN_L -> /CAN-
- JP86 pad 2: /CAN_H -> /CAN+
Routing:
- net /IGN_V5: track 0.00 -> 9.16 mm
- net /PB9: track 0.00 -> 8.31 mm
- net /PC11: track 0.00 -> 7.77 mm
- net /PC12: track 0.00 -> 7.71 mm
- net GND: track 378.7 -> 385.9 mm
- net /3.3V: track 0.00 -> 7.12 mm
- net /PC10: track 0.00 -> 6.58 mm
- net /OUT_IGN2: track 0.00 -> 5.07 mm
- net /IGN6: track 0.00 -> 4.89 mm
- net /IGN8: track 0.00 -> 4.75 mm
- net /IGN4: track 0.00 -> 4.70 mm
- net /IGN5: track 0.00 -> 4.69 mm
- net /IGN_V33: track 0.00 -> 4.69 mm
- net /OUT3: track 0.00 -> 4.65 mm
- net /INJ3: track 7.28 -> 11.9 mm
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
Commit message: Up 88
Parts:
- added KNOCK_RAW1: IN_KNOCK1_RAW, Connector_PinHeader_1.00mm:PinHeader_1x01_P1.00mm_Vertical, F.Cu at (212.8, 1.00)
- added R5: DNP, Resistor_SMD:R_0603_1608Metric, F.Cu at (100.8, 186.7)
- added R6: DNP, Resistor_SMD:R_0603_1608Metric, F.Cu at (102.8, 178.0)
- C1, C2, M5, U1: moved to B.Cu
- J2: footprint Connector_PinHeader_1.00mm:PinHeader_1x01_P1.00mm_Vertical -> Connector_PinHeader_2.00mm:PinHeader_1x05_P2.00mm_Vertical
- moved D17 317.4 mm to (247.8, 64.0)
- moved D20 306.9 mm to (251.5, 66.2)
- moved D21 294.9 mm to (252.5, 62.5)
- moved RN5 260.2 mm to (243.8, 66.5)
- moved D16 235.0 mm to (247.8, 68.5)
- moved MMCU28 229.5 mm to (252.5, 106.2)
- moved R2 220.5 mm to (153.2, 145.0)
- moved VOUT2 220.2 mm to (120.8, -29.0)
- moved VOUT4 220.0 mm to (120.8, -25.0)
- moved VIN13 213.8 mm to (160.8, 75.8)
- moved OUT_INJ8 209.5 mm to (130.8, -51.8)
- moved OUT_INJ1 208.4 mm to (131.5, -31.0)
- moved OUT_INJ2 208.4 mm to (131.2, -35.2)
- moved OUT_INJ3 208.4 mm to (131.8, -22.5)
- moved OUT_INJ4 208.4 mm to (131.5, -38.5)
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Routing:
- net Net-(M3-PadW2): track 0.00 -> 67.9 mm, vias 0 -> 1
- net Net-(M3-PadW3): track 0.00 -> 63.1 mm, vias 0 -> 1
- net Net-(M3-PadW4): track 0.00 -> 60.9 mm, vias 0 -> 1
- net GNDA: track 3.59 -> 49.7 mm
- net V5A: track 3.59 -> 35.4 mm
- net /NRESET: track 0.00 -> 28.3 mm, vias 0 -> 1
- net /USBM: track 0.00 -> 26.3 mm
- net /CAN_VIO: track 0.00 -> 25.0 mm
- net /VBUS: track 0.00 -> 23.5 mm
- net /BOOT0: track 0.00 -> 22.7 mm, vias 0 -> 1
- net /USBP: track 0.00 -> 21.3 mm
- net /CAM: track 20.3 -> 0.36 mm
- net /CAN_RX: track 0.00 -> 18.9 mm
- net /CAN_TX: track 0.00 -> 16.3 mm
- net +3V3: track 0.00 -> 15.8 mm, vias 0 -> 1
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