File: kicad/hellen88bmw.kicad_sch (KiCad schematic)
At the start: 251 parts, among them J10 Conn_01x12, J11 Conn_01x12, J12 Conn_01x12, J13 Conn_01x12, J3 Micro_SD_Card, J4 Conn_01x05, J5 Conn_01x12, J6 Conn_01x12, J7 Conn_01x12, J8 Conn_01x12, J9 Conn_01x12, Q1 NGD8201AN, Q2 NGD8201AN, Q3 NGD8201AN, Q4 NGD8201AN, Q5 NGD8201AN, Q6 NGD8201AN, Q7 NGD8201AN, Q8 NGD8201AN

Commit message: Up 88
Parts:
- removed D? (x4): LED, symbol Device:LED
- removed RN?: 470, symbol Device:R_Pack04
- C1, C2, C3: renamed from C?; footprint Capacitor_SMD:C_0805_2012Metric -> Capacitor_SMD:C_0603_1608Metric
- D1, D10, D11, D12, D13, D14, D15, D16, D17, D18, D19, D2, D20, D21, D22, D23, D24, D25, D26, D27, D28, D29, D3, D30, D31, D4, D5, D6, D7, D8, D9: renamed from D?; footprint (none) -> LED_SMD:LED_0603_1608Metric
- J14, J15, J16: renamed from J?; footprint Connector_PinHeader_2.54mm:PinHeader_1x01_P2.54mm_Vertical -> Connector_PinHeader_1.00mm:PinHeader_1x01_P1.00mm_Vertical
- J2: renamed from J?; footprint Connector_PinHeader_2.54mm:PinHeader_1x05_P2.54mm_Vertical -> Connector_PinHeader_1.00mm:PinHeader_1x01_P1.00mm_Vertical
- J3: footprint rusefi_lib:microSD_HC_Wuerth_693072010801 -> rusefi_lib_private:693072010801
- JP1, JP10, JP11, JP12, JP13, JP14, JP15, JP16, JP17, JP18, JP19, JP2, JP20, JP21, JP22, JP23, JP24, JP25, JP26, JP27, JP28, JP29, JP3, JP30, JP31, JP32, JP33, JP34, JP35, JP36, JP37, JP38, JP39, JP4, JP40, JP41, JP42, JP43, JP44, JP45, JP46, JP47, JP48, JP49, JP5, JP50, JP51, JP52, JP53, JP54, JP55, JP56, JP57, JP58, JP59, JP6, JP60, JP61, JP62, JP63, JP64, JP65, JP66, JP67, JP68, JP69, JP7, JP70, JP71, JP72, JP73, JP74, JP75, JP76, JP77, JP78, JP79, JP8, JP80, JP81, JP82, JP83, JP84, JP85, JP86, JP87, JP88, JP9: footprint rusefi_lib:SM0805_jumper -> rusefi_lib_private:SM0805_jumper
- M1: renamed from M?; footprint hellen-one-power12-0.1:power12 -> rusefi_lib_private:MOD_HELLEN_POWER_12
- M10: renamed from M?; footprint hellen-one-ign8-0.1:ign8 -> rusefi_lib_private:MOD_HELLEN_IGN8
- M11: renamed from M?; footprint hellen-one-mcu-0.1:mcu -> rusefi_lib_private:MOD_HELLEN_MCU
- M2, M4: renamed from M?; footprint hellen-one-can-0.1:can -> rusefi_lib_private:MOD_HELLEN_CAN
- M3: renamed from M?; footprint hellen-one-wbo-0.1:wbo -> rusefi_lib_private:MOD_HELLEN_WBO
- M5: renamed from M?; footprint hellen-one-power5-0.1:power5 -> rusefi_lib_private:MOD_HELLEN_POWER_5
- M6: renamed from M?; footprint hellen-one-vr-0.1:vr -> rusefi_lib_private:MOD_HELLEN_VR
- M7: renamed from M?; footprint hellen-one-input-0.1:input -> rusefi_lib_private:MOD_HELLEN_INPUT
- M8: renamed from M?; footprint hellen-one-knock-0.1:knock -> rusefi_lib_private:MOD_HELLEN_KNOCK
- M9: renamed from M?; footprint hellen-one-output-0.1:output -> rusefi_lib_private:MOD_HELLEN_OUTPUT
- MMCU1, MMCU10, MMCU11, MMCU12, MMCU13, MMCU14, MMCU15, MMCU16, MMCU17, MMCU18, MMCU19, MMCU2, MMCU20, MMCU21, MMCU22, MMCU23, MMCU24, MMCU25, MMCU26, MMCU27, MMCU28, MMCU29, MMCU3, MMCU30, MMCU31, MMCU32, MMCU33, MMCU34, MMCU35, MMCU36, MMCU4, MMCU5, MMCU6, MMCU7, MMCU8, MMCU9, VIN10, VIN11, VIN12, VIN13, VIN14, VIN15, VIN16, VIN17, VIN5, VIN6, VIN7, VIN8, VIN9, VOUT4, VOUT5, VOUT6: footprint Connector_PinHeader_2.54mm:PinHeader_1x01_P2.54mm_Vertical -> Connector_PinHeader_1.00mm:PinHeader_1x01_P1.00mm_Vertical
- R1, R2, R3: renamed from R?; footprint (none) -> Resistor_SMD:R_0603_1608Metric
- R4: renamed from R?; footprint Resistor_SMD:R_0805_2012Metric -> Resistor_SMD:R_0603_1608Metric
- RN1, RN2, RN3, RN4, RN5, RN6, RN7, RN8: renamed from RN?; footprint (none) -> Resistor_SMD:R_Array_Concave_4x0603
- SW1, SW2: renamed from SW?; footprint (none) -> Button_Switch_SMD:SW_SPST_B3U-1000P-B
- TP1, TP2, TP3, TP4: renamed from TP?; footprint (none) -> TestPoint:TestPoint_Pad_D1.0mm
- U2: renamed from U?; footprint MPX4-P -> rusefi_lib_private:MPX-4_MAP
- VIN1, VIN2, VIN3, VIN4, VOUT1, VOUT2, VOUT3: footprint hellen-one-common:PAD-TH -> Connector_PinHeader_1.00mm:PinHeader_1x01_P1.00mm_Vertical
- gave numbers to parts that had none: 2

Commit message: Up 88
Parts:
- added J17: SD, Connector_PinHeader_2.54mm:PinHeader_1x06_P2.54mm_Vertical, symbol Connector_Generic:Conn_01x06
- added KNOCK_RAW?: IN_KNOCK1_RAW, Connector_PinHeader_1.00mm:PinHeader_1x01_P1.00mm_Vertical, symbol Connector_Generic:Conn_01x01
- added OUT_IGN1: OUT_IGN1, Connector_PinHeader_1.00mm:PinHeader_1x01_P1.00mm_Vertical, symbol Connector_Generic:Conn_01x01
- added OUT_IGN2: OUT_IGN2, Connector_PinHeader_1.00mm:PinHeader_1x01_P1.00mm_Vertical, symbol Connector_Generic:Conn_01x01
- added OUT_IGN3: OUT_IGN3, Connector_PinHeader_1.00mm:PinHeader_1x01_P1.00mm_Vertical, symbol Connector_Generic:Conn_01x01
- added OUT_IGN4: OUT_IGN4, Connector_PinHeader_1.00mm:PinHeader_1x01_P1.00mm_Vertical, symbol Connector_Generic:Conn_01x01
- added OUT_IGN5: OUT_IGN5, Connector_PinHeader_1.00mm:PinHeader_1x01_P1.00mm_Vertical, symbol Connector_Generic:Conn_01x01
- added OUT_IGN6: OUT_IGN6, Connector_PinHeader_1.00mm:PinHeader_1x01_P1.00mm_Vertical, symbol Connector_Generic:Conn_01x01
- added OUT_IGN7: OUT_IGN7, Connector_PinHeader_1.00mm:PinHeader_1x01_P1.00mm_Vertical, symbol Connector_Generic:Conn_01x01
- added OUT_IGN8: OUT_IGN8, Connector_PinHeader_1.00mm:PinHeader_1x01_P1.00mm_Vertical, symbol Connector_Generic:Conn_01x01
- added OUT_INJ1: OUT_INJ1, Connector_PinHeader_1.00mm:PinHeader_1x01_P1.00mm_Vertical, symbol Connector_Generic:Conn_01x01
- added OUT_INJ2: OUT_INJ2, Connector_PinHeader_1.00mm:PinHeader_1x01_P1.00mm_Vertical, symbol Connector_Generic:Conn_01x01
- added OUT_INJ3: OUT_INJ3, Connector_PinHeader_1.00mm:PinHeader_1x01_P1.00mm_Vertical, symbol Connector_Generic:Conn_01x01
- added OUT_INJ4: OUT_INJ4, Connector_PinHeader_1.00mm:PinHeader_1x01_P1.00mm_Vertical, symbol Connector_Generic:Conn_01x01
- added OUT_INJ5: OUT_INJ5, Connector_PinHeader_1.00mm:PinHeader_1x01_P1.00mm_Vertical, symbol Connector_Generic:Conn_01x01
- added OUT_INJ6: OUT_INJ6, Connector_PinHeader_1.00mm:PinHeader_1x01_P1.00mm_Vertical, symbol Connector_Generic:Conn_01x01
- added OUT_INJ7: OUT_INJ7, Connector_PinHeader_1.00mm:PinHeader_1x01_P1.00mm_Vertical, symbol Connector_Generic:Conn_01x01
- added OUT_INJ8: OUT_INJ8, Connector_PinHeader_1.00mm:PinHeader_1x01_P1.00mm_Vertical, symbol Connector_Generic:Conn_01x01
- added R? (x2): DNP, Resistor_SMD:R_0603_1608Metric, symbol hellen-one-common:Res
Connections:
- net CAN_H is gone; now on net CAN+: JP86.2 (B)
- net CAN_L is gone; now on net CAN-: JP85.2 (B)
- net 3.3V: now also J17.3 (Pin_3)
- net GND: now also J17.5 (Pin_5)
- net IN_CRANK: now also R?.2
- net IN_KNOCK1_RAW: now also KNOCK_RAW?.1 (Pin_1)
- net OUT_IGN1: now also OUT_IGN1.1 (Pin_1)
- net OUT_IGN2: now also OUT_IGN2.1 (Pin_1)
- net OUT_IGN3: now also OUT_IGN3.1 (Pin_1)
- net OUT_IGN4: now also OUT_IGN4.1 (Pin_1)
- net OUT_IGN5: now also OUT_IGN5.1 (Pin_1)
- net OUT_IGN6: now also OUT_IGN6.1 (Pin_1)
- net OUT_IGN7: now also OUT_IGN7.1 (Pin_1)
- net OUT_IGN8: now also OUT_IGN8.1 (Pin_1)
- net OUT_INJ1: now also OUT_INJ1.1 (Pin_1)
- net OUT_INJ2: now also OUT_INJ2.1 (Pin_1)
- net OUT_INJ3: now also OUT_INJ3.1 (Pin_1)
- net OUT_INJ4: now also OUT_INJ4.1 (Pin_1)
- net OUT_INJ5: now also OUT_INJ5.1 (Pin_1)
- net OUT_INJ6: now also OUT_INJ6.1 (Pin_1)
- net OUT_INJ7: now also OUT_INJ7.1 (Pin_1)
- net OUT_INJ8: now also OUT_INJ8.1 (Pin_1)
- net PB9: now also J17.1 (Pin_1)
- net PC10: now also J17.4 (Pin_4)
- net PC11: now also J17.6 (Pin_6)
- net PC12: now also J17.2 (Pin_2)
- net VREF1: now also R?.2
- new net IN_CRANK+: R?.1
- new net IN_CRANK-: R?.1
Other:
- moved on the sheet: C3, D1, D10, D11, D12, D13, D14, D15, D16, D17, D18, D19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

Commit message: Up 88
Parts:
- J2: footprint Connector_PinHeader_1.00mm:PinHeader_1x01_P1.00mm_Vertical -> Connector_PinHeader_2.00mm:PinHeader_1x05_P2.00mm_Vertical
- gave numbers to parts that had none: 3
Connections:
- net CRANK: no longer M6.W2 (OUT_VR1)
- net CRANK+: no longer M6.E2 (IN_VR1+)
- net CRANK-: no longer M6.E1 (IN_VR1-)
- net IN_CRANK: now also M6.W2 (OUT_VR1)
- net IN_CRANK+: now also M6.E2 (IN_VR1+)
- net IN_CRANK-: now also M6.E1 (IN_VR1-)
Changed lines of the file:
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@@
     (effects (font (size 1.27 1.27)) (justify right bottom))
   )
-  (label "CRANK+" (at 101.6 312.42 180)
+  (label "IN_CRANK+" (at 101.6 312.42 180)
     (effects (font (size 1.27 1.27)) (justify right bottom))
   )
-  (label "CRANK-" (at 101.6 314.96 180)
+  (label "IN_CRANK-" (at 101.6 314.96 180)
     (effects (font (size 1.27 1.27)) (justify right bottom))
   )
@@
     (effects (font (size 1.27 1.27)) (justify left bottom))
   )
-  (label "CRANK" (at 149.86 314.96 0)
+  (label "IN_CRANK" (at 149.86 314.96 0)
     (effects (font (size 1.27 1.27)) (justify left bottom))
   )
@@
   (symbol (lib_id "Connector_Generic:Conn_01x01") (at 204.47 369.57 90) (unit 1)
     (in_bom yes) (on_board yes)
-    (property "Reference" "KNOCK_RAW?" (id 0) (at 204.47 367.03 0)
+    (property "Reference" "KNOCK_RAW1" (id 0) (at 204.47 367.03 0)
       (effects (font (size 1.27 1.27)) (justify left))
     )
@@
   (symbol (lib_id "hellen-one-common:Res") (at 118.11 391.16 0) (unit 1)
     (in_bom yes) (on_board yes)
-    (property "Reference" "R?" (id 0) (at 119.38 386.9498 0))
+    (property "Reference" "R5" (id 0) (at 119.38 386.9498 0))
     (property "Value" "DNP" (id 1) (at 123.19 387.9785 0))
     (property "Footprint" "Resistor_SMD:R_0603_1608Metric" (id 2) (at 121.92 394.97 0)
@@
   (symbol (lib_id "hellen-one-common:Res") (at 118.11 397.51 0) (unit 1)
     (in_bom yes) (on_board yes)
-    (property "Reference" "R?" (id 0) (at 119.38 393.2998 0))
+    (property "Reference" "R6" (id 0) (at 119.38 393.2998 0))
     (property "Value" "DNP" (id 1) (at 123.19 394.3285 0))
     (property "Footprint" "Resistor_SMD:R_0603_1608Metric" (id 2) (at 121.92 401.32 0)
@@
       (effects (font (size 1.27 1.27)) (justify left))
     )
-    (property "Footprint" "Connector_PinHeader_1.00mm:PinHeader_1x01_P1.00mm_Vertical" (id 2) (at 118.11 64.77 0)
+    (property "Footprint" "Connector_PinHeader_2.00mm:PinHeader_1x05_P2.00mm_Vertical" (id 2) (at 118.11 64.77 0)
       (effects (font (size 1.27 1.27)) hide)
     )
@@
     )
     (path "/b7ba4c3d-5d4c-4bf5-b353-2713dfc28ba6"
-      (reference "J2") (unit 1) (value "UB-20PMFP-LC7002") (footprint "Connector_PinHeader_1.00mm:PinHeader_1x01_P1.00mm_Vertical")
+      (reference "J2") (unit 1) (value "UB-20PMFP-LC7002") (footprint "Connector_PinHeader_2.00mm:PinHeader_1x05_P2.00mm_Vertical")
     )
     (path "/00000000-0000-0000-0000-000060bde589"
@@
     )
     (path "/38db208f-6a11-4100-a872-f7e228085d88"
-      (reference "KNOCK_RAW?") (unit 1) (value "IN_KNOCK1_RAW") (footprint "Connector_PinHeader_1.00mm:PinHeader_1x01_P1.00mm_Vertical")
+      (reference "KNOCK_RAW1") (unit 1) (value "IN_KNOCK1_RAW") (footprint "Connector_PinHeader_1.00mm:PinHeader_1x01_P1.00mm_Vertical")
     )
     (path "/d2da829a-6cb9-4cba-934a-cec3dc1f31ab"
@@
       (reference "R4") (unit 1) (value "1k") (footprint "Resistor_SMD:R_0603_1608Metric")
     )
-    (path "/08b25796-70dd-45ec-b49e-9604f33474f7"
-      (reference "R?") (unit 1) (value "DNP") (footprint "Resistor_SMD:R_0603_1608Metric")
-    )
     (path "/40e5e4bd-db91-429a-aa04-1aafd1b4ce09"
-      (reference "R?") (unit 1) (value "DNP") (footprint "Resistor_SMD:R_0603_1608Metric")
+      (reference "R5") (unit 1) (value "DNP") (footprint "Resistor_SMD:R_0603_1608Metric")
+    )
+    (path "/08b25796-70dd-45ec-b49e-9604f33474f7"
+      (reference "R6") (unit 1) (value "DNP") (footprint "Resistor_SMD:R_0603_1608Metric")
     )
     (path "/bbd8a8a3-1884-44de-bae5-46a536e539ec"
