File: boards/hellen88bmw/kicad6/hellen88bmw.kicad_pcb (KiCad board)
At the start: 2 copper layers, 160 x 118 mm, 259 parts, among them J1 920-462A2021Y10101, J10 Conn_01x12, J11 Conn_01x12, J12 Conn_01x12, J13 Conn_01x12, J14 VRIN1, J15 VRIN2, J16 VROUT1, J17 SD, J2 UB-20PMFP-LC7002, J3 Micro_SD_Card, J4 Conn_01x05, J5 Conn_01x12, J6 Conn_01x12, J7 Conn_01x12, J8 Conn_01x12, J9 Conn_01x12, M1 Module-power12-0.1, M10 Module-ign8-0.1, M11 Module-mcu-0.1, M2 Module-can-0.1, M3 Module-wbo-0.1, M4 Module-can-0.1, M5 Module-power5-0.1, M6 Module-vr-0.1, M7 Module-input-0.1, M8 Module-knock-0.1, M9 Module-output-0.1, Q1 NGD8201AN, Q2 NGD8201AN, Q3 NGD8201AN, Q4 NGD8201AN, Q5 NGD8201AN, Q6 NGD8201AN, Q7 NGD8201AN, Q8 NGD8201AN, SW1 BOOT0, SW2 RESET, U1 MPXA6115A, U2 MPX4_MAP

Commit message: Up 88
Parts:
- removed MMCU14, MMCU15, MMCU16, MMCU17, MMCU22, MMCU23: MMCU, Connector_PinHeader_1.00mm:PinHeader_1x01_P1.00mm_Vertical
- removed OUT_IGN1: OUT_IGN1, Connector_PinHeader_1.00mm:PinHeader_1x01_P1.00mm_Vertical
- removed OUT_IGN2: OUT_IGN2, Connector_PinHeader_1.00mm:PinHeader_1x01_P1.00mm_Vertical
- removed OUT_IGN3: OUT_IGN3, Connector_PinHeader_1.00mm:PinHeader_1x01_P1.00mm_Vertical
- removed OUT_IGN4: OUT_IGN4, Connector_PinHeader_1.00mm:PinHeader_1x01_P1.00mm_Vertical
- removed OUT_IGN5: OUT_IGN5, Connector_PinHeader_1.00mm:PinHeader_1x01_P1.00mm_Vertical
- removed OUT_IGN6: OUT_IGN6, Connector_PinHeader_1.00mm:PinHeader_1x01_P1.00mm_Vertical
- removed OUT_IGN7: OUT_IGN7, Connector_PinHeader_1.00mm:PinHeader_1x01_P1.00mm_Vertical
- removed OUT_IGN8: OUT_IGN8, Connector_PinHeader_1.00mm:PinHeader_1x01_P1.00mm_Vertical
- added C4: 100nF, Capacitor_SMD:C_0603_1608Metric, B.Cu at (148.8, 165.2)
- added C5: 100nF, Capacitor_SMD:C_0603_1608Metric, B.Cu at (139.7, 161.9)
- added C6: 100nF, Capacitor_SMD:C_0603_1608Metric, F.Cu at (53.0, 94.2)
- added C7: 10uF, Capacitor_SMD:C_0402_1005Metric, F.Cu at (48.5, 94.5)
- added J18: C165947, Connector_Audio:Jack_3.5mm_CUI_SJ1-3535NG_Horizontal, F.Cu at (81.2, 98.1)
- added R10: DNP, Resistor_SMD:R_2512_6332Metric, F.Cu at (200.2, 132.5)
- added R11: DNP, Resistor_SMD:R_2512_6332Metric, F.Cu at (193.2, 75.8)
- added R12: DNP, Resistor_SMD:R_2512_6332Metric, F.Cu at (193.2, 80.8)
- added R13: DNP, Resistor_SMD:R_2512_6332Metric, F.Cu at (200.2, 82.5)
- added R14: DNP, Resistor_SMD:R_2512_6332Metric, F.Cu at (200.2, 142.0)
- added R15: 4k7, Resistor_SMD:R_0402_1005Metric, B.Cu at (150.5, 161.8)
- added R16: 4k7, Resistor_SMD:R_0402_1005Metric, B.Cu at (147.6, 161.8)
- added R7: DNP, Resistor_SMD:R_2512_6332Metric, F.Cu at (200.2, 122.8)
- added R8: DNP, Resistor_SMD:R_2512_6332Metric, F.Cu at (200.2, 113.2)
- added R9: DNP, Resistor_SMD:R_2512_6332Metric, F.Cu at (200.2, 92.5)
- added U3: LIS2DW12TR, Package_LGA:Kionix_LGA-12_2x2mm_P0.5mm_LayoutBorder2x4y, B.Cu at (135.9, 161.7)
- added U4: LPS25HB, Package_LGA:ST_HLGA-10_2.5x2.5mm_P0.6mm_LayoutBorder3x2y, B.Cu at (154.0, 164.0)
- added U5: MCP6002-xSN, Package_SO:SOIC-8_3.9x4.9mm_P1.27mm, F.Cu at (51.8, 100.0)
- moved Q8 133.8 mm to (208.0, 143.0), turned to 0 degrees
- moved Q7 130.4 mm to (208.0, 133.0), turned to 0 degrees
- moved M1 49.7 mm to (50.5, 131.5)
- moved Q3 24.9 mm to (208.0, 93.0), turned to 0 degrees
- moved C1 21.2 mm to (82.0, 126.3), turned to 0 degrees
- moved Q1 20.2 mm to (208.0, 123.5), turned to 0 degrees
- moved J3 19.3 mm to (71.3, 112.7)
- moved J17 19.3 mm to (80.5, 106.3)
- moved C2 18.4 mm to (82.0, 128.3), turned to 0 degrees
- moved Q2 17.8 mm to (208.0, 113.5), turned to 0 degrees
- moved Q4 11.2 mm to (208.0, 83.0), turned to 0 degrees
- moved Q5 9.27 mm to (208.0, 73.5), turned to 0 degrees
- moved U1 8.47 mm to (82.0, 135.3), turned to -90 degrees
- moved Q6 8.30 mm to (208.0, 63.5), turned to 0 degrees
- moved M3 7.60 mm to (113.1, 145.7)
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Connections:
- net /IN_KNOCK1_RAW renamed /IN_KNOCK_RAW
- JP69 pad 2: /KNOCK_4_5 -> unconnected-(JP69-Pad2)
- JP70 pad 2: /KNOCK_1_3 -> unconnected-(JP70-Pad2)
- M11 pad N18: Net-(M11-PadN18) -> /LPS_SDA
- M11 pad N19: Net-(M11-PadN19) -> /LPS_SCL
- M11 pad N20: Net-(M11-PadN20) -> /SPI_SCK
- M11 pad N21: Net-(M11-PadN21) -> /SPI_MISO
- M11 pad N22: Net-(M11-PadN22) -> /SPI_MOSI
- M11 pad N23: Net-(M11-PadN23) -> /SPI_CS
- Q1 pad 1: /IGN_1 -> /OUT_IGN1
- Q2 pad 1: /IGN_2 -> /OUT_IGN2
- Q3 pad 1: /IGN_3 -> /OUT_IGN3
- Q4 pad 1: /IGN_4 -> /OUT_IGN4
- Q5 pad 1: /GP6 -> /OUT_IGN6
- Q6 pad 1: /GP5 -> /OUT_IGN5
- Q7 pad 1: /IGN_7 -> /OUT_IGN7
- Q8 pad 1: /IGN_8 -> /OUT_IGN8
Routing:
- net GND: track 385.9 -> 176.1 mm, vias 7 -> 0
- net /COIL_6: track 80.7 -> 22.7 mm, vias 20 -> 43
- net /COIL_5: track 53.5 -> 18.5 mm, vias 21 -> 36
- net /COIL_4: track 66.1 -> 32.5 mm, vias 20 -> 36
- net /GP6: track 30.8 -> 0.00 mm, vias 1 -> 0
- net /GP5: track 23.0 -> 0.00 mm
- net /MAIN_RELAY: track 37.2 -> 14.4 mm
- net /IGN_3: track 22.0 -> 0.00 mm
- net /COIL_3: track 32.5 -> 11.5 mm, vias 20 -> 41
- net /COIL_2: track 29.6 -> 8.73 mm, vias 20 -> 42
- net /IGN_4: track 20.1 -> 0.00 mm
- net /COIL_1: track 26.9 -> 10.8 mm, vias 20 -> 36
- net /IGN_1: track 10.8 -> 0.00 mm
- net /OUT_IGN6: track 7.51 -> 0.00 mm
- net /OUT_IGN4: track 6.14 -> 0.00 mm
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- removed copper zone on F.Cu, net GND

Commit message: Up 88
Parts:
- removed J17: SD, Connector_PinHeader_2.54mm:PinHeader_1x06_P2.54mm_Vertical
- removed JP10, JP11, JP12, JP15, JP19, JP28, JP30, JP34, JP36, JP37, JP38, JP39, JP40, JP45, JP53, JP55, JP57, JP58, JP6, JP60, JP61, JP62, JP63, JP66, JP67, JP68, JP69, JP70, JP71, JP72, JP74, JP75, JP76, JP79, JP80, JP82, JP83, JP84, JP87, JP88, JP9: Jumper_2_Open, rusefi_lib_private:SM0805_jumper
- removed MMCU18, MMCU19, MMCU20, MMCU21: MMCU, Connector_PinHeader_1.00mm:PinHeader_1x01_P1.00mm_Vertical
- added R17: 0, Resistor_SMD:R_0402_1005Metric, F.Cu at (248.8, 88.2)
- added R18: 0, Resistor_SMD:R_0402_1005Metric, F.Cu at (245.8, 84.3)
- added R19: 0, Resistor_SMD:R_0402_1005Metric, F.Cu at (251.7, 86.3)
- added R20: 0, Resistor_SMD:R_0402_1005Metric, F.Cu at (251.7, 84.3)
- added R21: 0, Resistor_SMD:R_0402_1005Metric, F.Cu at (245.8, 86.3)
- added R22: 0, Resistor_SMD:R_0402_1005Metric, F.Cu at (245.8, 88.2)
- added R23: 0, Resistor_SMD:R_0402_1005Metric, F.Cu at (248.8, 84.3)
- added R24: 0, Resistor_SMD:R_0402_1005Metric, F.Cu at (248.8, 86.3)
- J3: moved to B.Cu
- moved J3 94.5 mm to (159.5, 146.5), turned to 0 degrees
Connections:
- *ref1 pad 10: Net-(*ref1-Pad10) -> unconnected-(*ref1-Pad10)
- *ref1 pad 11: Net-(*ref1-Pad11) -> unconnected-(*ref1-Pad11)
- *ref1 pad 12: Net-(*ref1-Pad12) -> unconnected-(*ref1-Pad12)
- *ref1 pad 15: Net-(*ref1-Pad15) -> GND
- *ref1 pad 19: Net-(*ref1-Pad19) -> unconnected-(*ref1-Pad19)
- *ref1 pad 28: Net-(*ref1-Pad28) -> GND
- *ref1 pad 30: Net-(*ref1-Pad30) -> unconnected-(*ref1-Pad30)
- *ref1 pad 34: Net-(*ref1-Pad34) -> GND
- *ref1 pad 36: Net-(*ref1-Pad36) -> unconnected-(*ref1-Pad36)
- *ref1 pad 37: Net-(*ref1-Pad37) -> unconnected-(*ref1-Pad37)
- *ref1 pad 38: Net-(*ref1-Pad38) -> unconnected-(*ref1-Pad38)
- *ref1 pad 39: Net-(*ref1-Pad39) -> GND
- *ref1 pad 40: Net-(*ref1-Pad40) -> GND
- *ref1 pad 45: Net-(*ref1-Pad45) -> GND
- *ref1 pad 53: Net-(*ref1-Pad53) -> unconnected-(*ref1-Pad53)
- *ref1 pad 55: Net-(*ref1-Pad55) -> unconnected-(*ref1-Pad55)
- *ref1 pad 57: Net-(*ref1-Pad57) -> unconnected-(*ref1-Pad57)
- *ref1 pad 58: Net-(*ref1-Pad58) -> unconnected-(*ref1-Pad58)
- *ref1 pad 6: Net-(*ref1-Pad6) -> GND
- *ref1 pad 60: Net-(*ref1-Pad60) -> unconnected-(*ref1-Pad60)
- *ref1 pad 61: Net-(*ref1-Pad61) -> unconnected-(*ref1-Pad61)
- *ref1 pad 62: Net-(*ref1-Pad62) -> unconnected-(*ref1-Pad62)
- *ref1 pad 63: Net-(*ref1-Pad63) -> unconnected-(*ref1-Pad63)
- *ref1 pad 66: Net-(*ref1-Pad66) -> unconnected-(*ref1-Pad66)
- *ref1 pad 67: Net-(*ref1-Pad67) -> unconnected-(*ref1-Pad67)
- *ref1 pad 68: Net-(*ref1-Pad68) -> unconnected-(*ref1-Pad68)
- *ref1 pad 69: Net-(*ref1-Pad69) -> unconnected-(*ref1-Pad69)
- *ref1 pad 70: Net-(*ref1-Pad70) -> unconnected-(*ref1-Pad70)
- *ref1 pad 71: Net-(*ref1-Pad71) -> unconnected-(*ref1-Pad71)
- *ref1 pad 72: Net-(*ref1-Pad72) -> unconnected-(*ref1-Pad72)
- *ref1 pad 74: Net-(*ref1-Pad74) -> unconnected-(*ref1-Pad74)
- *ref1 pad 75: Net-(*ref1-Pad75) -> unconnected-(*ref1-Pad75)
- *ref1 pad 76: Net-(*ref1-Pad76) -> unconnected-(*ref1-Pad76)
- *ref1 pad 79: Net-(*ref1-Pad79) -> unconnected-(*ref1-Pad79)
- *ref1 pad 80: Net-(*ref1-Pad80) -> unconnected-(*ref1-Pad80)
- *ref1 pad 82: Net-(*ref1-Pad82) -> unconnected-(*ref1-Pad82)
- *ref1 pad 83: Net-(*ref1-Pad83) -> unconnected-(*ref1-Pad83)
- *ref1 pad 84: Net-(*ref1-Pad84) -> GND
- *ref1 pad 87: Net-(*ref1-Pad87) -> unconnected-(*ref1-Pad87)
- *ref1 pad 88: Net-(*ref1-Pad88) -> unconnected-(*ref1-Pad88)
- *ref1 pad 9: Net-(*ref1-Pad9) -> unconnected-(*ref1-Pad9)
- J3 pad 2: /PB9 -> /SD_CS
- J3 pad 3: /PC12 -> /SD_MOSI
- J3 pad 5: /PC10 -> /SD_CLK
- J3 pad 7: /PC11 -> /SD_MISO
- JP20 pad 2: /USBD+ -> /USBP
- JP21 pad 2: /USBD- -> /USBM
- M11 pad N10: Net-(M11-PadN10) -> /SD_MISO
- M11 pad N11: Net-(M11-PadN11) -> /SD_MOSI
- M11 pad N8: Net-(M11-PadN8) -> /SD_CS
- M11 pad N9: Net-(M11-PadN9) -> /SD_CLK
- Q1 pad 1: /OUT_IGN1 -> Net-(Q1-Pad1)
- Q2 pad 1: /OUT_IGN2 -> Net-(Q2-Pad1)
- Q3 pad 1: /OUT_IGN3 -> Net-(Q3-Pad1)
- Q4 pad 1: /OUT_IGN4 -> Net-(Q4-Pad1)
- Q5 pad 1: /OUT_IGN6 -> Net-(Q5-Pad1)
- Q6 pad 1: /OUT_IGN5 -> Net-(Q6-Pad1)
- Q7 pad 1: /OUT_IGN7 -> Net-(Q7-Pad1)
- Q8 pad 1: /OUT_IGN8 -> Net-(Q8-Pad1)
Routing:
- net GND: track 176.1 -> 0.00 mm
- net /12V_KEY: track 158.1 -> 1.22 mm
- net /COIL_4: track 32.5 -> 0.00 mm
- net /FUEL_RELAY_GP1: track 26.6 -> 1.07 mm
- net Net-(*ref1-Pad88): track 23.8 -> 0.00 mm
- net /ICV_CLOSE_LS1: track 24.3 -> 1.07 mm
- net Net-(*ref1-Pad56): track 22.9 -> 0.00 mm
- net /COIL_6: track 22.7 -> 0.00 mm
- net Net-(*ref1-Pad59): track 22.5 -> 0.00 mm
- net /CRANK+: track 22.2 -> 0.00 mm
- net Net-(*ref1-Pad62): track 21.6 -> 0.00 mm
- net Net-(*ref1-Pad83): track 21.5 -> 0.00 mm
- net Net-(*ref1-Pad80): track 21.1 -> 0.00 mm
- net Net-(*ref1-Pad60): track 21.0 -> 0.00 mm
- net Net-(*ref1-Pad63): track 20.9 -> 0.00 mm
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
Commit message: Up hellen88bmw
Parts:
- removed JP13, JP18, JP2, JP64, JP65, JP8, JP81: Jumper_2_Open, rusefi_lib_private:SM0805_jumper
- added C8: 10uF, Capacitor_SMD:C_0402_1005Metric, F.Cu at (19.7, 108.5)
- added KNOCK_RAW2: IN_KNOCK2_RAW, Connector_PinHeader_1.00mm:PinHeader_1x01_P1.00mm_Vertical, F.Cu at (47.5, 136.8)
- added M12: Module-knock-0.1, knock:knock, F.Cu at (21.8, 70.6)
- added R25: 2k7, Resistor_SMD:R_0603_1608Metric, F.Cu at (24.5, 113.2)
- added R26: 2k7, Resistor_SMD:R_0603_1608Metric, F.Cu at (24.2, 109.0)
- added R27: DNP, Resistor_SMD:R_0603_1608Metric, F.Cu at (20.5, 113.1)
- added cr1: cr, Connector_PinHeader_1.00mm:PinHeader_1x01_P1.00mm_Vertical, F.Cu at (134.8, 27.2)
- added cr10: cr, Connector_PinHeader_1.00mm:PinHeader_1x01_P1.00mm_Vertical, F.Cu at (129.0, 27.5)
- added cr11: cr, Connector_PinHeader_1.00mm:PinHeader_1x01_P1.00mm_Vertical, F.Cu at (132.5, 27.0)
- added cr12: cr, Connector_PinHeader_1.00mm:PinHeader_1x01_P1.00mm_Vertical, F.Cu at (106.5, 27.8)
- added cr13: cr, Connector_PinHeader_1.00mm:PinHeader_1x01_P1.00mm_Vertical, F.Cu at (113.2, 27.8)
- added cr14: cr, Connector_PinHeader_1.00mm:PinHeader_1x01_P1.00mm_Vertical, F.Cu at (120.0, 28.0)
- added cr15: cr, Connector_PinHeader_1.00mm:PinHeader_1x01_P1.00mm_Vertical, F.Cu at (123.5, 27.2)
- added cr16: cr, Connector_PinHeader_1.00mm:PinHeader_1x01_P1.00mm_Vertical, F.Cu at (126.8, 22.8)
- added cr17: cr, Connector_PinHeader_1.00mm:PinHeader_1x01_P1.00mm_Vertical, F.Cu at (130.2, 22.8)
- added cr18: cr, Connector_PinHeader_1.00mm:PinHeader_1x01_P1.00mm_Vertical, F.Cu at (133.2, 23.0)
- added cr19: cr, Connector_PinHeader_1.00mm:PinHeader_1x01_P1.00mm_Vertical, F.Cu at (175.2, 27.2)
- added cr2: cr, Connector_PinHeader_1.00mm:PinHeader_1x01_P1.00mm_Vertical, F.Cu at (137.0, 23.8)
- added cr20: cr, Connector_PinHeader_1.00mm:PinHeader_1x01_P1.00mm_Vertical, F.Cu at (178.0, 27.5)
- added cr21: cr, Connector_PinHeader_1.00mm:PinHeader_1x01_P1.00mm_Vertical, F.Cu at (181.5, 27.5)
- added cr22: cr, Connector_PinHeader_1.00mm:PinHeader_1x01_P1.00mm_Vertical, F.Cu at (194.8, 27.5)
- added cr23: cr, Connector_PinHeader_1.00mm:PinHeader_1x01_P1.00mm_Vertical, F.Cu at (197.5, 27.5)
- added cr3: cr, Connector_PinHeader_1.00mm:PinHeader_1x01_P1.00mm_Vertical, F.Cu at (141.8, 26.2)
- added cr4: cr, Connector_PinHeader_1.00mm:PinHeader_1x01_P1.00mm_Vertical, F.Cu at (96.5, 27.8)
- added cr5: cr, Connector_PinHeader_1.00mm:PinHeader_1x01_P1.00mm_Vertical, F.Cu at (124.5, 22.8)
- added cr6: cr, Connector_PinHeader_1.00mm:PinHeader_1x01_P1.00mm_Vertical, F.Cu at (156.5, 28.0)
- added cr7: cr, Connector_PinHeader_1.00mm:PinHeader_1x01_P1.00mm_Vertical, F.Cu at (159.2, 28.0)
- added cr8: cr, Connector_PinHeader_1.00mm:PinHeader_1x01_P1.00mm_Vertical, F.Cu at (100.2, 26.8)
- added cr9: cr, Connector_PinHeader_1.00mm:PinHeader_1x01_P1.00mm_Vertical, F.Cu at (125.8, 27.5)
- JP1, JP14, JP16, JP17, JP20, JP21, JP22, JP23, JP24, JP25, JP26, JP27, JP29, JP3, JP31, JP32, JP33, JP35, JP4, JP41, JP42, JP43, JP44, JP46, JP47, JP48, JP49, JP5, JP50, JP51, JP52, JP54, JP56, JP59, JP7, JP73, JP77, JP78, JP85, JP86: footprint rusefi_lib_private:SM0805_jumper -> rusefi_lib:SM0805_jumper
- M1: footprint rusefi_lib_private:MOD_HELLEN_POWER_12 -> power12:power12
- M10: footprint rusefi_lib_private:MOD_HELLEN_IGN8 -> ign8:ign8
- M11: footprint rusefi_lib_private:MOD_HELLEN_MCU -> mcu:mcu
- M2, M4: footprint rusefi_lib_private:MOD_HELLEN_CAN -> can:can
- M3: footprint rusefi_lib_private:MOD_HELLEN_WBO -> wbo:wbo
- M5: footprint rusefi_lib_private:MOD_HELLEN_POWER_5 -> power5:power5
- M6: footprint rusefi_lib_private:MOD_HELLEN_VR -> vr:vr
- M7: footprint rusefi_lib_private:MOD_HELLEN_INPUT -> input:input
- M8: footprint rusefi_lib_private:MOD_HELLEN_KNOCK -> knock:knock
- M9: footprint rusefi_lib_private:MOD_HELLEN_OUTPUT -> output:output
- U2: footprint rusefi_lib_private:MPX-4_MAP -> rusefi_lib:MPX-4_MAP
- moved M8 135.0 mm to (47.0, 69.4)
- moved KNOCK_RAW1 78.9 mm to (135.5, 17.2)
- moved R24 69.4 mm to (202.2, 137.8), turned to 180 degrees
- moved R20 66.1 mm to (202.2, 128.2)
- moved R17 55.5 mm to (202.2, 118.5)
- moved R21 51.5 mm to (202.2, 58.8), turned to 180 degrees
- moved R18 50.9 mm to (201.5, 109.2)
- moved R19 49.5 mm to (202.2, 88.2)
- moved R22 47.8 mm to (202.2, 68.8), turned to 180 degrees
- moved R23 46.9 mm to (202.3, 78.2), turned to 180 degrees
- moved M9 23.5 mm to (125.4, 81.6)
- moved M3 21.5 mm to (133.3, 138.2)
- moved M5 20.3 mm to (143.4, 145.9)
- moved M11 18.6 mm to (177.2, 95.6)
- moved M7 17.2 mm to (177.2, 78.0)
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Connections:
- net /FUEL_RELAY_GP1 renamed /FUEL_RELAY
- net /TPS1 renamed /TPS
- *ref1 pad 11: unconnected-(*ref1-Pad11) -> Net-(*ref1-Pad11)
- *ref1 pad 12: unconnected-(*ref1-Pad12) -> Net-(*ref1-Pad12)
- *ref1 pad 19: unconnected-(*ref1-Pad19) -> Net-(*ref1-Pad19)
- *ref1 pad 30: unconnected-(*ref1-Pad30) -> Net-(*ref1-Pad30)
- *ref1 pad 36: unconnected-(*ref1-Pad36) -> Net-(*ref1-Pad36)
- *ref1 pad 37: unconnected-(*ref1-Pad37) -> Net-(*ref1-Pad37)
- *ref1 pad 38: unconnected-(*ref1-Pad38) -> Net-(*ref1-Pad38)
- *ref1 pad 55: unconnected-(*ref1-Pad55) -> GND
- *ref1 pad 60: unconnected-(*ref1-Pad60) -> Net-(*ref1-Pad60)
- *ref1 pad 62: unconnected-(*ref1-Pad62) -> Net-(*ref1-Pad62)
- *ref1 pad 66: unconnected-(*ref1-Pad66) -> Net-(*ref1-Pad66)
- *ref1 pad 67: unconnected-(*ref1-Pad67) -> Net-(*ref1-Pad67)
- *ref1 pad 68: unconnected-(*ref1-Pad68) -> Net-(*ref1-Pad68)
- *ref1 pad 69: unconnected-(*ref1-Pad69) -> /IN_KNOCK1_RAW
- *ref1 pad 70: unconnected-(*ref1-Pad70) -> /IN_KNOCK2_RAW
- *ref1 pad 71: unconnected-(*ref1-Pad71) -> GND
- *ref1 pad 82: unconnected-(*ref1-Pad82) -> Net-(*ref1-Pad82)
- *ref1 pad 83: unconnected-(*ref1-Pad83) -> Net-(*ref1-Pad83)
- *ref1 pad 87: unconnected-(*ref1-Pad87) -> Net-(*ref1-Pad87)
- *ref1 pad 88: unconnected-(*ref1-Pad88) -> Net-(*ref1-Pad88)
- D12 pad 2: /12_MAIN_RELAY -> V12_RAW
- J18 pad R: unconnected-(J18-PadR) -> Net-(J18-PadR)
- J4 pad 5: /12_MAIN_RELAY -> V12_RAW
- JP17 pad 2: /CAM -> /IN_CAM
- JP26 pad 2: /12V_KEY -> V12_RAW
- JP35 pad 2: /INJ7 -> /INJ8
- JP54 pad 2: /12_MAIN_RELAY -> V12_RAW
- JP56 pad 2: /12V_KEY -> V12_RAW
- JP7 pad 2: /INJ8 -> /INJ7
- JP73 pad 2: /TPS_AV2 -> /IN_TPS
- JP77 pad 2: /IAT_AT2 -> /IAT
- JP78 pad 2: /CLT_AT1 -> /CLT
- KNOCK_RAW1 pad 1: /IN_KNOCK_RAW -> /IN_KNOCK1_RAW
- M11 pad E6: /MAIN -> /OUT_MAIN
- M11 pad S15: /CAM1 -> /CAM
- M11 pad S24: /TPS2 -> unconnected-(M11-PadS24)
- M11 pad S27: /CAM2 -> unconnected-(M11-PadS27)
- M7 pad N19: /CAM1 -> /CAM
- M7 pad N22: /KNOCK1 -> /IN_KNOCK1
- M7 pad N24: /KNOCK2 -> /IN_KNOCK2
- M7 pad N7: /CAM2 -> unconnected-(M7-PadN7)
- M7 pad S10: /IN_TPS1 -> /IN_TPS
- M7 pad S15: /IN_CLT -> /CLT
- M7 pad S16: /IN_IAT -> /IAT
- M7 pad S17: /IN_TPS2 -> unconnected-(M7-PadS17)
- M7 pad S21: /IN_CAM2 -> unconnected-(M7-PadS21)
- M7 pad S5: /IN_CAM1 -> /IN_CAM
- M8 pad W1: /IN_KNOCK_RAW -> /IN_KNOCK1_RAW
- M9 pad W40: /MAIN -> /MAIN_RELAY
- U5 pad 5: GND -> /IN_KNOCK2
Routing:
- net /OUT_MAIN: track 0.00 -> 6.80 mm
- net /MAIN: track 6.80 -> 0.00 mm
- net /CAM1: track 3.59 -> 0.00 mm
- net unconnected-(M7-PadN7): track 0.00 -> 3.59 mm
- net /KNOCK1: track 3.59 -> 0.00 mm
- net /IN_KNOCK1: track 0.00 -> 3.59 mm
- net /CAM2: track 3.59 -> 0.00 mm
- net /CAM: track 0.36 -> 3.59 mm
- net V12_RAW: track 0.00 -> 1.22 mm
- net /12V_KEY: track 1.22 -> 0.00 mm
- net (no net): track 0.00 -> 1.09 mm
- net /ICV_CLOSE_LS1: track 1.07 -> 0.00 mm
- net /TPS_AV2: track 1.02 -> 0.00 mm
- net /IN_TPS: track 0.00 -> 1.02 mm
- net /MIL_GP3: track 0.73 -> 0.00 mm
Other:
- board text added: "Always looking for C/C++/PHP/Java developers"
- board text added: "https://rusefi.com/s/mission"

Commit message: Up hellen88bmw
Parts:
- removed JP48: Jumper_2_Open, rusefi_lib:SM0805_jumper
- added MMCU14: MMCU, Connector_PinHeader_1.00mm:PinHeader_1x01_P1.00mm_Vertical, F.Cu at (79.8, -5.50)
- added MMCU15: MMCU, Connector_PinHeader_1.00mm:PinHeader_1x01_P1.00mm_Vertical, F.Cu at (79.8, -11.6)
- added MMCU16: MMCU, Connector_PinHeader_1.00mm:PinHeader_1x01_P1.00mm_Vertical, F.Cu at (83.1, -5.50)
- added MMCU17: MMCU, Connector_PinHeader_1.00mm:PinHeader_1x01_P1.00mm_Vertical, F.Cu at (96.5, -11.6)
- added MMCU18: MMCU, Connector_PinHeader_1.00mm:PinHeader_1x01_P1.00mm_Vertical, F.Cu at (89.8, -5.50)
- added MMCU19: MMCU, Connector_PinHeader_1.00mm:PinHeader_1x01_P1.00mm_Vertical, F.Cu at (89.8, -8.55)
- added VOUT10: Pad, Connector_PinHeader_1.00mm:PinHeader_1x01_P1.00mm_Vertical, F.Cu at (83.1, -8.55)
- added VOUT11: Pad, Connector_PinHeader_1.00mm:PinHeader_1x01_P1.00mm_Vertical, F.Cu at (83.1, -14.7)
- added VOUT12: Pad, Connector_PinHeader_1.00mm:PinHeader_1x01_P1.00mm_Vertical, F.Cu at (93.2, -11.6)
- added VOUT13: Pad, Connector_PinHeader_1.00mm:PinHeader_1x01_P1.00mm_Vertical, F.Cu at (79.8, -14.7)
- added VOUT14: VOUT4, Connector_PinHeader_1.00mm:PinHeader_1x01_P1.00mm_Vertical, F.Cu at (96.5, -14.7)
- added VOUT15: VOUT4, Connector_PinHeader_1.00mm:PinHeader_1x01_P1.00mm_Vertical, F.Cu at (89.8, -11.6)
- added VOUT16: Pad, Connector_PinHeader_1.00mm:PinHeader_1x01_P1.00mm_Vertical, F.Cu at (83.1, -11.6)
- added VOUT17: Pad, Connector_PinHeader_1.00mm:PinHeader_1x01_P1.00mm_Vertical, F.Cu at (86.5, -8.55)
- added VOUT18: Pad, Connector_PinHeader_1.00mm:PinHeader_1x01_P1.00mm_Vertical, F.Cu at (79.8, -8.55)
- added VOUT19: Pad, Connector_PinHeader_1.00mm:PinHeader_1x01_P1.00mm_Vertical, F.Cu at (86.5, -5.50)
- added VOUT20: Pad, Connector_PinHeader_1.00mm:PinHeader_1x01_P1.00mm_Vertical, F.Cu at (86.5, -11.6)
- added VOUT7: Pad, Connector_PinHeader_1.00mm:PinHeader_1x01_P1.00mm_Vertical, F.Cu at (86.5, -14.7)
- added VOUT8: Pad, Connector_PinHeader_1.00mm:PinHeader_1x01_P1.00mm_Vertical, F.Cu at (93.2, -14.7)
- added VOUT9: Pad, Connector_PinHeader_1.00mm:PinHeader_1x01_P1.00mm_Vertical, F.Cu at (89.8, -14.7)
- added cr24: cr, Connector_PinHeader_1.00mm:PinHeader_1x01_P1.00mm_Vertical, F.Cu at (93.2, -8.55)
- moved cr22 25.5 mm to (195.2, 53.0)
- moved cr20 25.5 mm to (177.8, 53.0)
- moved cr21 25.5 mm to (181.2, 53.0)
- moved cr23 25.5 mm to (197.5, 53.0)
- moved JP23 11.9 mm to (174.0, 67.0)
- moved JP85 7.43 mm to (187.8, 62.0)
- moved JP86 7.41 mm to (191.0, 62.0)
- moved JP54 7.24 mm to (193.0, 55.0)
- moved JP24 6.87 mm to (180.2, 62.0)
- moved JP27 5.44 mm to (199.8, 55.0)
- moved JP52 1.39 mm to (183.0, 62.0)
- moved JP25 1.21 mm to (186.0, 55.1)
- moved JP51 0.97 mm to (177.5, 62.0)
- moved JP26 0.40 mm to (189.5, 55.0)
Connections:
- D14 pad 2: /IDLE_LS2 -> /OUT_IDLE
- D15 pad 2: /FUEL_RELAY -> /OUT_PUMP
- JP1 pad 2: /FUEL_RELAY -> /OUT_PUMP
- JP29 pad 2: /IDLE_LS2 -> /OUT_IDLE
- JP41 pad 2: /MAF_AV4 -> /IN_MAF
- JP42 pad 2: /VSS_AV3 -> /IN_VSS
- JP46 pad 2: /ECON -> /OUT_FUEL_CONSUM
- JP47 pad 2: /TACH_GP4 -> /OUT_TACH
- M11 pad E10: /VVT1_1 -> Net-(M11-PadE10)
- M11 pad E12: /WASTEGATE -> unconnected-(M11-PadE12)
- M11 pad E16: /VVT2_B1 -> Net-(M11-PadE16)
- M11 pad E17: /VVT2_B2 -> Net-(M11-PadE17)
- M11 pad E21: /VVT1_2 -> Net-(M11-PadE21)
- M11 pad S24: unconnected-(M11-PadS24) -> Net-(M11-PadS24)
- M11 pad S27: unconnected-(M11-PadS27) -> Net-(M11-PadS27)
- M9 pad S13: /OUT_VVT1_1 -> Net-(M9-PadS13)
- M9 pad S14: /OUT_VVT1_1 -> Net-(M9-PadS14)
- M9 pad S4: /OUT_VVT2_B1 -> Net-(M9-PadS4)
- M9 pad S5: /OUT_VVT2_B2 -> Net-(M9-PadS5)
- M9 pad W1: /OUT_VVT1_2 -> Net-(M9-PadW1)
- M9 pad W2: /OUT_VVT1_2 -> Net-(M9-PadW2)
- M9 pad W26: /VVT1_2 -> Net-(M9-PadW26)
- M9 pad W27: /VVT1_1 -> Net-(M9-PadW27)
- M9 pad W29: /VVT1_2 -> Net-(M9-PadW29)
- M9 pad W30: /VVT2_B2 -> Net-(M9-PadW30)
- M9 pad W31: /VVT2_B1 -> Net-(M9-PadW31)
- M9 pad W34: /WASTEGATE -> Net-(M9-PadW34)
- M9 pad W36: /VVT1_1 -> Net-(M9-PadW36)
- M9 pad W4: /OUT_WASTEGATE -> Net-(M9-PadW4)
- R4 pad 2: /MAF_AV4 -> /IN_MAF
Routing:
- net /COIL_6: track 0.00 -> 46.2 mm
- net GNDA: track 48.6 -> 6.54 mm
- net V5A: track 37.5 -> 79.6 mm
- net /COIL_3: track 0.00 -> 39.7 mm
- net /COIL_5: track 0.00 -> 38.6 mm
- net Net-(*ref1-Pad24): track 0.00 -> 19.2 mm
- net Net-(*ref1-Pad52): track 0.00 -> 18.7 mm
- net Net-(*ref1-Pad27): track 0.00 -> 12.5 mm
- net /COIL_1: track 0.00 -> 12.5 mm
- net Net-(*ref1-Pad26): track 0.00 -> 12.0 mm
- net Net-(*ref1-Pad86): track 0.00 -> 11.9 mm
- net Net-(*ref1-Pad85): track 0.00 -> 11.9 mm
- net Net-(*ref1-Pad54): track 0.00 -> 11.7 mm
- net /COIL_2: track 0.00 -> 11.6 mm
- net /COIL_7: track 0.00 -> 11.6 mm
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Other:
- board text added: "87"
- board text added: "88"

Commit message: Up hellen88bmw 5.07.2021
Parts:
- moved OUT_INJ1 273.0 mm to (-37.0, 183.8)
- moved OUT_INJ2 273.0 mm to (-37.2, 179.5)
- moved OUT_INJ3 273.0 mm to (-36.8, 192.2)
- moved OUT_INJ4 273.0 mm to (-37.0, 176.2)
- moved OUT_INJ5 273.0 mm to (-37.0, 168.2)
- moved OUT_INJ7 273.0 mm to (-37.0, 188.0)
- moved OUT_INJ8 273.0 mm to (-37.8, 163.0)
- moved VOUT1 273.0 mm to (-47.5, 172.5)
- moved VOUT4 273.0 mm to (-47.8, 189.8)
- moved VOUT6 273.0 mm to (-47.5, 175.5)
- moved MMCU16 234.0 mm to (270.4, 134.8)
- moved MMCU19 234.0 mm to (277.1, 131.8)
- moved VOUT10 234.0 mm to (270.4, 131.8)
- moved VOUT11 234.0 mm to (270.4, 125.7)
- moved VOUT16 234.0 mm to (270.4, 128.8)
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Connections:
- J3 pad 4: /3.3V -> +3V3
- J4 pad 3: /3.3V -> +3V3
- Q2 pad 2: /COIL_2 -> /COIL_4
- Q3 pad 2: /COIL_3 -> /COIL_2
- Q4 pad 2: /COIL_4 -> /COIL_6
- Q5 pad 2: /COIL_5 -> /COIL_3
- Q6 pad 2: /COIL_6 -> /COIL_5
- R11 pad 2: /COIL_6 -> /COIL_5
- R12 pad 1: /OUT_IGN6 -> /OUT_IGN3
- R12 pad 2: /COIL_5 -> /COIL_3
- R13 pad 1: /OUT_IGN4 -> /OUT_IGN6
- R13 pad 2: /COIL_4 -> /COIL_6
- R18 pad 1: /OUT_IGN2 -> /OUT_IGN4
- R19 pad 1: /OUT_IGN3 -> /OUT_IGN2
- R22 pad 2: /OUT_IGN6 -> /OUT_IGN3
- R23 pad 2: /OUT_IGN4 -> /OUT_IGN6
- R8 pad 1: /COIL_2 -> /COIL_4
- R8 pad 2: /OUT_IGN2 -> /OUT_IGN4
- R9 pad 1: /COIL_3 -> /COIL_2
- R9 pad 2: /OUT_IGN3 -> /OUT_IGN2
Routing:
- net V12_RAW: track 1.22 -> 128.0 mm
- net /COIL_8: track 10.7 -> 104.1 mm
- net /CAN+: track 11.6 -> 97.2 mm
- net /COIL_7: track 11.6 -> 93.9 mm
- net /CAN-: track 9.76 -> 90.7 mm
- net /COIL_1: track 12.5 -> 83.6 mm
- net /COIL_4: track 0.00 -> 64.0 mm, vias 36 -> 42
- net /OUT_IGN5: track 2.02 -> 58.4 mm
- net /OUT_IDLE: track 0.00 -> 53.8 mm
- net /OUT_PUMP: track 1.07 -> 51.5 mm
- net /OUT_IGN8: track 2.03 -> 49.4 mm, vias 0 -> 2
- net /OUT_IGN3: track 2.04 -> 47.8 mm
- net /OUT_IGN7: track 2.02 -> 46.9 mm, vias 0 -> 2
- net /COIL_2: track 11.6 -> 51.2 mm, vias 42 -> 41
- net /OUT_IGN6: track 2.02 -> 41.1 mm, vias 0 -> 2
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