File: boards/hellen88bmw/kicad6/hellen88bmw.kicad_pcb (KiCad board)
At the start: 2 copper layers, 160 x 118 mm, 267 parts, among them J1 920-462A2021Y10101, J10 Conn_01x12, J11 Conn_01x12, J12 Conn_01x12, J13 Conn_01x12, J14 VRIN1, J15 VRIN2, J16 VROUT1, J18 C165947, J2 UB-20PMFP-LC7002, J3 Micro_SD_Card, J4 Conn_01x05, J5 Conn_01x12, J6 Conn_01x12, J7 Conn_01x12, J8 Conn_01x12, J9 Conn_01x12, M1 Module-power12-0.1, M10 Module-ign8-0.1, M11 Module-mcu-0.1, M12 Module-knock-0.1, M2 Module-can-0.1, M3 Module-wbo-0.1, M4 Module-can-0.1, M5 Module-power5-0.1, M6 Module-vr-0.1, M7 Module-input-0.1, M8 Module-knock-0.1, M9 Module-output-0.1, Q1 NGD8201AN, Q2 NGD8201AN, Q3 NGD8201AN, Q4 NGD8201AN, Q5 NGD8201AN, Q6 NGD8201AN, Q7 NGD8201AN, Q8 NGD8201AN, SW1 BOOT0, SW2 RESET, U1 MPXA6115A, U2 MPX4_MAP, U3 LIS2DW12TR, U4 LPS25HB, U5 MCP6002-xSN

Commit message: Up hellen88bmw 6.07.2021
Parts:
- removed OUT_INJ1: OUT_INJ1, Connector_PinHeader_1.00mm:PinHeader_1x01_P1.00mm_Vertical
- removed OUT_INJ2: OUT_INJ2, Connector_PinHeader_1.00mm:PinHeader_1x01_P1.00mm_Vertical
- removed OUT_INJ3: OUT_INJ3, Connector_PinHeader_1.00mm:PinHeader_1x01_P1.00mm_Vertical
- removed OUT_INJ4: OUT_INJ4, Connector_PinHeader_1.00mm:PinHeader_1x01_P1.00mm_Vertical
- removed OUT_INJ5: OUT_INJ5, Connector_PinHeader_1.00mm:PinHeader_1x01_P1.00mm_Vertical
- removed OUT_INJ6: OUT_INJ6, Connector_PinHeader_1.00mm:PinHeader_1x01_P1.00mm_Vertical
- removed OUT_INJ7: OUT_INJ7, Connector_PinHeader_1.00mm:PinHeader_1x01_P1.00mm_Vertical
- removed OUT_INJ8: OUT_INJ8, Connector_PinHeader_1.00mm:PinHeader_1x01_P1.00mm_Vertical
- added JP2: Jumper_2_Open, rusefi_lib:SM0805_jumper, F.Cu at (-18.5, 23.0)
- added MMCU20: MMCU, Connector_PinHeader_1.00mm:PinHeader_1x01_P1.00mm_Vertical, F.Cu at (0.11, 29.3)
- added MMCU21: MMCU, Connector_PinHeader_1.00mm:PinHeader_1x01_P1.00mm_Vertical, F.Cu at (-6.59, 29.3)
- added MMCU22: MMCU, Connector_PinHeader_1.00mm:PinHeader_1x01_P1.00mm_Vertical, F.Cu at (-3.61, 23.2)
- added MMCU23: MMCU, Connector_PinHeader_1.00mm:PinHeader_1x01_P1.00mm_Vertical, F.Cu at (-6.59, 35.4)
- added MMCU37: MMCU, Connector_PinHeader_1.00mm:PinHeader_1x01_P1.00mm_Vertical, F.Cu at (-13.7, 23.2)
- added MMCU38: MMCU, Connector_PinHeader_1.00mm:PinHeader_1x01_P1.00mm_Vertical, F.Cu at (-3.24, 29.3)
- added MMCU39: MMCU, Connector_PinHeader_1.00mm:PinHeader_1x01_P1.00mm_Vertical, F.Cu at (-9.94, 35.4)
- added MMCU40: MMCU, Connector_PinHeader_1.00mm:PinHeader_1x01_P1.00mm_Vertical, F.Cu at (-13.3, 32.4)
- added MMCU41: MMCU, Connector_PinHeader_1.00mm:PinHeader_1x01_P1.00mm_Vertical, F.Cu at (-20.0, 26.0)
- added P1: P, Connector_PinHeader_1.00mm:PinHeader_1x01_P1.00mm_Vertical, F.Cu at (-13.3, 26.3)
- added P2: P, Connector_PinHeader_1.00mm:PinHeader_1x01_P1.00mm_Vertical, F.Cu at (-13.3, 29.3)
- added P3: P, Connector_PinHeader_1.00mm:PinHeader_1x01_P1.00mm_Vertical, F.Cu at (-20.0, 35.1)
- added P4: P, Connector_PinHeader_1.00mm:PinHeader_1x01_P1.00mm_Vertical, F.Cu at (-9.94, 29.3)
- added P5: P, Connector_PinHeader_1.00mm:PinHeader_1x01_P1.00mm_Vertical, F.Cu at (-9.94, 26.3)
- added P6: P, Connector_PinHeader_1.00mm:PinHeader_1x01_P1.00mm_Vertical, F.Cu at (3.09, 23.2)
- added VIN18: Pad, Connector_PinHeader_1.00mm:PinHeader_1x01_P1.00mm_Vertical, F.Cu at (-16.6, 32.4)
- added VIN19: Pad, Connector_PinHeader_1.00mm:PinHeader_1x01_P1.00mm_Vertical, F.Cu at (-16.6, 29.3)
- added VIN20: Pad, Connector_PinHeader_1.00mm:PinHeader_1x01_P1.00mm_Vertical, F.Cu at (-6.59, 26.3)
- added VIN21: Pad, Connector_PinHeader_1.00mm:PinHeader_1x01_P1.00mm_Vertical, F.Cu at (-9.94, 32.4)
- added VIN22: VIN5, Connector_PinHeader_1.00mm:PinHeader_1x01_P1.00mm_Vertical, F.Cu at (-13.3, 35.4)
- added VIN23: Pad, Connector_PinHeader_1.00mm:PinHeader_1x01_P1.00mm_Vertical, F.Cu at (-16.6, 35.4)
- added VIN24: Pad, Connector_PinHeader_1.00mm:PinHeader_1x01_P1.00mm_Vertical, F.Cu at (-20.0, 29.0)
- added VIN25: Pad, Connector_PinHeader_1.00mm:PinHeader_1x01_P1.00mm_Vertical, F.Cu at (-16.6, 26.3)
- added VOUT21: Pad, Connector_PinHeader_1.00mm:PinHeader_1x01_P1.00mm_Vertical, F.Cu at (-3.24, 32.4)
- added VOUT22: VOUT4, Connector_PinHeader_1.00mm:PinHeader_1x01_P1.00mm_Vertical, F.Cu at (3.46, 26.3)
- added VOUT23: VOUT4, Connector_PinHeader_1.00mm:PinHeader_1x01_P1.00mm_Vertical, F.Cu at (-3.24, 26.3)
- added VOUT24: Pad, Connector_PinHeader_1.00mm:PinHeader_1x01_P1.00mm_Vertical, F.Cu at (-20.0, 32.1)
- added VOUT25: Pad, Connector_PinHeader_1.00mm:PinHeader_1x01_P1.00mm_Vertical, F.Cu at (-6.59, 32.4)
- added VOUT26: Pad, Connector_PinHeader_1.00mm:PinHeader_1x01_P1.00mm_Vertical, F.Cu at (-6.96, 23.2)
- added VOUT27: Pad, Connector_PinHeader_1.00mm:PinHeader_1x01_P1.00mm_Vertical, F.Cu at (-0.26, 23.2)
- added VOUT28: Pad, Connector_PinHeader_1.00mm:PinHeader_1x01_P1.00mm_Vertical, F.Cu at (0.11, 26.3)
- added VOUT29: Pad, Connector_PinHeader_1.00mm:PinHeader_1x01_P1.00mm_Vertical, F.Cu at (-10.3, 23.2)
- moved MMCU35 7.06 mm to (144.0, 90.8)
- moved M7 1.80 mm to (180.7, 76.0)
- moved MMCU33 1.80 mm to (144.0, 89.0)
- moved MMCU34 1.80 mm to (144.0, 87.3)
- moved MMCU36 1.80 mm to (154.7, 92.0)
- moved VIN1 1.80 mm to (174.2, 75.0)
- moved VIN10 1.80 mm to (155.5, 73.8)
- moved VIN11 1.80 mm to (147.5, 74.0)
- moved VIN12 1.80 mm to (154.2, 73.8)
- moved VIN13 1.80 mm to (156.7, 73.8)
- moved VIN14 1.80 mm to (163.5, 75.0)
- moved VIN15 1.80 mm to (161.7, 75.0)
- moved VIN16 1.80 mm to (148.5, 78.8)
- moved VIN17 1.80 mm to (148.5, 80.5)
- moved VIN2 1.80 mm to (168.2, 75.0)
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Connections:
- net /IN_A1 renamed Net-(M7-PadS25)
- net /IN_A2 renamed Net-(M7-PadS19)
- net /IN_A4 renamed Net-(M7-PadS22)
- D3 pad 2: /CRANK+ -> /IN_CRANK+
- D7 pad 2: /CRANK -> /IN_CRANK
- D8 pad 2: /CRANK- -> /IN_CRANK-
- JP16 pad 2: /CRANK+ -> /IN_CRANK+
- JP3 pad 2: /INJ5 -> /OUT_INJ5
- JP31 pad 2: /INJ3 -> /OUT_INJ3
- JP32 pad 2: /INJ2 -> /OUT_INJ2
- JP33 pad 2: /INJ1 -> /OUT_INJ1
- JP35 pad 2: /INJ8 -> /OUT_INJ8
- JP4 pad 2: /INJ6 -> /OUT_INJ6
- JP43 pad 2: /CRANK- -> /IN_CRANK-
- JP5 pad 2: /INJ4 -> /OUT_INJ4
- JP59 pad 2: /5V_SENS1 -> /5V_SENS2
- JP7 pad 2: /INJ7 -> /OUT_INJ7
- M11 pad E12: unconnected-(M11-PadE12) -> Net-(M11-PadE12)
- M11 pad E14: /COIL_A1 -> Net-(M11-PadE14)
- M11 pad E15: /COIL_A2 -> Net-(M11-PadE15)
- M11 pad E22: /CE -> Net-(M11-PadE22)
- M11 pad E28: /OUT3 -> Net-(M11-PadE28)
- M11 pad E7: /OUT1 -> Net-(M11-PadE7)
- M11 pad E9: /OUT2 -> Net-(M11-PadE9)
- M11 pad S10: Net-(M11-PadS10) -> /INK2
- M11 pad S12: /KNOCK1 -> /INK1
- M11 pad S27: Net-(M11-PadS27) -> /BARO
- M11 pad S3: /D1 -> Net-(M11-PadS3)
- M11 pad S4: /D2 -> Net-(M11-PadS4)
- M11 pad S5: /D3 -> Net-(M11-PadS5)
- M11 pad S6: /D4 -> Net-(M11-PadS6)
- M7 pad N22: /IN_KNOCK1 -> /INK1
- M7 pad N24: /IN_KNOCK2 -> /INK2
- M7 pad N7: unconnected-(M7-PadN7) -> Net-(M7-PadN7)
- M7 pad S17: unconnected-(M7-PadS17) -> Net-(M7-PadS17)
- M7 pad S18: /IN_PPS2 -> Net-(M7-PadS18)
- M7 pad S20: /IN_A3 -> Net-(M7-PadS20)
- M7 pad S21: unconnected-(M7-PadS21) -> Net-(M7-PadS21)
- M7 pad S23: /IN_RES1 -> Net-(M7-PadS23)
- M7 pad S24: /IN_PPS1 -> Net-(M7-PadS24)
- M7 pad S26: /IN_RES2 -> Net-(M7-PadS26)
- M7 pad S9: /IN_AFR -> Net-(M7-PadS9)
- M9 pad S1: /OUT_COIL_A1 -> Net-(M9-PadS1)
- M9 pad S2: /OUT_COIL_A2 -> Net-(M9-PadS2)
- M9 pad W21: /OUT3 -> Net-(M9-PadW21)
- M9 pad W25: /CE -> Net-(M9-PadW25)
- M9 pad W3: /OUT_CE -> Net-(M9-PadW3)
- M9 pad W32: /COIL_A2 -> Net-(M9-PadW32)
- M9 pad W33: /COIL_A1 -> Net-(M9-PadW33)
- M9 pad W37: /OUT2 -> Net-(M9-PadW37)
- M9 pad W39: /OUT1 -> Net-(M9-PadW39)
- MMCU16 pad 1: Net-(M11-PadS27) -> Net-(M11-PadE14)
- MMCU35 pad 1: Net-(M11-PadS10) -> Net-(M11-PadS5)
- U1 pad 4: /BARO_AV5 -> /BARO
- U2 pad 1: /MAP_AV1 -> /IN_MAP2
- VIN3 pad 1: /IN_A3 -> Net-(M7-PadS18)
Routing:
- net Net-(M11-PadS10): track 15.8 -> 0.00 mm
- net /INJ2: track 10.6 -> 0.00 mm
- net /INJ1: track 10.5 -> 0.00 mm
- net /PUMP: track 0.00 -> 9.77 mm
- net /OUT2: track 9.73 -> 0.00 mm
- net Net-(M9-PadW26): track 9.22 -> 0.00 mm
- net Net-(M9-PadW34): track 7.83 -> 0.00 mm
- net Net-(M9-PadW36): track 6.90 -> 0.00 mm
- net /MAIN_RELAY: track 6.80 -> 0.00 mm
- net /OUT1: track 6.70 -> 0.00 mm
- net /TACH: track 6.65 -> 0.00 mm
- net /OUT3: track 6.50 -> 0.00 mm
- net Net-(M9-PadW31): track 6.48 -> 0.00 mm
- net /COIL_A1: track 6.43 -> 0.00 mm
- net Net-(M9-PadW30): track 6.42 -> 0.00 mm
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
Commit message: Up issue 26.28.29
Parts:
- M1: value Module-power12-0.1 -> Module-power12-0.2; footprint power12:power12 -> hellen-one-power12-0.2:power12
- M10: footprint ign8:ign8 -> hellen-one-ign8-0.1:ign8
- M11: value Module-mcu-0.1 -> Module-mcu-0.4; footprint mcu:mcu -> hellen-one-mcu-0.4:mcu
- M12, M8: footprint knock:knock -> hellen-one-knock-0.1:knock
- M2, M4: footprint can:can -> hellen-one-can-0.1:can
- M3: value Module-wbo-0.1 -> Module-wbo-0.2; footprint wbo:wbo -> hellen-one-wbo-0.2:wbo
- M5: footprint power5:power5 -> hellen-one-power5-0.1:power5
- M6: footprint vr:vr -> hellen-one-vr-0.1:vr
- M7: footprint input:input -> hellen-one-input-0.1:input
- M9: value Module-output-0.1 -> Module-output-0.2; footprint output:output -> hellen-one-output-0.2:output
- moved VOUT8 153.8 mm to (127.0, 114.8)
- moved VOUT9 151.8 mm to (125.2, 127.2)
Connections:
- M11 pad E17: Net-(M11-PadE17) -> /IDLE
- M11 pad E18: /IDLE -> /FUEL_CONSUM
- M11 pad E19: /FUEL_CONSUM -> /TACH
- M11 pad E27: /TACH -> Net-(M11-PadE27)
- M11 pad E6: /OUT_MAIN -> /PUMP
- M11 pad E8: /PUMP -> /OUT_MAIN
- M11 pad S32: GNDA -> GND
- M3 pad W5: (no net) -> unconnected-(M3-PadW5)
- M3 pad W6: (no net) -> unconnected-(M3-PadW6)
- M3 pad W7: (no net) -> unconnected-(M3-PadW7)
- M3 pad W8: (no net) -> unconnected-(M3-PadW8)
- M9 pad S10: /OUT_PUMP -> Net-(M9-PadS10)
- M9 pad S7: /OUT_IDLE -> Net-(VOUT20-Pad1)
- M9 pad S8: Net-(M9-PadS8) -> /OUT_IDLE
- M9 pad W1: Net-(M9-PadW1) -> Net-(VOUT19-Pad1)
- M9 pad W2: Net-(M9-PadW2) -> /OUT_PUMP
- M9 pad W21: Net-(M9-PadW21) -> /IDLE
- M9 pad W26: Net-(M9-PadW26) -> /PUMP
- M9 pad W27: Net-(M9-PadW27) -> Net-(VOUT25-Pad1)
- M9 pad W29: Net-(M9-PadW29) -> Net-(VOUT10-Pad1)
- M9 pad W30: Net-(M9-PadW30) -> Net-(VOUT8-Pad1)
- M9 pad W35: /PUMP -> Net-(VOUT13-Pad1)
- M9 pad W37: Net-(M9-PadW37) -> Net-(VOUT24-Pad1)
- M9 pad W38: /IDLE -> Net-(VOUT11-Pad1)
- MMCU14 pad 1: Net-(M11-PadE16) -> Net-(M11-PadE15)
- MMCU15 pad 1: Net-(M11-PadE17) -> Net-(M11-PadE16)
- MMCU16 pad 1: Net-(M11-PadE14) -> Net-(M11-PadE27)
- MMCU18 pad 1: Net-(M11-PadE21) -> Net-(M11-PadE10)
- MMCU19 pad 1: Net-(M11-PadE10) -> Net-(M11-PadE7)
- MMCU20 pad 1: Net-(M11-PadE15) -> Net-(M11-PadE14)
- MMCU28 pad 1: Net-(M11-PadE11) -> Net-(M11-PadE9)
- MMCU29 pad 1: Net-(M11-PadE13) -> Net-(M11-PadE22)
- MMCU30 pad 1: Net-(M11-PadE20) -> Net-(M11-PadE11)
- MMCU31 pad 1: Net-(M11-PadE23) -> Net-(M11-PadE13)
- MMCU38 pad 1: Net-(M11-PadE9) -> Net-(M11-PadE23)
- MMCU39 pad 1: Net-(M11-PadE12) -> Net-(M11-PadE21)
- MMCU40 pad 1: Net-(M11-PadE22) -> Net-(M11-PadE20)
- MMCU41 pad 1: Net-(M11-PadE7) -> Net-(M11-PadE12)
- VOUT10 pad 1: Net-(M9-PadW36) -> Net-(VOUT10-Pad1)
- VOUT11 pad 1: Net-(M9-PadW29) -> Net-(VOUT11-Pad1)
- VOUT12 pad 1: Net-(M9-PadW31) -> Net-(M9-PadW36)
- VOUT13 pad 1: Net-(M9-PadW30) -> Net-(VOUT13-Pad1)
- VOUT16 pad 1: Net-(M9-PadW4) -> Net-(M9-PadS10)
- VOUT18 pad 1: Net-(M9-PadW2) -> Net-(M9-PadS13)
- VOUT19 pad 1: Net-(M9-PadS13) -> Net-(VOUT19-Pad1)
- VOUT20 pad 1: Net-(M9-PadW1) -> Net-(VOUT20-Pad1)
- VOUT24 pad 1: Net-(M9-PadW33) -> Net-(VOUT24-Pad1)
- VOUT25 pad 1: Net-(M9-PadW32) -> Net-(VOUT25-Pad1)
- VOUT26 pad 1: Net-(M9-PadW25) -> Net-(M9-PadW33)
- VOUT27 pad 1: Net-(M9-PadW39) -> Net-(M9-PadW32)
- VOUT28 pad 1: Net-(M9-PadW37) -> Net-(M9-PadW31)
- VOUT29 pad 1: Net-(M9-PadW21) -> Net-(M9-PadW25)
- VOUT3 pad 1: Net-(M9-PadS8) -> Net-(M9-PadW4)
- VOUT8 pad 1: Net-(M9-PadW27) -> Net-(VOUT8-Pad1)
- VOUT9 pad 1: Net-(M9-PadW26) -> Net-(M9-PadW39)
Routing:
- net V12_RAW: track 128.0 -> 162.3 mm
- net /PUMP: track 9.77 -> 0.00 mm
- net /OUT_MAIN: track 0.00 -> 9.77 mm
- net GNDA: track 8.82 -> 2.96 mm
- net GND: track 0.00 -> 5.86 mm
- net Net-(M9-PadW4): track 0.00 -> 4.40 mm
- net Net-(M9-PadS8): track 4.40 -> 0.00 mm
- net /OUT_INJ6: track 4.49 -> 2.26 mm
Other:
- copper layers 2 -> 4
- board text added: "1"
- board text added: "11"
- board text added: "12"
- board text added: "13"
- board text added: "14"
- board text added: "15"
- board text added: "16"
- board text added: "17"
- board text added: "18"
- board text added: "19"
- board text added: "2"
- board text added: "20"
- board text added: "21"
- board text added: "22"
- board text added: "23"
- board text added: "24"
- board text added: "25"
- board text added: "26"
- board text added: "27"
- board text added: "28"
- board text added: "29"
- board text added: "3"
- board text added: "30"
- board text added: "31"
- board text added: "32"
- board text added: "33"
- board text added: "34"
- board text added: "35"
- board text added: "36"
- board text added: "37"
- board text added: "38"
- board text added: "39"
- board text added: "4"
- board text added: "40"
- board text added: "41"
- board text added: "42"
- board text added: "43"
- board text added: "44"
- board text added: "45"
- board text added: "46"
- board text added: "47"
- board text added: "48"
- board text added: "49"
- board text added: "5"
- board text added: "50"
- board text added: "51"
- board text added: "52"
- board text added: "54"
- board text added: "55"
- board text added: "56"
- board text added: "59"
- board text added: "6"
- board text added: "60"
- board text added: "62"
- board text added: "64"
- board text added: "65"
- board text added: "66"
- board text added: "67"
- board text added: "68"
- board text added: "69"
- board text added: "7"
- board text added: "70"
- board text added: "71"
- board text added: "73"
- board text added: "77"
- board text added: "78"
- board text added: "8"
- board text added: "81"
- board text added: "82"
- board text added: "83"
- board text added: "84"
- board text added: "85"
- board text added: "86"
- board text added: "Hellen 88bmw rev A"

Commit message: Up issue 30
Parts:
- moved M1 59.3 mm to (80.3, 131.1)
Changed lines of the file:
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@@
     )
     (pad_to_mask_clearance 0)
+    (aux_axis_origin 64.074 153.523)
     (pcbplotparams
-      (layerselection 0x00010f0_ffffffff)
-      (disableapertmacros false)
-      (usegerberextensions false)
+      (layerselection 0x00010fc_ffffffff)
+      (disableapertmacros true)
+      (usegerberextensions true)
       (usegerberattributes false)
-      (usegerberadvancedattributes false)
+      (usegerberadvancedattributes true)
       (creategerberjobfile false)
       (svguseinch false)
@@
       (viasonmask false)
       (mode 1)
-      (useauxorigin false)
+      (useauxorigin true)
       (hpglpennumber 1)
       (hpglpenspeed 20)
@@
       (psa4output false)
       (plotreference true)
-      (plotvalue true)
+      (plotvalue false)
       (plotinvisibletext false)
       (sketchpadsonfab false)
@@
       (drillshape 0)
       (scaleselection 1)
-      (outputdirectory "Motronic_88pin_Gerbers/")
+      (outputdirectory "../../../gerber/")
     )
   )
@@
     (fp_line (start 3.15 1.6) (end -3.15 1.6) (layer "F.Fab") (width 0.1))
     (fp_line (start -3.15 1.6) (end -3.15 -1.6) (layer "F.Fab") (width 0.1))
-    (pad "1" smd roundrect locked (at -2.9625 0 90) (size 1.225 3.35) (layers "F.Cu" "F.Paste" "F.Mask") (roundrect_rratio 0.204082)
+    (pad "1" smd roundrect locked (at -2.9625 0 90) (size 1.225 3.35) (layers "F.Cu" "F.Paste" "F.Mask") (roundrect_rratio 0.2040816327)
       (net 153 "/COIL_7") (pintype "passive"))
-    (pad "2" smd roundrect locked (at 2.9625 0 90) (size 1.225 3.35) (layers "F.Cu" "F.Paste" "F.Mask") (roundrect_rratio 0.204082)
+    (pad "2" smd roundrect locked (at 2.9625 0 90) (size 1.225 3.35) (layers "F.Cu" "F.Paste" "F.Mask") (roundrect_rratio 0.2040816327)
       (net 405 "/OUT_IGN7") (pintype "passive"))
     (model "${KICAD6_3DMODEL_DIR}/Resistor_SMD.3dshapes/R_2512_6332Metric.wrl"
@@
     (fp_line (start -3.15 1.6) (end -3.15 -1.6) (layer "F.Fab") (width 0.1))
     (fp_line (start -3.15 -1.6) (end 3.15 -1.6) (layer "F.Fab") (width 0.1))
-    (pad "1" smd roundrect locked (at -2.9625 0 90) (size 1.225 3.35) (layers "F.Cu" "F.Paste" "F.Mask") (roundrect_rratio 0.204082)
+    (pad "1" smd roundrect locked (at -2.9625 0 90) (size 1.225 3.35) (layers "F.Cu" "F.Paste" "F.Mask") (roundrect_rratio 0.2040816327)
       (net 114 "/COIL_2") (pintype "passive"))
-    (pad "2" smd roundrect locked (at 2.9625 0 90) (size 1.225 3.35) (layers "F.Cu" "F.Paste" "F.Mask") (roundrect_rratio 0.204082)
+    (pad "2" smd roundrect locked (at 2.9625 0 90) (size 1.225 3.35) (layers "F.Cu" "F.Paste" "F.Mask") (roundrect_rratio 0.2040816327)
       (net 400 "/OUT_IGN2") (pintype "passive"))
     (model "${KICAD6_3DMODEL_DIR}/Resistor_SMD.3dshapes/R_2512_6332Metric.wrl"
@@
     (fp_line (start -3.15 1.6) (end -3.15 -1.6) (layer "F.Fab") (width 0.1))
     (fp_line (start -3.15 -1.6) (end 3.15 -1.6) (layer "F.Fab") (width 0.1))
-    (pad "1" smd roundrect locked (at -2.9625 0 270) (size 1.225 3.35) (layers "F.Cu" "F.Paste" "F.Mask") (roundrect_rratio 0.204082)
+    (pad "1" smd roundrect locked (at -2.9625 0 270) (size 1.225 3.35) (layers "F.Cu" "F.Paste" "F.Mask") (roundrect_rratio 0.2040816327)
       (net 406 "/OUT_IGN8") (pintype "passive"))
-    (pad "2" smd roundrect locked (at 2.9625 0 270) (size 1.225 3.35) (layers "F.Cu" "F.Paste" "F.Mask") (roundrect_rratio 0.204082)
+    (pad "2" smd roundrect locked (at 2.9625 0 270) (size 1.225 3.35) (layers "F.Cu" "F.Paste" "F.Mask") (roundrect_rratio 0.2040816327)
       (net 158 "/COIL_8") (pintype "passive"))
     (model "${KICAD6_3DMODEL_DIR}/Resistor_SMD.3dshapes/R_2512_6332Metric.wrl"
@@
     (fp_line (start -3.15 -1.6) (end 3.15 -1.6) (layer "F.Fab") (width 0.1))
     (fp_line (start -3.15 1.6) (end -3.15 -1.6) (layer "F.Fab") (width 0.1))
-    (pad "1" smd roundrect locked (at -2.9625 0 90) (size 1.225 3.35) (layers "F.Cu" "F.Paste" "F.Mask") (roundrect_rratio 0.204082)
+    (pad "1" smd roundrect locked (at -2.9625 0 90) (size 1.225 3.35) (layers "F.Cu" "F.Paste" "F.Mask") (roundrect_rratio 0.2040816327)
       (net 113 "/COIL_1") (pintype "passive"))
-    (pad "2" smd roundrect locked (at 2.9625 0 90) (size 1.225 3.35) (layers "F.Cu" "F.Paste" "F.Mask") (roundrect_rratio 0.204082)
+    (pad "2" smd roundrect locked (at 2.9625 0 90) (size 1.225 3.35) (layers "F.Cu" "F.Paste" "F.Mask") (roundrect_rratio 0.2040816327)
       (net 399 "/OUT_IGN1") (pintype "passive"))
     (model "${KICAD6_3DMODEL_DIR}/Resistor_SMD.3dshapes/R_2512_6332Metric.wrl"
@@
     (fp_line (start 3.15 1.6) (end -3.15 1.6) (layer "F.Fab") (width 0.1))
     (fp_line (start -3.15 1.6) (end -3.15 -1.6) (layer "F.Fab") (width 0.1))
-    (pad "1" smd roundrect locked (at -2.9625 0 270) (size 1.225 3.35) (layers "F.Cu" "F.Paste" "F.Mask") (roundrect_rratio 0.204082)
+    (pad "1" smd roundrect locked (at -2.9625 0 270) (size 1.225 3.35) (layers "F.Cu" "F.Paste" "F.Mask") (roundrect_rratio 0.2040816327)
       (net 401 "/OUT_IGN3") (pintype "passive"))
-    (pad "2" smd roundrect locked (at 2.9625 0 270) (size 1.225 3.35) (layers "F.Cu" "F.Paste" "F.Mask") (roundrect_rratio 0.204082)
+    (pad "2" smd roundrect locked (at 2.9625 0 270) (size 1.225 3.35) (layers "F.Cu" "F.Paste" "F.Mask") (roundrect_rratio 0.2040816327)
       (net 115 "/COIL_3") (pintype "passive"))
     (model "${KICAD6_3DMODEL_DIR}/Resistor_SMD.3dshapes/R_2512_6332Metric.wrl"
@@
     (fp_line (start 3.15 -1.6) (end 3.15 1.6) (layer "F.Fab") (width 0.1))
     (fp_line (start -3.15 1.6) (end -3.15 -1.6) (layer "F.Fab") (width 0.1))
-    (pad "1" smd roundrect locked (at -2.9625 0 90) (size 1.225 3.35) (layers "F.Cu" "F.Paste" "F.Mask") (roundrect_rratio 0.204082)
+    (pad "1" smd roundrect locked (at -2.9625 0 90) (size 1.225 3.35) (layers "F.Cu" "F.Paste" "F.Mask") (roundrect_rratio 0.2040816327)
       (net 102 "/COIL_4") (pintype "passive"))
-    (pad "2" smd roundrect locked (at 2.9625 0 90) (size 1.225 3.35) (layers "F.Cu" "F.Paste" "F.Mask") (roundrect_rratio 0.204082)
+    (pad "2" smd roundrect locked (at 2.9625 0 90) (size 1.225 3.35) (layers "F.Cu" "F.Paste" "F.Mask") (roundrect_rratio 0.2040816327)
       (net 402 "/OUT_IGN4") (pintype "passive"))
     (model "${KICAD6_3DMODEL_DIR}/Resistor_SMD.3dshapes/R_2512_6332Metric.wrl"
@@
     (fp_line (start -3.15 -1.6) (end 3.15 -1.6) (layer "F.Fab") (width 0.1))
     (fp_line (start 3.15 -1.6) (end 3.15 1.6) (layer "F.Fab") (width 0.1))
-    (pad "1" smd roundrect locked (at -2.9625 0 270) (size 1.225 3.35) (layers "F.Cu" "F.Paste" "F.Mask") (roundrect_rratio 0.204082)
+    (pad "1" smd roundrect locked (at -2.9625 0 270) (size 1.225 3.35) (layers "F.Cu" "F.Paste" "F.Mask") (roundrect_rratio 0.2040816327)
       (net 404 "/OUT_IGN6") (pintype "passive"))
-    (pad "2" smd roundrect locked (at 2.9625 0 270) (size 1.225 3.35) (layers "F.Cu" "F.Paste" "F.Mask") (roundrect_rratio 0.204082)
+    (pad "2" smd roundrect locked (at 2.9625 0 270) (size 1.225 3.35) (layers "F.Cu" "F.Paste" "F.Mask") (roundrect_rratio 0.2040816327)
       (net 103 "/COIL_6") (pintype "passive"))
     (model "${KICAD6_3DMODEL_DIR}/Resistor_SMD.3dshapes/R_2512_6332Metric.wrl"
@@
     (fp_line (start -3.15 1.6) (end -3.15 -1.6) (layer "F.Fab") (width 0.1))
     (fp_line (start -3.15 -1.6) (end 3.15 -1.6) (layer "F.Fab") (width 0.1))
-    (pad "1" smd roundrect locked (at -2.9625 0 270) (size 1.225 3.35) (layers "F.Cu" "F.Paste" "F.Mask") (roundrect_rratio 0.204082)
+    (pad "1" smd roundrect locked (at -2.9625 0 270) (size 1.225 3.35) (layers "F.Cu" "F.Paste" "F.Mask") (roundrect_rratio 0.2040816327)
       (net 403 "/OUT_IGN5") (pintype "passive"))
-    (pad "2" smd roundrect locked (at 2.9625 0 270) (size 1.225 3.35) (layers "F.Cu" "F.Paste" "F.Mask") (roundrect_rratio 0.204082)
+    (pad "2" smd roundrect locked (at 2.9625 0 270) (size 1.225 3.35) (layers "F.Cu" "F.Paste" "F.Mask") (roundrect_rratio 0.2040816327)
       (net 104 "/COIL_5") (pintype "passive"))
     (model "${KICAD6_3DMODEL_DIR}/Resistor_SMD.3dshapes/R_2512_6332Metric.wrl"
@@
   )
   (footprint "hellen-one-power12-0.2:power12" (layer "F.Cu")
-    (at 58.087891 186.116015 90)
+    (at 80.337891 131.116015 90)
     (property "Sheetfile" "hellen88bmw.kicad_sch")
     (property "Sheetname" "")
@@
       (polygon
         (pts
-          (xy 51.662892 185.891014)
-          (xy 51.637894 185.866015)
-          (xy 42.537892 185.866015)
-          (xy 42.537892 172.241016)
-          (xy 42.512893 172.216017)
-          (xy 42.163757 172.21605)
-          (xy 42.162109 169.878161)
-          (xy 42.46289 169.633985)
-          (xy 57.255805 169.633985)
-          (xy 57.255828 169.743134)
-          (xy 57.762834 170.141015)
-          (xy 57.762834 178.740866)
-          (xy 56.812892 179.690978)
-          (xy 51.712892 179.691014)
-          (xy 51.687891 179.716015)
+          (xy 73.912892 130.891014)
+          (xy 73.887894 130.866015)
+          (xy 64.787892 130.866015)
+          (xy 64.787892 117.241016)
+          (xy 64.762893 117.216017)
+          (xy 64.413757 117.21605)
+          (xy 64.412109 114.878161)
+          (xy 64.71289 114.633985)
+          (xy 79.505805 114.633985)
+          (xy 79.505828 114.743134)
+          (xy 80.012834 115.141015)
+          (xy 80.012834 123.740866)
+          (xy 79.062892 124.690978)
+          (xy 73.962892 124.691014)
+          (xy 73.937891 124.716015)
         )
       )
@@
   (gr_line (start 64.0738 38.5648) (end 67.0738 35.5648) (layer "Edge.Cuts") (width 0.2))
   (gr_line (start 210 53) (end 74 53) (layer "F.Fab") (width 0.1))
+  (gr_line (start 72 153.5228) (end 59 153.5228) (layer "F.Fab") (width 0.001))
+  (gr_line (start 64.0738 147) (end 64.0738 155) (layer "F.Fab") (width 0.001))
   (gr_line (start 209 103) (end 201 103) (layer "F.Fab") (width 0.1))
   (gr_line (start 227 60.5) (end 60 60.5) (layer "F.Fab") (width 0.1))
