File: boards/hellen88bmw/kicad6/hellen88bmw.kicad_pcb (KiCad board)
At the start: 4 copper layers, 160 x 118 mm, 292 parts, among them J1 920-462A2021Y10101, J10 Conn_01x12, J11 Conn_01x12, J12 Conn_01x12, J13 Conn_01x12, J14 VRIN1, J15 VRIN2, J16 VROUT1, J18 C165947, J2 UB-20PMFP-LC7002, J3 Micro_SD_Card, J4 Conn_01x05, J5 Conn_01x12, J6 Conn_01x12, J7 Conn_01x12, J8 Conn_01x12, J9 Conn_01x12, M1 Module-power12-0.2, M10 Module-ign8-0.1, M11 Module-mcu-0.4, M12 Module-knock-0.1, M2 Module-can-0.1, M3 Module-wbo-0.2, M4 Module-can-0.1, M5 Module-power5-0.1, M6 Module-vr-0.1, M7 Module-input-0.1, M8 Module-knock-0.1, M9 Module-output-0.2, P1 P, P2 P, P3 P, P4 P, P5 P, P6 P, Q1 NGD8201AN, Q2 NGD8201AN, Q3 NGD8201AN, Q4 NGD8201AN, Q5 NGD8201AN, Q6 NGD8201AN, Q7 NGD8201AN, Q8 NGD8201AN, SW1 BOOT0, SW2 RESET, U1 MPXA6115A, U2 MPX4_MAP, U3 LIS2DW12TR, U4 LPS25HB, U5 MCP6002-xSN

Commit message: Up 20/072021
Parts:
- removed MMCU15, MMCU16, MMCU20, MMCU37: MMCU, Connector_PinHeader_1.00mm:PinHeader_1x01_P1.00mm_Vertical
- removed VIN23: Pad, Connector_PinHeader_1.00mm:PinHeader_1x01_P1.00mm_Vertical
- added C10: 5.6nF, Capacitor_SMD:C_0402_1005Metric, F.Cu at (60.0, 201.0)
- added C11: 10uF, Capacitor_SMD:C_0603_1608Metric, F.Cu at (57.0, 196.8)
- added C12: 10nF, Capacitor_SMD:C_0402_1005Metric, F.Cu at (59.3, 199.0)
- added C13: 10uF, Capacitor_SMD:C_0603_1608Metric, F.Cu at (52.6, 201.8)
- added C14: 10uF, Capacitor_SMD:C_0603_1608Metric, F.Cu at (53.0, 196.6)
- added C15: 220nF, Capacitor_SMD:C_0402_1005Metric, F.Cu at (62.2, 198.8)
- added C16: 10uF, Capacitor_SMD:C_0603_1608Metric, F.Cu at (61.0, 196.6)
- added C17: 10uF, Capacitor_SMD:C_0603_1608Metric, F.Cu at (77.3, 191.7)
- added C18: 100nF, Capacitor_SMD:C_0402_1005Metric, F.Cu at (64.5, 196.3)
- added C19: 10uF, Capacitor_SMD:C_0603_1608Metric, F.Cu at (56.6, 201.6)
- added C20: 100nF, Capacitor_SMD:C_0402_1005Metric, F.Cu at (54.9, 204.0)
- added C21: 10uF, Capacitor_SMD:C_0603_1608Metric, F.Cu at (82.0, 179.4)
- added C9: 10uF, Capacitor_SMD:C_0603_1608Metric, F.Cu at (53.0, 199.1)
- added D32: 1N4148WS, Diode_SMD:D_SOD-323, F.Cu at (48.5, 202.0)
- added D33: 1N4148WS, Diode_SMD:D_SOD-323, F.Cu at (41.0, 202.9)
- added J17: XH-8A, Connector_PinHeader_2.54mm:PinHeader_1x08_P2.54mm_Vertical, F.Cu at (100.9, 151.8)
- added J19: MiniFit, Connector_Molex:Molex_Mini-Fit_Jr_5569-02A2_2x01_P4.20mm_Horizontal, F.Cu at (78.2, 143.0)
- added J20: ETB_6p, Connector_PinHeader_2.54mm:PinHeader_1x06_P2.54mm_Vertical, F.Cu at (66.0, 127.9)
- added J21: ETB_4p, Connector_PinHeader_2.54mm:PinHeader_1x04_P2.54mm_Vertical, F.Cu at (71.8, 133.2)
- added R28: 100k, Resistor_SMD:R_0402_1005Metric, F.Cu at (44.6, 202.4)
- added R29: 10k, Resistor_SMD:R_0402_1005Metric, F.Cu at (56.5, 199.0)
- added R30: 100R, Resistor_SMD:R_0402_1005Metric, F.Cu at (52.0, 204.1)
- added U6: L6205PD, kicad6:SO20POWER, F.Cu at (60.8, 186.7)
- C1, C2, C3, C4, C5, C6: footprint Capacitor_SMD:C_0603_1608Metric -> Capacitor_SMD:C_0402_1005Metric
- C7, C8: footprint Capacitor_SMD:C_0402_1005Metric -> Capacitor_SMD:C_0603_1608Metric
- J3: moved to F.Cu
- R1, R2, R25, R26, R27, R3, R4, R5: footprint Resistor_SMD:R_0603_1608Metric -> Resistor_SMD:R_0402_1005Metric
- R6: footprint Resistor_SMD:R_0603_1608Metric -> Resistor_SMD:R_0402_1005Metric; moved to B.Cu
- U3: footprint Package_LGA:Kionix_LGA-12_2x2mm_P0.5mm_LayoutBorder2x4y -> kicad6:LGA12R50P4X4_200X200X70
- moved D18 230.9 mm to (192.7, 28.6)
- moved D19 230.9 mm to (192.4, 24.6)
- moved D22 230.9 mm to (195.9, 26.6)
- moved D23 230.9 mm to (195.9, 22.9)
- moved RN6 230.9 mm to (187.4, 26.9)
- moved VOUT4 207.5 mm to (124.5, 74.0)
- moved VOUT6 201.2 mm to (126.8, 75.0)
- moved VOUT1 197.2 mm to (124.5, 76.0)
- moved VOUT14 195.1 mm to (97.8, 66.8)
- moved VIN24 193.3 mm to (168.8, 70.8)
- moved VIN22 193.3 mm to (172.2, 89.5)
- moved VIN19 192.7 mm to (172.0, 68.8)
- moved VIN25 191.2 mm to (169.8, 68.8)
- moved VOUT15 187.6 mm to (100.0, 66.8)
- moved VIN20 187.4 mm to (175.5, 70.8)
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Connections:
- M11 pad E14: Net-(M11-PadE14) -> /+ETB
- M11 pad E15: Net-(M11-PadE15) -> /-ETB
- M11 pad E27: Net-(M11-PadE27) -> /ETB_EN
- M11 pad S6: Net-(MMCU37-Pad1) -> /V12_PERM
- MMCU14 pad 1: Net-(M11-PadE15) -> Net-(M11-PadE16)
Routing:
- net /USBM: track 26.3 -> 154.8 mm
- net /USBP: track 21.3 -> 146.5 mm
- net /IN_KNOCK2_RAW: track 8.85 -> 127.5 mm, vias 0 -> 1
- net /IN_KNOCK1_RAW: track 8.95 -> 122.7 mm, vias 0 -> 1
- net GNDA: track 2.96 -> 101.2 mm, vias 0 -> 1
- net /GND_SENS: track 7.56 -> 93.3 mm
- net +5V: track 17.2 -> 96.5 mm
- net V12_RAW: track 162.3 -> 230.5 mm
- net /IN_CRANK-: track 0.00 -> 58.2 mm
- net /OUT_INJ5: track 0.00 -> 52.7 mm, vias 0 -> 1
- net /OUT_TACH: track 0.00 -> 41.6 mm
- net /IAT: track 5.86 -> 42.6 mm
- net /OUT_INJ3: track 0.00 -> 33.8 mm
- net /OUT_INJ7: track 0.00 -> 33.3 mm, vias 0 -> 1
- net /IN_CRANK+: track 0.00 -> 30.6 mm
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
Commit message: Up 21/072021
Parts:
- C1, C2, U1: moved to F.Cu
- C10, C11, C12, C13, C14, C15, C16, C17, C18, C19, C20, C21, C9, D32, D33, R28, R29, R30, U6: moved to B.Cu
- J17: footprint Connector_PinHeader_2.54mm:PinHeader_1x08_P2.54mm_Vertical -> kicad6:XH-8A
- P1, P2, P3, P4, P5, P6: footprint Connector_PinHeader_1.00mm:PinHeader_1x01_P1.00mm_Vertical -> Connector_Pin:Pin_D1.0mm_L10.0mm
- moved D24 237.9 mm to (185.0, 5.50)
- moved D25 237.9 mm to (185.2, 2.50)
- moved D26 237.9 mm to (182.8, 24.9)
- moved D27 237.9 mm to (182.5, 21.9)
- moved D28 237.9 mm to (189.0, 4.00)
- moved D29 237.9 mm to (189.0, 1.00)
- moved D30 237.9 mm to (186.7, 23.4)
- moved D31 237.9 mm to (186.5, 20.7)
- moved D4 237.9 mm to (192.8, 11.5)
- moved D5 237.9 mm to (185.0, 14.5)
- moved D6 237.9 mm to (192.2, 14.5)
- moved R3 237.9 mm to (184.5, 11.2)
- moved RN2 237.9 mm to (180.0, 12.5)
- moved RN7 237.9 mm to (180.4, 3.95)
- moved RN8 237.9 mm to (179.0, 23.4)
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Connections:
- C11 pad 1: +12V_RAW -> V12_RAW
- C13 pad 1: +12V_RAW -> V12_RAW
- C14 pad 1: +12V_RAW -> V12_RAW
- C15 pad 1: +12V_RAW -> V12_RAW
- C16 pad 1: +12V_RAW -> V12_RAW
- C17 pad 1: +12V_RAW -> V12_RAW
- C18 pad 1: +12V_RAW -> V12_RAW
- C19 pad 1: +12V_RAW -> V12_RAW
- C20 pad 1: +12V_RAW -> V12_RAW
- C21 pad 1: +12V_RAW -> V12_RAW
- C9 pad 1: +12V_RAW -> V12_RAW
- D16 pad 2: /COIL_1 -> /COIL_5
- D17 pad 2: /COIL_3 -> /COIL_6
- D18 pad 2: /COIL_5 -> /COIL_4
- D20 pad 2: /COIL_2 -> /COIL_3
- D21 pad 2: /COIL_4 -> /COIL_2
- D22 pad 2: /COIL_6 -> /COIL_1
- D32 pad 2: +12V_RAW -> V12_RAW
- U6 pad 19: +12V_RAW -> V12_RAW
- U6 pad 2: +12V_RAW -> V12_RAW
Routing:
- net Net-(J20-Pad4): track 9.20 -> 190.3 mm
- net +12V: track 0.00 -> 139.7 mm, vias 0 -> 1
- net /IN_TPS: track 27.3 -> 161.2 mm
- net /BARO: track 0.93 -> 127.3 mm, vias 1 -> 2
- net /V12_PERM: track 0.00 -> 121.4 mm, vias 0 -> 1
- net /VIGN: track 0.00 -> 120.7 mm, vias 0 -> 1
- net /VBAT: track 0.00 -> 99.4 mm, vias 0 -> 2
- net /+ETB: track 0.00 -> 76.1 mm, vias 0 -> 2
- net /-ETB: track 0.00 -> 74.8 mm, vias 0 -> 2
- net V12_RAW: track 230.5 -> 301.4 mm
- net /CLT: track 25.3 -> 87.9 mm, vias 0 -> 2
- net /IAT: track 42.6 -> 101.3 mm, vias 0 -> 2
- net /OUT_MAIN: track 0.16 -> 51.4 mm, vias 0 -> 2
- net Net-(M9-PadW33): track 0.00 -> 50.5 mm
- net /ETB_EN: track 0.00 -> 49.6 mm, vias 0 -> 2
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