File: boards/hellen88bmw/kicad6/hellen88bmw.kicad_sch (KiCad schematic)
At the start: 259 parts, among them J1 920-462A2021Y10101, J10 Conn_01x12, J11 Conn_01x12, J12 Conn_01x12, J13 Conn_01x12, J14 VRIN1, J15 VRIN2, J16 VROUT1, J17 SD, J2 UB-20PMFP-LC7002, J3 Micro_SD_Card, J4 Conn_01x05, J5 Conn_01x12, J6 Conn_01x12, J7 Conn_01x12, J8 Conn_01x12, J9 Conn_01x12, M1 Module-power12-0.1, M10 Module-ign8-0.1, M11 Module-mcu-0.1, M2 Module-can-0.1, M3 Module-wbo-0.1, M4 Module-can-0.1, M5 Module-power5-0.1, M6 Module-vr-0.1, M7 Module-input-0.1, M8 Module-knock-0.1, M9 Module-output-0.1, Q1 NGD8201AN, Q2 NGD8201AN, Q3 NGD8201AN, Q4 NGD8201AN, Q5 NGD8201AN, Q6 NGD8201AN, Q7 NGD8201AN, Q8 NGD8201AN, SW1 BOOT0, SW2 RESET, U1 MPXA6115A, U2 MPX4_MAP

Commit message: Up 88
Parts:
- removed MMCU14, MMCU15, MMCU16, MMCU17, MMCU22, MMCU23: MMCU, Connector_PinHeader_1.00mm:PinHeader_1x01_P1.00mm_Vertical, symbol Connector_Generic:Conn_01x01
- removed OUT_IGN1: OUT_IGN1, Connector_PinHeader_1.00mm:PinHeader_1x01_P1.00mm_Vertical, symbol Connector_Generic:Conn_01x01
- removed OUT_IGN2: OUT_IGN2, Connector_PinHeader_1.00mm:PinHeader_1x01_P1.00mm_Vertical, symbol Connector_Generic:Conn_01x01
- removed OUT_IGN3: OUT_IGN3, Connector_PinHeader_1.00mm:PinHeader_1x01_P1.00mm_Vertical, symbol Connector_Generic:Conn_01x01
- removed OUT_IGN4: OUT_IGN4, Connector_PinHeader_1.00mm:PinHeader_1x01_P1.00mm_Vertical, symbol Connector_Generic:Conn_01x01
- removed OUT_IGN5: OUT_IGN5, Connector_PinHeader_1.00mm:PinHeader_1x01_P1.00mm_Vertical, symbol Connector_Generic:Conn_01x01
- removed OUT_IGN6: OUT_IGN6, Connector_PinHeader_1.00mm:PinHeader_1x01_P1.00mm_Vertical, symbol Connector_Generic:Conn_01x01
- removed OUT_IGN7: OUT_IGN7, Connector_PinHeader_1.00mm:PinHeader_1x01_P1.00mm_Vertical, symbol Connector_Generic:Conn_01x01
- removed OUT_IGN8: OUT_IGN8, Connector_PinHeader_1.00mm:PinHeader_1x01_P1.00mm_Vertical, symbol Connector_Generic:Conn_01x01
- added C4, C5, C6: 100nF, Capacitor_SMD:C_0603_1608Metric, symbol Device:C
- added C7: 10uF, Capacitor_SMD:C_0402_1005Metric, symbol Device:C
- added J18: C165947, Connector_Audio:Jack_3.5mm_CUI_SJ1-3535NG_Horizontal, symbol Connector:AudioJack3_Switch
- added R10, R11, R12, R13, R14, R7, R8, R9: DNP, Resistor_SMD:R_2512_6332Metric, symbol Device:R
- added R15, R16: 4k7, Resistor_SMD:R_0402_1005Metric, symbol Device:R
- added U3: LIS2DW12TR, Package_LGA:Kionix_LGA-12_2x2mm_P0.5mm_LayoutBorder2x4y, symbol LIS2DW12TR:LIS2DW12TR
- added U4: LPS25HB, Package_LGA:ST_HLGA-10_2.5x2.5mm_P0.6mm_LayoutBorder3x2y, symbol Sensor_Pressure:LPS25HB
- added U5: MCP6002-xSN, Package_SO:SOIC-8_3.9x4.9mm_P1.27mm, symbol Amplifier_Operational:MCP6002-xSN
Connections:
- net GP5 is gone; now on net OUT_IGN5: Q6.1 (G)
- net GP6 is gone; now on net OUT_IGN6: Q5.1 (G)
- net IGN_1 is gone; now on net OUT_IGN1: Q1.1 (G)
- net IGN_2 is gone; now on net OUT_IGN2: Q2.1 (G)
- net IGN_3 is gone; now on net OUT_IGN3: Q3.1 (G)
- net IGN_4 is gone; now on net OUT_IGN4: Q4.1 (G)
- net IGN_7 is gone; now on net OUT_IGN7: Q7.1 (G)
- net IGN_8 is gone; now on net OUT_IGN8: Q8.1 (G)
- net +3V3: now also C4.1, C5.1, R15.1, R16.1, U3.10 (VDD_IO), U3.9 (VDD), U4.1 (VDDio), U4.10 (VDD), U4.6 (~CS)
- net +5V: now also C6.1, U5.8 (V+)
- net COIL_1: now also R7.1
- net COIL_2: now also R8.1
- net COIL_3: now also R9.1
- net COIL_4: now also R13.2
- net COIL_5: now also R12.2
- net COIL_6: now also R11.2
- net COIL_7: now also R10.1
- net COIL_8: now also R14.2
- net GND: now also C4.2, C5.2, C6.2, J18.S, U3.6 (GND), U3.7 (RES), U3.8 (GND), U4.3 (GND), U4.5 (SA0/MISO), U4.8 (GND), U4.9 (GND), U5.4 (V-), U5.5 (+)
- net IN_KNOCK1: now also U5.3 (+)
- net OUT_IGN1: now also R7.2
- net OUT_IGN2: now also R8.2
- net OUT_IGN3: now also R9.2
- net OUT_IGN4: now also R13.1
- net OUT_IGN5: now also R11.1
- net OUT_IGN6: now also R12.1
- net OUT_IGN7: now also R10.2
- net OUT_IGN8: now also R14.1
- net SPI_MISO: now reaches M11.N21 (SPI2_MISO)
- net SPI_MISO: now also U3.3 (SDO/SDA0)
- net LPS_SCL: now reaches M11.N19 (I2C_SCL)
- net LPS_SCL: now also R16.2, U4.2 (SCL/SCLK)
- net SPI_CS: now reaches M11.N23 (SPI2_CS)
- net SPI_CS: now also U3.2 (CS)
- net LPS_SDA: now reaches M11.N18 (I2C_SDA)
- net LPS_SDA: now also R15.2, U4.4 (SDA/MOSI)
- net SPI_SCK: now reaches M11.N20 (SPI2_SCK)
- net SPI_SCK: now also U3.1 (SCL/SPC)
- net SPI_MOSI: now reaches M11.N22 (SPI2_MOSI)
- net SPI_MOSI: now also U3.4 (SDA/SDI/SDO)
- net IN_KNOCK1_RAW renamed IN_KNOCK_RAW
- net KNOCK_1_3: no longer names the net of JP70.2 (B)
- net KNOCK_4_5: no longer names the net of JP69.2 (B)
- new net: C7.2, J18.T
- new net: C7.1, U5.1, U5.2 (-)
- new net: U5.6 (-), U5.7
- no-connect marks 150 -> 157
Other:
- moved on the sheet: *ref1A, *ref1B, *ref1C, C1, C2, C3, D1, D10, D11, D12, D13, D14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

Commit message: Up 88
Parts:
- removed J17: SD, Connector_PinHeader_2.54mm:PinHeader_1x06_P2.54mm_Vertical, symbol Connector_Generic:Conn_01x06
- removed JP10, JP11, JP12, JP15, JP19, JP28, JP30, JP34, JP36, JP37, JP38, JP39, JP40, JP45, JP53, JP55, JP57, JP58, JP6, JP60, JP61, JP62, JP63, JP66, JP67, JP68, JP69, JP70, JP71, JP72, JP74, JP75, JP76, JP79, JP80, JP82, JP83, JP84, JP87, JP88, JP9: Jumper_2_Open, rusefi_lib_private:SM0805_jumper, symbol Jumper:Jumper_2_Open
- removed MMCU18, MMCU19, MMCU20, MMCU21: MMCU, Connector_PinHeader_1.00mm:PinHeader_1x01_P1.00mm_Vertical, symbol Connector_Generic:Conn_01x01
- added R17, R18, R19, R20, R21, R22, R23, R24: 0, Resistor_SMD:R_0402_1005Metric, symbol Device:R
Connections:
- net PB9 is gone; now on net SD_CS: J3.2 (DAT3/CD)
- net PC10 is gone; now on net SD_CLK: J3.5 (CLK)
- net PC11 is gone; now on net SD_MISO: J3.7 (DAT0)
- net PC12 is gone; now on net SD_MOSI: J3.3 (CMD)
- net USBD+ is gone; now on net USBP: JP20.2 (B)
- net USBD- is gone; now on net USBM: JP21.2 (B)
- net GND: now also *ref1.15, *ref1.28, *ref1.34, *ref1.39, *ref1.40, *ref1.45, *ref1.6, *ref1.84
- net OUT_IGN1: now also R17.1; no longer Q1.1 (G)
- net OUT_IGN2: now also R18.1; no longer Q2.1 (G)
- net OUT_IGN3: now also R19.1; no longer Q3.1 (G)
- net OUT_IGN4: now also R23.2; no longer Q4.1 (G)
- net OUT_IGN5: now also R21.2; no longer Q6.1 (G)
- net OUT_IGN6: now also R22.2; no longer Q5.1 (G)
- net OUT_IGN7: now also R20.1; no longer Q7.1 (G)
- net OUT_IGN8: now also R24.2; no longer Q8.1 (G)
- net SD_MOSI: now reaches M11.N11 (SPI3_MOSI)
- net SD_MISO: now reaches M11.N10 (SPI3_MISO)
- net SD_CS: now reaches M11.N8 (SPI3_CS)
- net SD_CLK: now reaches M11.N9 (SPI3_SCK)
- new net: Q6.1 (G), R21.1
- new net: Q5.1 (G), R22.1
- new net: Q4.1 (G), R23.1
- new net: Q1.1 (G), R17.2
- new net: Q2.1 (G), R18.2
- new net: Q3.1 (G), R19.2
- new net: Q7.1 (G), R20.2
- new net: Q8.1 (G), R24.1
- no-connect marks 157 -> 127
Other:
- note removed: "CLK"
- note removed: "CS"
- note removed: "MISO"
- note removed: "MOSI"
- moved on the sheet: R10, R11, R12, R13, R14, R7, R8, R9

Commit message: Up hellen88bmw
Parts:
- removed JP13, JP18, JP2, JP64, JP65, JP8, JP81: Jumper_2_Open, rusefi_lib_private:SM0805_jumper, symbol Jumper:Jumper_2_Open
- added C8: 10uF, Capacitor_SMD:C_0402_1005Metric, symbol Device:C
- added KNOCK_RAW2: IN_KNOCK2_RAW, Connector_PinHeader_1.00mm:PinHeader_1x01_P1.00mm_Vertical, symbol Connector_Generic:Conn_01x01
- added M12: Module-knock-0.1, knock:knock, symbol hellen-one-knock-0.1:Module-knock-0.1
- added R25, R26: 2k7, Resistor_SMD:R_0603_1608Metric, symbol Device:R
- added R27: DNP, Resistor_SMD:R_0603_1608Metric, symbol Device:R
- added cr1, cr10, cr11, cr12, cr13, cr14, cr15, cr16, cr17, cr18, cr19, cr2, cr20, cr21, cr22, cr23, cr3, cr4, cr5, cr6, cr7, cr8, cr9: cr, Connector_PinHeader_1.00mm:PinHeader_1x01_P1.00mm_Vertical, symbol Connector_Generic:Conn_01x01
- JP1, JP14, JP16, JP17, JP20, JP21, JP22, JP23, JP24, JP25, JP26, JP27, JP29, JP3, JP31, JP32, JP33, JP35, JP4, JP41, JP42, JP43, JP44, JP46, JP47, JP48, JP49, JP5, JP50, JP51, JP52, JP54, JP56, JP59, JP7, JP73, JP77, JP78, JP85, JP86: footprint rusefi_lib_private:SM0805_jumper -> rusefi_lib:SM0805_jumper
- M1: footprint rusefi_lib_private:MOD_HELLEN_POWER_12 -> power12:power12
- M10: footprint rusefi_lib_private:MOD_HELLEN_IGN8 -> ign8:ign8
- M11: footprint rusefi_lib_private:MOD_HELLEN_MCU -> mcu:mcu
- M2, M4: footprint rusefi_lib_private:MOD_HELLEN_CAN -> can:can
- M3: footprint rusefi_lib_private:MOD_HELLEN_WBO -> wbo:wbo
- M5: footprint rusefi_lib_private:MOD_HELLEN_POWER_5 -> power5:power5
- M6: footprint rusefi_lib_private:MOD_HELLEN_VR -> vr:vr
- M7: footprint rusefi_lib_private:MOD_HELLEN_INPUT -> input:input
- M8: footprint rusefi_lib_private:MOD_HELLEN_KNOCK -> knock:knock
- M9: footprint rusefi_lib_private:MOD_HELLEN_OUTPUT -> output:output
- U2: footprint rusefi_lib_private:MPX-4_MAP -> rusefi_lib:MPX-4_MAP
Connections:
- net 12V_KEY is gone; now on net V12_RAW: JP26.2 (B), JP56.2 (B)
- net 12_MAIN_RELAY is gone; now on net V12_RAW: D12.2 (A), J4.5 (Pin_5), JP54.2 (B)
- net CAM1 is gone; now on net CAM: M11.S15 (IN_CAM), M7.N19 (CAM)
- net CLT_AT1 is gone; now on net CLT: JP78.2 (B)
- net IAT_AT2 is gone; now on net IAT: JP77.2 (B)
- net IN_CLT is gone; now on net CLT: M7.S15 (IN_CLT)
- net IN_IAT is gone; now on net IAT: M7.S16 (IN_IAT)
- net IN_KNOCK_RAW is gone; now on net IN_KNOCK1_RAW: KNOCK_RAW1.1 (Pin_1), M8.W1 (IN_KNOCK)
- net KNOCK2 is gone; now on net IN_KNOCK2: M7.N24 (SENS3)
- net TPS_AV2 is gone; now on net IN_TPS: JP73.2 (B)
- net +5V: now also R25.1, R26.1
- net CAM: no longer JP17.2 (B)
- net CLT: now also R25.2
- net GND: now also *ref1.55, *ref1.71, M12.E2 (GND), R27.2; no longer U5.5 (+)
- net GND_SENS: now also R27.1
- net IAT: now also R26.2
- net INJ7: now also JP7.2 (B); no longer JP35.2 (B)
- net INJ8: now also JP35.2 (B); no longer JP7.2 (B)
- net IN_KNOCK1: now also M7.N22 (KNOCK)
- net IN_KNOCK2: now also U5.5 (+), M12.E3 (OUT_KNOCK)
- net KNOCK1: no longer M7.N22 (KNOCK)
- net MAIN_RELAY: now also M9.W40 (LOW3_MAIN)
- net OUT_MAIN: now also M11.E6 (OUT_IO1)
- net TPS2: no longer M11.S24 (IN_AUX1)
- net V5A: now also M12.E1 (V5A)
- net VREF2: now also M12.W2 (VREF)
- net at *ref1.11: now also cr1.1 (Pin_1)
- net at *ref1.12: now also cr2.1 (Pin_1)
- net at *ref1.13: now also cr3.1 (Pin_1)
- net at *ref1.18: now also cr6.1 (Pin_1)
- net at *ref1.19: now also cr7.1 (Pin_1)
- net at *ref1.2: now also cr4.1 (Pin_1)
- net at *ref1.8: now also cr5.1 (Pin_1)
- net at *ref1.64: now also cr14.1 (Pin_1)
- net at *ref1.65: now also cr15.1 (Pin_1)
- net at *ref1.81: now also cr19.1 (Pin_1)
- net at *ref1.60: now also cr12.1 (Pin_1)
- net at *ref1.62: now also cr13.1 (Pin_1)
- net at *ref1.66: now also cr16.1 (Pin_1)
- net at *ref1.67: now also cr17.1 (Pin_1)
- net at *ref1.68: now also cr18.1 (Pin_1)
- net IN_KNOCK1_RAW: now reaches *ref1.69
- net IN_KNOCK2_RAW: now reaches *ref1.70
- net IN_KNOCK2_RAW: now also KNOCK_RAW2.1 (Pin_1), M12.W1 (IN_KNOCK)
- net at *ref1.82: now also cr20.1 (Pin_1)
- net at *ref1.83: now also cr21.1 (Pin_1)
- net at *ref1.87: now also cr22.1 (Pin_1)
- net at *ref1.88: now also cr23.1 (Pin_1)
- net at *ref1.30: now also cr8.1 (Pin_1)
- net at *ref1.36: now also cr9.1 (Pin_1)
- net at *ref1.37: now also cr10.1 (Pin_1)
- net at *ref1.38: now also cr11.1 (Pin_1)
- net at J18.R: now also C8.2
- net at U5.6 (-), U5.7: now also C8.1
- net CAM2: no longer names the net of M11.S27 (IN_AUX4)
- net CAM2: no longer M7.N7 (AUX4)
- net FUEL_RELAY_GP1 renamed FUEL_RELAY
- net IN_CAM1 renamed IN_CAM
- net IN_CAM: now also JP17.2 (B)
- net IN_CAM2: no longer names the net of M7.S21 (IN_AUX4)
- net IN_TPS1 renamed IN_TPS
- net IN_TPS2: no longer names the net of M7.S17 (IN_AUX1)
- removed net MAIN: M11.E6 (OUT_IO1), M9.W40 (LOW3_MAIN)
- net TPS1 renamed TPS
- no-connect marks 127 -> 139
Other:
- note added: "1 | Low side | Fuel pump 2 | Low side | ICV close 3 | Low side | Inj 5 4 | Low side | Inj 6 5 | Low side | Inj 4 6 | GND | gnd injectors 7 | Low side| VVT Solenoid | Inj7 8 | Low side | CEL 9 | Spare | 10 | Spare | 11 | NC | Trans TPS out 12 | Analogue in | 13 | Analogue in | Lambda signal 14 | GND | MAF gnd 15 | GND | gnd (Resistor?) 16 | CPS | CPS + 17 | Digi in | Cam sensor signal 18 | Jumper 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"
- note removed: "1 | Low side | Fuel pump 2 | Low side | ICV close 3 | Low side | Inj 5 4 | Low side | inj 6 5 | Low side | inj 4 6 | GND | gnd injectors 7 | Low side | VVT Solenoid 8 | Low side | CEL 9 | Spare | 10 | Spare | 11 | NC | Trans TPS out 12 | Analogue in | 13 | Analogue in | Lambda signal 14 | GND | MAF gnd 15 | GND | gnd (Resistor?) 16 | CPS | CPS + 17 | Digi in | Cam sensor signal 18 | Jumper low si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"
- moved on the sheet: C6, C7, J18, KNOCK_RAW1, M1, M5, M8, U5A, U5B, U5C

Commit message: Up hellen88bmw
Parts:
- removed JP48: Jumper_2_Open, rusefi_lib:SM0805_jumper, symbol Jumper:Jumper_2_Open
- added MMCU14, MMCU15, MMCU16, MMCU17, MMCU18, MMCU19: MMCU, Connector_PinHeader_1.00mm:PinHeader_1x01_P1.00mm_Vertical, symbol Connector_Generic:Conn_01x01
- added VOUT10, VOUT11, VOUT12, VOUT13, VOUT16, VOUT17, VOUT18, VOUT19, VOUT20, VOUT7, VOUT8, VOUT9: Pad, Connector_PinHeader_1.00mm:PinHeader_1x01_P1.00mm_Vertical, symbol hellen-one-common:Pad
- added VOUT14, VOUT15: VOUT4, Connector_PinHeader_1.00mm:PinHeader_1x01_P1.00mm_Vertical, symbol Connector_Generic:Conn_01x01
- added cr24: cr, Connector_PinHeader_1.00mm:PinHeader_1x01_P1.00mm_Vertical, symbol Connector_Generic:Conn_01x01
Connections:
- net ECON is gone; now on net OUT_FUEL_CONSUM: JP46.2 (B)
- net FUEL_RELAY is gone; now on net OUT_PUMP: D15.2 (A), JP1.2 (B)
- net IDLE_LS2 is gone; now on net OUT_IDLE: D14.2 (A), JP29.2 (B)
- net MAF_AV4 is gone; now on net IN_MAF: JP41.2 (B), R4.2
- net TACH_GP4 is gone; now on net OUT_TACH: JP47.2 (B)
- net VSS_AV3 is gone; now on net IN_VSS: JP42.2 (B)
- net WASTEGATE: no longer M11.E12 (OUT_IO7), M9.W34 (LOW2_DUAL)
- net at *ref1.48: now also cr24.1 (Pin_1)
- net at M11.S24 (IN_AUX1): now also MMCU17.1 (Pin_1)
- net at M11.S27 (IN_AUX4): now also MMCU16.1 (Pin_1)
- net OUT_VVT1_1: no longer names the net of M9.S13 (OUT_LOW11)
- net OUT_VVT1_1: now also VOUT19.1 (Pin_1); no longer M9.S14 (OUT_LOW7)
- net OUT_VVT1_2: no longer names the net of M9.W2 (OUT_LOW9)
- net OUT_VVT1_2: now also VOUT18.1 (Pin_1); no longer M9.W1 (OUT_LOW12)
- net OUT_VVT2_B1: no longer names the net of M9.S4 (OUT_SOLENOID_B1)
- net OUT_VVT2_B1: now also VOUT14.1 (Pin_1)
- net OUT_VVT2_B2: no longer names the net of M9.S5 (OUT_SOLENOID_B2)
- net OUT_VVT2_B2: now also VOUT15.1 (Pin_1)
- net OUT_WASTEGATE: no longer names the net of M9.W4 (OUT_LOW2_DUAL)
- net OUT_WASTEGATE: now also VOUT16.1 (Pin_1)
- removed net VVT1_1: M11.E10 (OUT_IO5), M9.W27 (LOW7), M9.W36 (LOW11)
- removed net VVT1_2: M11.E21 (OUT_IO10), M9.W26 (LOW9), M9.W29 (LOW12)
- net VVT2_B1: no longer names the net of M11.E16 (OUT_PWM3)
- net VVT2_B1: now also MMCU14.1 (Pin_1); no longer M9.W31 (SOLENOID_B1)
- net VVT2_B2: no longer names the net of M9.W30 (SOLENOID_B2)
- net VVT2_B2: now also VOUT13.1 (Pin_1); no longer M11.E17 (OUT_PWM4)
- new net: M11.E17 (OUT_PWM4), MMCU15.1 (Pin_1)
- new net: M9.W29 (LOW12), VOUT11.1 (Pin_1)
- new net: M9.W34 (LOW2_DUAL), VOUT7.1 (Pin_1)
- new net: M11.E10 (OUT_IO5), MMCU19.1 (Pin_1)
- new net: M11.E21 (OUT_IO10), MMCU18.1 (Pin_1)
- new net: M9.W36 (LOW11), VOUT10.1 (Pin_1)
- new net: M9.W1 (OUT_LOW12), VOUT20.1 (Pin_1)
- new net: M9.S14 (OUT_LOW7), VOUT17.1 (Pin_1)
- new net: M9.W26 (LOW9), VOUT9.1 (Pin_1)
- new net: M9.W27 (LOW7), VOUT8.1 (Pin_1)
- new net: M9.W31 (SOLENOID_B1), VOUT12.1 (Pin_1)
Other:
- moved on the sheet: *ref1A, *ref1B, *ref1C, C1, C2, C3, C4, C5, D1, D10, D11, D12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

Commit message: Up hellen88bmw 5.07.2021
Connections:
- net 3.3V is gone; now on net +3V3: J3.4 (VDD), J4.3 (Pin_3)
- net COIL_2: now also Q3.2 (C), R9.1; no longer Q2.2 (C), R8.1
- net COIL_3: now also Q5.2 (C), R12.2; no longer Q3.2 (C), R9.1
- net COIL_4: now also Q2.2 (C), R8.1; no longer Q4.2 (C), R13.2
- net COIL_5: now also Q6.2 (C), R11.2; no longer Q5.2 (C), R12.2
- net COIL_6: now also Q4.2 (C), R13.2; no longer Q6.2 (C), R11.2
- net OUT_IGN2: now also R19.1, R9.2; no longer R18.1, R8.2
- net OUT_IGN3: now also R12.1, R22.2; no longer R19.1, R9.2
- net OUT_IGN4: now also R18.1, R8.2; no longer R13.1, R23.2
- net OUT_IGN6: now also R13.1, R23.2; no longer R12.1, R22.2
Changed lines of the file:
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@@
     (stroke (width 0) (type solid) (color 0 0 0 0))
   )
-  (wire (pts (xy 106.68 549.91) (xy 107.95 549.91))
+  (wire (pts (xy 106.68 549.91) (xy 120.65 549.91))
     (stroke (width 0) (type solid) (color 0 0 0 0))
   )
@@
     (stroke (width 0) (type solid) (color 0 0 0 0))
   )
+  (wire (pts (xy 120.65 549.91) (xy 120.65 546.1))
+    (stroke (width 0) (type solid) (color 0 0 0 0))
+  )
   (wire (pts (xy 176.53 39.37) (xy 177.8 39.37))
     (stroke (width 0) (type solid) (color 0 0 0 0))
@@
     (stroke (width 0) (type solid) (color 0 0 0 0))
   )
-  (wire (pts (xy 353.06 330.2) (xy 355.6 330.2))
+  (wire (pts (xy 353.06 330.2) (xy 367.03 330.2))
     (stroke (width 0) (type solid) (color 0 0 0 0))
   )
@@
     (stroke (width 0) (type solid) (color 0 0 0 0))
   )
+  (wire (pts (xy 367.03 330.2) (xy 367.03 327.66))
+    (stroke (width 0) (type solid) (color 0 0 0 0))
+  )
   (wire (pts (xy 391.16 328.93) (xy 394.97 328.93))
     (stroke (width 0) (type solid) (color 0 0 0 0))
@@
     (effects (font (size 1.27 1.27)) (justify left bottom))
   )
-  (label "3.3V" (at 107.95 549.91 0)
-    (effects (font (size 1.27 1.27)) (justify left bottom))
-  )
   (label "GND_SENS" (at 107.95 554.99 0)
     (effects (font (size 1.27 1.27)) (justify left bottom))
@@
     (effects (font (size 1.27 1.27)) (justify right bottom))
   )
-  (label "COIL_2" (at 176.53 72.39 180)
+  (label "COIL_4" (at 176.53 72.39 180)
     (effects (font (size 1.27 1.27)) (justify right bottom))
   )
-  (label "COIL_3" (at 176.53 105.41 180)
+  (label "COIL_2" (at 176.53 105.41 180)
     (effects (font (size 1.27 1.27)) (justify right bottom))
   )
@@
     (effects (font (size 1.27 1.27)) (justify left bottom))
   )
-  (label "OUT_IGN2" (at 187.96 66.04 90)
+  (label "OUT_IGN4" (at 187.96 66.04 90)
     (effects (font (size 1.27 1.27)) (justify left bottom))
   )
-  (label "OUT_IGN3" (at 187.96 99.06 90)
+  (label "OUT_IGN2" (at 187.96 99.06 90)
     (effects (font (size 1.27 1.27)) (justify left bottom))
   )
@@
     (effects (font (size 1.27 1.27)) (justify left bottom))
   )
-  (label "OUT_IGN6" (at 190.5 66.04 90)
+  (label "OUT_IGN3" (at 190.5 66.04 90)
     (effects (font (size 1.27 1.27)) (justify left bottom))
   )
-  (label "OUT_IGN4" (at 190.5 99.06 90)
+  (label "OUT_IGN6" (at 190.5 99.06 90)
     (effects (font (size 1.27 1.27)) (justify left bottom))
   )
@@
     (effects (font (size 1.27 1.27)) (justify left bottom))
   )
-  (label "COIL_6" (at 201.93 39.37 0)
+  (label "COIL_5" (at 201.93 39.37 0)
     (effects (font (size 1.27 1.27)) (justify left bottom))
   )
-  (label "COIL_5" (at 201.93 72.39 0)
+  (label "COIL_3" (at 201.93 72.39 0)
     (effects (font (size 1.27 1.27)) (justify left bottom))
   )
-  (label "COIL_4" (at 201.93 105.41 0)
+  (label "COIL_6" (at 201.93 105.41 0)
     (effects (font (size 1.27 1.27)) (justify left bottom))
   )
@@
     (effects (font (size 1.27 1.27)) (justify left bottom))
   )
-  (label "3.3V" (at 355.6 330.2 0)
-    (effects (font (size 1.27 1.27)) (justify left bottom))
-  )
   (label "SD_CLK" (at 355.6 332.74 0)
     (effects (font (size 1.27 1.27)) (justify left bottom))
@@
     (pin "1")
   )
+  (symbol (lib_id "power:+3V3") (at 120.65 546.1 0) (unit 1)
+    (in_bom yes) (on_board yes) (fields_autoplaced)
+    (property "Reference" "#PWR?" (id 0) (at 120.65 549.91 0)
+      (effects (font (size 1.27 1.27)) hide)
+    )
+    (property "Value" "+3V3" (id 1) (at 120.65 541.02 0))
+    (property "Footprint" "" (id 2) (at 120.65 546.1 0)
+      (effects (font (size 1.27 1.27)) hide)
+    )
+    (property "Datasheet" "" (id 3) (at 120.65 546.1 0)
+      (effects (font (size 1.27 1.27)) hide)
+    )
+    (pin "1")
+  )
   (symbol (lib_name "power:V12_RAW_1") (lib_id "power:V12_RAW") (at 299.72 434.34 0) (unit 1)
     (in_bom yes) (on_board yes)
@@
     (pin "1")
   )
+  (symbol (lib_id "power:+3V3") (at 367.03 327.66 0) (unit 1)
+    (in_bom yes) (on_board yes)
+    (property "Reference" "#PWR?" (id 0) (at 367.03 331.47 0)
+      (effects (font (size 1.27 1.27)) hide)
+    )
+    (property "Value" "+3V3" (id 1) (at 367.3983 322.0656 90))
+    (property "Footprint" "" (id 2) (at 367.03 327.66 0)
+      (effects (font (size 1.27 1.27)) hide)
+    )
+    (property "Datasheet" "" (id 3) (at 367.03 327.66 0)
+      (effects (font (size 1.27 1.27)) hide)
+    )
+    (pin "1")
+  )
   (symbol (lib_id "power:+3V3") (at 394.97 318.77 0) (unit 1)
     (in_bom yes) (on_board yes)
@@
       (reference "#PWR0171") (unit 1) (value "V5A") (footprint "")
     )
+    (path "/8b22620b-1702-4a05-8d08-a497382f5cd6"
+      (reference "#PWR?") (unit 1) (value "+3V3") (footprint "")
+    )
+    (path "/a3551de4-396b-4ed5-a944-647a6815ce4f"
+      (reference "#PWR?") (unit 1) (value "+3V3") (footprint "")
+    )
     (path "/00000000-0000-0000-0000-00005f7b99ce"
