File: boards/hellen88bmw/kicad6/hellen88bmw.kicad_sch (KiCad schematic)
At the start: 293 parts, among them J1 920-462A2021Y10101, J10 Conn_01x12, J11 Conn_01x12, J12 Conn_01x12, J13 Conn_01x12, J14 VRIN1, J15 VRIN2, J16 VROUT1, J17 XH-8A, J18 C165947, J2 UB-20PMFP-LC7002, J3 Micro_SD_Card, J4 Conn_01x05, J5 Conn_01x12, J6 Conn_01x12, J7 Conn_01x12, J8 Conn_01x12, J9 Conn_01x12, M1 Module-power12-0.2, M10 Module-ign8-0.1, M11 Module-mcu-0.4, M12 Module-knock-0.1, M2 Module-can-0.1, M3 Module-wbo-0.2, M4 Module-can-0.1, M5 Module-power5-0.1, M6 Module-vr-0.1, M7 Module-input-0.1, M8 Module-knock-0.1, M9 Module-output-0.2, P1 P, P2 P, P3 P, P4 P, P5 P, P6 P, Q1 NGD8201AN, Q2 NGD8201AN, Q3 NGD8201AN, Q4 NGD8201AN, Q5 NGD8201AN, Q6 NGD8201AN, Q7 NGD8201AN, Q8 NGD8201AN, SW1 BOOT0, SW2 RESET, U1 MPXA6115A, U2 MPX4_MAP, U3 LIS2DW12TR, U4 LPS25HB, U5 MCP6002-xSN

Commit message: Up 20/072021
Parts:
- removed MMCU15, MMCU16, MMCU20, MMCU37: MMCU, Connector_PinHeader_1.00mm:PinHeader_1x01_P1.00mm_Vertical, symbol Connector_Generic:Conn_01x01
- removed VIN23: Pad, Connector_PinHeader_1.00mm:PinHeader_1x01_P1.00mm_Vertical, symbol hellen-one-common:Pad
- added C10: 5.6nF, Capacitor_SMD:C_0402_1005Metric, symbol Device:C
- added C11, C13, C14, C16, C17, C19, C21, C9: 10uF, Capacitor_SMD:C_0603_1608Metric, symbol Device:C
- added C12: 10nF, Capacitor_SMD:C_0402_1005Metric, symbol Device:C
- added C15: 220nF, Capacitor_SMD:C_0402_1005Metric, symbol Device:C
- added C18, C20: 100nF, Capacitor_SMD:C_0402_1005Metric, symbol Device:C
- added D32, D33: 1N4148WS, Diode_SMD:D_SOD-323, symbol Device:D
- added J19: MiniFit, Connector_Molex:Molex_Mini-Fit_Jr_5569-02A2_2x01_P4.20mm_Horizontal, symbol Connector_Generic:Conn_01x02
- added J20: ETB_6p, Connector_PinHeader_2.54mm:PinHeader_1x06_P2.54mm_Vertical, symbol Connector_Generic:Conn_01x06
- added J21: ETB_4p, Connector_PinHeader_2.54mm:PinHeader_1x04_P2.54mm_Vertical, symbol Connector_Generic:Conn_01x04
- added R28: 100k, Resistor_SMD:R_0402_1005Metric, symbol Device:R
- added R29: 10k, Resistor_SMD:R_0402_1005Metric, symbol Device:R
- added R30: 100R, Resistor_SMD:R_0402_1005Metric, symbol Device:R
- added U6: L6205PD, kicad6:SO20POWER, symbol L6205PD:L6205PD
- C1, C2, C3, C4, C5, C6: footprint Capacitor_SMD:C_0603_1608Metric -> Capacitor_SMD:C_0402_1005Metric; LCSC C49678 -> C105882
- C7, C8: footprint Capacitor_SMD:C_0402_1005Metric -> Capacitor_SMD:C_0603_1608Metric; LCSC (none) -> C87152
- J17: footprint (none) -> Connector_PinHeader_2.54mm:PinHeader_1x08_P2.54mm_Vertical
- J2: LCSC C13453 -> NA
- M7: footprint input:input -> hellen-one-input-0.1:input
- R1, R2, R25, R26, R27, R3, R4, R5, R6: footprint Resistor_SMD:R_0603_1608Metric -> Resistor_SMD:R_0402_1005Metric
- U3: footprint Package_LGA:Kionix_LGA-12_2x2mm_P0.5mm_LayoutBorder2x4y -> kicad6:LGA12R50P4X4_200X200X70
Connections:
- net +5V: now also J20.1 (Pin_1), J20.2 (Pin_2), J21.1 (Pin_1)
- net GND: now also C10.2, C11.2, C13.2, C14.2, C16.2, C17.2, C18.2, C19.2, C20.2, C21.2, C9.2, J20.5 (Pin_5), J20.6 (Pin_6), J21.4 (Pin_4), R29.1, U6.1 (GND@1), U6.10 (GND@2), U6.11 (GND@3), U6.13 (SENSEB), U6.20 (GND@4), U6.8 (SENSEA), U6.SLUG1 (SLUG@1), U6.SLUG2 (SLUG@2), U6.SLUG3 (SLUG@3)
- net IN_TPS: now also J20.3 (Pin_3), J21.2 (Pin_2)
- net V12_PERM: now also M11.S6 (IN_D4)
- net at M11.E16 (OUT_PWM4): now also MMCU14.1 (Pin_1)
- net at M7.S17 (IN_AUX1): now also J20.4 (Pin_4), J21.3 (Pin_3)
- net -ETB: now reaches M11.E15 (OUT_PWM3)
- net -ETB: now also U6.14 (IN1B), U6.6 (IN1A); no longer MMCU14.1 (Pin_1)
- net +ETB: now reaches M11.E14 (OUT_PWM2)
- net +ETB: now also U6.15 (IN2B), U6.7 (IN2A)
- net ETB_EN: now reaches M11.E27 (OUT_PWM1)
- net ETB_EN: now also R28.2, R29.2
- new net: C10.1, R28.1, U6.16 (ENB), U6.5 (ENA)
- new net: C12.1, R30.1
- new net: C12.2, U6.4 (VCP)
- new net: C15.2, D33.1 (K), U6.17 (VBOOT)
- new net: D32.1 (K), D33.2 (A), R30.2
- new net +12V_RAW: C11.1, C13.1, C14.1, C15.1, C16.1, C17.1, C18.1, C19.1, C20.1, C21.1, C9.1, D32.2 (A), U6.19 (VSB), U6.2 (VSA)
- new net OUT_ETB+: J19.2 (Pin_2), U6.18 (OUT2B), U6.3 (OUT2A)
- new net OUT_ETB-: J19.1 (Pin_1), U6.12 (OUT1B), U6.9 (OUT1A)
Other:
- note added: "ETB driver"
- moved on the sheet: C3, D1, D2, D4, D5, D6, H1, H2, M1, M11D, M5, MMCU14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

Commit message: Up 21/072021
Parts:
- J17: footprint Connector_PinHeader_2.54mm:PinHeader_1x08_P2.54mm_Vertical -> kicad6:XH-8A
- P1, P2, P3, P4, P5, P6: footprint Connector_PinHeader_1.00mm:PinHeader_1x01_P1.00mm_Vertical -> Connector_Pin:Pin_D1.0mm_L10.0mm
Connections:
- net +12V_RAW is gone; now on net V12_RAW: C11.1, C13.1, C14.1, C15.1, C16.1, C17.1, C18.1, C19.1, C20.1, C21.1, C9.1, D32.2 (A), U6.19 (VSB), U6.2 (VSA)
- net COIL_1: now also D22.2 (A); no longer D16.2 (A)
- net COIL_2: now also D21.2 (A); no longer D20.2 (A)
- net COIL_3: now also D20.2 (A); no longer D17.2 (A)
- net COIL_4: now also D18.2 (A); no longer D21.2 (A)
- net COIL_5: now also D16.2 (A); no longer D18.2 (A)
- net COIL_6: now also D17.2 (A); no longer D22.2 (A)
Changed lines of the file:
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@@
   (junction (at 326.39 101.6) (diameter 0.9144) (color 0 0 0 0))
   (junction (at 326.39 529.59) (diameter 1.016) (color 0 0 0 0))
-  (junction (at 336.55 529.59) (diameter 1.016) (color 0 0 0 0))
+  (junction (at 336.55 529.59) (diameter 0.9144) (color 0 0 0 0))
   (junction (at 401.828 511.81) (diameter 0.9144) (color 0 0 0 0))
   (junction (at 407.162 527.05) (diameter 0.9144) (color 0 0 0 0))
@@
     (stroke (width 0) (type solid) (color 0 0 0 0))
   )
+  (wire (pts (xy 336.55 528.828) (xy 336.55 529.59))
+    (stroke (width 0) (type solid) (color 0 0 0 0))
+  )
   (wire (pts (xy 339.09 124.46) (xy 339.09 212.09))
     (stroke (width 0) (type solid) (color 0 0 0 0))
@@
     (effects (font (size 1.27 1.27)) (justify left bottom))
   )
-  (label "COIL_1" (at 147.32 91.44 0)
+  (label "COIL_1" (at 147.32 121.92 0)
     (effects (font (size 1.27 1.27)) (justify left bottom))
   )
-  (label "COIL_2" (at 147.32 93.98 0)
+  (label "COIL_7" (at 147.32 124.46 0)
     (effects (font (size 1.27 1.27)) (justify left bottom))
   )
-  (label "COIL_3" (at 147.32 96.52 0)
+  (label "COIL_8" (at 147.32 127 0)
     (effects (font (size 1.27 1.27)) (justify left bottom))
   )
-  (label "COIL_4" (at 147.32 99.06 0)
+  (label "COIL_5" (at 147.574 91.44 0)
     (effects (font (size 1.27 1.27)) (justify left bottom))
   )
-  (label "COIL_5" (at 147.32 119.38 0)
+  (label "COIL_3" (at 147.574 93.98 0)
     (effects (font (size 1.27 1.27)) (justify left bottom))
   )
-  (label "COIL_6" (at 147.32 121.92 0)
+  (label "COIL_6" (at 147.574 96.52 0)
     (effects (font (size 1.27 1.27)) (justify left bottom))
   )
-  (label "COIL_7" (at 147.32 124.46 0)
+  (label "COIL_2" (at 147.574 99.06 0)
     (effects (font (size 1.27 1.27)) (justify left bottom))
   )
-  (label "COIL_8" (at 147.32 127 0)
+  (label "COIL_4" (at 147.574 119.38 0)
     (effects (font (size 1.27 1.27)) (justify left bottom))
   )
@@
     (pin "1")
   )
-  (symbol (lib_id "hellen-one-common:+12V_RAW") (at 336.55 529.59 0) (mirror y) (unit 1)
+  (symbol (lib_name "power:V12_RAW_1") (lib_id "power:V12_RAW") (at 336.55 528.828 0) (unit 1)
     (in_bom yes) (on_board yes)
-    (property "Reference" "#PWR084" (id 0) (at 336.55 533.4 0)
+    (property "Reference" "#PWR0101" (id 0) (at 336.55 532.638 0)
       (effects (font (size 1.27 1.27)) hide)
     )
-    (property "Value" "+12V_RAW" (id 1) (at 339.09 526.0426 0))
-    (property "Footprint" "" (id 2) (at 336.55 529.59 0)
+    (property "Value" "V12_RAW" (id 1) (at 336.55 524.002 0))
+    (property "Footprint" "" (id 2) (at 336.55 528.828 0)
       (effects (font (size 1.27 1.27)) hide)
     )
-    (property "Datasheet" "" (id 3) (at 336.55 529.59 0)
+    (property "Datasheet" "" (id 3) (at 336.55 528.828 0)
       (effects (font (size 1.27 1.27)) hide)
     )
@@
       (effects (font (size 1.27 1.27)) (justify left) hide)
     )
-    (property "Footprint" "Connector_PinHeader_1.00mm:PinHeader_1x01_P1.00mm_Vertical" (id 2) (at 727.71 88.9 0)
+    (property "Footprint" "Connector_Pin:Pin_D1.0mm_L10.0mm" (id 2) (at 727.71 88.9 0)
       (effects (font (size 1.27 1.27)) hide)
     )
@@
       (effects (font (size 1.27 1.27)) (justify left) hide)
     )
-    (property "Footprint" "Connector_PinHeader_1.00mm:PinHeader_1x01_P1.00mm_Vertical" (id 2) (at 727.71 93.98 0)
+    (property "Footprint" "Connector_Pin:Pin_D1.0mm_L10.0mm" (id 2) (at 727.71 93.98 0)
       (effects (font (size 1.27 1.27)) hide)
     )
@@
       (effects (font (size 1.27 1.27)) (justify left) hide)
     )
-    (property "Footprint" "Connector_PinHeader_1.00mm:PinHeader_1x01_P1.00mm_Vertical" (id 2) (at 727.71 96.52 0)
+    (property "Footprint" "Connector_Pin:Pin_D1.0mm_L10.0mm" (id 2) (at 727.71 96.52 0)
       (effects (font (size 1.27 1.27)) hide)
     )
@@
       (effects (font (size 1.27 1.27)) (justify left) hide)
     )
-    (property "Footprint" "Connector_PinHeader_1.00mm:PinHeader_1x01_P1.00mm_Vertical" (id 2) (at 727.71 99.06 0)
+    (property "Footprint" "Connector_Pin:Pin_D1.0mm_L10.0mm" (id 2) (at 727.71 99.06 0)
       (effects (font (size 1.27 1.27)) hide)
     )
@@
       (effects (font (size 1.27 1.27)) (justify left) hide)
     )
-    (property "Footprint" "Connector_PinHeader_1.00mm:PinHeader_1x01_P1.00mm_Vertical" (id 2) (at 727.71 101.6 0)
+    (property "Footprint" "Connector_Pin:Pin_D1.0mm_L10.0mm" (id 2) (at 727.71 101.6 0)
       (effects (font (size 1.27 1.27)) hide)
     )
@@
       (effects (font (size 1.27 1.27)) (justify left) hide)
     )
-    (property "Footprint" "Connector_PinHeader_1.00mm:PinHeader_1x01_P1.00mm_Vertical" (id 2) (at 727.71 104.14 0)
+    (property "Footprint" "Connector_Pin:Pin_D1.0mm_L10.0mm" (id 2) (at 727.71 104.14 0)
       (effects (font (size 1.27 1.27)) hide)
     )
@@
       (effects (font (size 1.27 1.27)) (justify left))
     )
-    (property "Footprint" "Connector_PinHeader_2.54mm:PinHeader_1x08_P2.54mm_Vertical" (id 2) (at 718.82 93.98 0)
+    (property "Footprint" "kicad6:XH-8A" (id 2) (at 718.82 93.98 0)
       (effects (font (size 1.27 1.27)) hide)
     )
@@
       (reference "#PWR083") (unit 1) (value "GND") (footprint "")
     )
-    (path "/c27d986d-66d9-47ee-a228-b8bf4ac5f184"
-      (reference "#PWR084") (unit 1) (value "+12V_RAW") (footprint "")
-    )
     (path "/42c67703-e69c-40c7-bc66-de90d22f668d"
       (reference "#PWR085") (unit 1) (value "GND") (footprint "")
@@
       (reference "#PWR089") (unit 1) (value "GND") (footprint "")
     )
+    (path "/be3e7b18-1a68-4dc2-85c7-931099cf192f"
+      (reference "#PWR0101") (unit 1) (value "V12_RAW") (footprint "")
+    )
     (path "/190660b4-bcdd-4e59-b6d3-776a67e84bf4"
       (reference "#PWR0103") (unit 1) (value "GND") (footprint "")
@@
     )
     (path "/23675e65-3c89-4da5-9d44-df14f7138d42"
-      (reference "J17") (unit 1) (value "XH-8A") (footprint "Connector_PinHeader_2.54mm:PinHeader_1x08_P2.54mm_Vertical")
+      (reference "J17") (unit 1) (value "XH-8A") (footprint "kicad6:XH-8A")
     )
     (path "/6dce4d10-bd79-40ae-949c-0691816e6446"
@@
     )
     (path "/2517c1e8-64ff-48a7-80d6-e3cf32500647"
-      (reference "P1") (unit 1) (value "P") (footprint "Connector_PinHeader_1.00mm:PinHeader_1x01_P1.00mm_Vertical")
+      (reference "P1") (unit 1) (value "P") (footprint "Connector_Pin:Pin_D1.0mm_L10.0mm")
     )
     (path "/4126dcb2-5f09-4722-b81d-a1bb2e3fa05a"
-      (reference "P2") (unit 1) (value "P") (footprint "Connector_PinHeader_1.00mm:PinHeader_1x01_P1.00mm_Vertical")
+      (reference "P2") (unit 1) (value "P") (footprint "Connector_Pin:Pin_D1.0mm_L10.0mm")
     )
     (path "/2ad0c7d8-daf1-48e3-bf3f-9a1d560e59d5"
-      (reference "P3") (unit 1) (value "P") (footprint "Connector_PinHeader_1.00mm:PinHeader_1x01_P1.00mm_Vertical")
+      (reference "P3") (unit 1) (value "P") (footprint "Connector_Pin:Pin_D1.0mm_L10.0mm")
     )
     (path "/5bd3a627-dbcb-4254-876c-98a88b378aac"
-      (reference "P4") (unit 1) (value "P") (footprint "Connector_PinHeader_1.00mm:PinHeader_1x01_P1.00mm_Vertical")
+      (reference "P4") (unit 1) (value "P") (footprint "Connector_Pin:Pin_D1.0mm_L10.0mm")
     )
     (path "/42c53423-459a-435f-8dcf-332824394e37"
-      (reference "P5") (unit 1) (value "P") (footprint "Connector_PinHeader_1.00mm:PinHeader_1x01_P1.00mm_Vertical")
+      (reference "P5") (unit 1) (value "P") (footprint "Connector_Pin:Pin_D1.0mm_L10.0mm")
     )
     (path "/c460f24f-20f1-4eab-98f7-3976e80ade92"
-      (reference "P6") (unit 1) (value "P") (footprint "Connector_PinHeader_1.00mm:PinHeader_1x01_P1.00mm_Vertical")
+      (reference "P6") (unit 1) (value "P") (footprint "Connector_Pin:Pin_D1.0mm_L10.0mm")
     )
     (path "/00000000-0000-0000-0000-00005fc69d39"

Commit message: Up 04/082021
Parts:
- D1, D10, D11, D12, D13, D14, D15, D16, D17, D18, D19, D2, D20, D21, D22, D23, D24, D25, D26, D27, D28, D29, D3, D30, D31, D4, D5, D6, D7, D8, D9: LCSC (none) -> C72041
- MMCU1: value MMCU1 -> MMCU
- renumbered MMCU41 to MMCU15
Changed lines of the file:
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@@
       (effects (font (size 1.27 1.27)) (justify left))
     )
-    (property "Value" "MMCU1" (id 1) (at 400.05 242.57 0)
+    (property "Value" "MMCU" (id 1) (at 400.05 242.57 0)
       (effects (font (size 1.27 1.27)) (justify left) hide)
     )
@@
   (symbol (lib_id "Connector_Generic:Conn_01x01") (at 463.55 242.57 0) (unit 1)
     (in_bom yes) (on_board yes)
-    (property "Reference" "MMCU41" (id 0) (at 466.09 242.57 0)
+    (property "Reference" "MMCU15" (id 0) (at 466.09 242.57 0)
       (effects (font (size 1.27 1.27)) (justify left))
     )
@@
       (effects (font (size 1.27 1.27)) hide)
     )
+    (property "LCSC" "C72041" (id 4) (at 129.54 93.98 0)
+      (effects (font (size 1.27 1.27)) hide)
+    )
     (pin "1")
     (pin "2")
@@
       (effects (font (size 1.27 1.27)) hide)
     )
+    (property "LCSC" "C72041" (id 4) (at 129.54 99.06 0)
+      (effects (font (size 1.27 1.27)) hide)
+    )
     (pin "1")
     (pin "2")
@@
       (effects (font (size 1.27 1.27)) hide)
     )
+    (property "LCSC" "C72041" (id 4) (at 129.54 121.92 0)
+      (effects (font (size 1.27 1.27)) hide)
+    )
     (pin "1")
     (pin "2")
@@
       (effects (font (size 1.27 1.27)) hide)
     )
+    (property "LCSC" "C72041" (id 4) (at 129.54 127 0)
+      (effects (font (size 1.27 1.27)) hide)
+    )
     (pin "1")
     (pin "2")
@@
       (effects (font (size 1.27 1.27)) hide)
     )
+    (property "LCSC" "C72041" (id 4) (at 140.97 91.44 0)
+      (effects (font (size 1.27 1.27)) hide)
+    )
     (pin "1")
     (pin "2")
@@
       (effects (font (size 1.27 1.27)) hide)
     )
+    (property "LCSC" "C72041" (id 4) (at 140.97 96.52 0)
+      (effects (font (size 1.27 1.27)) hide)
+    )
     (pin "1")
     (pin "2")
@@
       (effects (font (size 1.27 1.27)) hide)
     )
+    (property "LCSC" "C72041" (id 4) (at 140.97 119.38 0)
+      (effects (font (size 1.27 1.27)) hide)
+    )
     (pin "1")
     (pin "2")
@@
       (effects (font (size 1.27 1.27)) hide)
     )
+    (property "LCSC" "C72041" (id 4) (at 140.97 124.46 0)
+      (effects (font (size 1.27 1.27)) hide)
+    )
     (pin "1")
     (pin "2")
@@
       (effects (font (size 1.27 1.27)) hide)
     )
+    (property "LCSC" "C72041" (id 4) (at 486.41 124.46 0)
+      (effects (font (size 1.27 1.27)) hide)
+    )
     (pin "1")
     (pin "2")
@@
       (effects (font (size 1.27 1.27)) hide)
     )
+    (property "LCSC" "C72041" (id 4) (at 486.41 129.54 0)
+      (effects (font (size 1.27 1.27)) hide)
+    )
     (pin "1")
     (pin "2")
@@
       (effects (font (size 1.27 1.27)) hide)
     )
+    (property "LCSC" "C72041" (id 4) (at 486.41 146.05 0)
+      (effects (font (size 1.27 1.27)) hide)
+    )
     (pin "1")
     (pin "2")
@@
       (effects (font (size 1.27 1.27)) hide)
     )
+    (property "LCSC" "C72041" (id 4) (at 486.41 151.13 0)
+      (effects (font (size 1.27 1.27)) hide)
+    )
     (pin "1")
     (pin "2")
@@
       (effects (font (size 1.27 1.27)) hide)
     )
+    (property "LCSC" "C72041" (id 4) (at 497.84 127 0)
+      (effects (font (size 1.27 1.27)) hide)
+    )
     (pin "1")
     (pin "2")
@@
       (effects (font (size 1.27 1.27)) hide)
     )
+    (property "LCSC" "C72041" (id 4) (at 497.84 132.08 0)
+      (effects (font (size 1.27 1.27)) hide)
+    )
     (pin "1")
     (pin "2")
@@
       (effects (font (size 1.27 1.27)) hide)
     )
+    (property "LCSC" "C72041" (id 4) (at 497.84 148.59 0)
+      (effects (font (size 1.27 1.27)) hide)
+    )
     (pin "1")
     (pin "2")
@@
       (effects (font (size 1.27 1.27)) hide)
     )
+    (property "LCSC" "C72041" (id 4) (at 497.84 153.67 0)
+      (effects (font (size 1.27 1.27)) hide)
+    )
     (pin "1")
     (pin "2")
@@
       (effects (font (size 1.27 1.27)) hide)
     )
+    (property "LCSC" "C72041" (id 4) (at 604.52 181.61 0)
+      (effects (font (size 1.27 1.27)) hide)
+    )
     (pin "1")
     (pin "2")
@@
       (effects (font (size 1.27 1.27)) hide)
     )
+    (property "LCSC" "C72041" (id 4) (at 613.41 193.04 0)
+      (effects (font (size 1.27 1.27)) hide)
+    )
     (pin "1")
     (pin "2")
@@
       (effects (font (size 1.27 1.27)) hide)
     )
+    (property "LCSC" "C72041" (id 4) (at 633.73 62.23 0)
+      (effects (font (size 1.27 1.27)) hide)
+    )
     (pin "1")
     (pin "2")
@@
       (effects (font (size 1.27 1.27)) hide)
     )
+    (property "LCSC" "C72041" (id 4) (at 633.73 67.31 0)
+      (effects (font (size 1.27 1.27)) hide)
+    )
     (pin "1")
     (pin "2")
@@
       (effects (font (size 1.27 1.27)) hide)
     )
+    (property "LCSC" "C72041" (id 4) (at 645.16 59.69 0)
+      (effects (font (size 1.27 1.27)) hide)
+    )
     (pin "1")
     (pin "2")
@@
       (effects (font (size 1.27 1.27)) hide)
     )
+    (property "LCSC" "C72041" (id 4) (at 645.16 64.77 0)
+      (effects (font (size 1.27 1.27)) hide)
+    )
     (pin "1")
     (pin "2")
@@
       (effects (font (size 1.27 1.27)) hide)
     )
+    (property "LCSC" "C72041" (id 4) (at 659.13 459.74 0)
+      (effects (font (size 1.27 1.27)) hide)
+    )
     (pin "1")
     (pin "2")
@@
       (effects (font (size 1.27 1.27)) hide)
     )
+    (property "LCSC" "C72041" (id 4) (at 670.56 454.66 0)
+      (effects (font (size 1.27 1.27)) hide)
+    )
     (pin "1")
     (pin "2")
@@
       (effects (font (size 1.27 1.27)) hide)
     )
+    (property "LCSC" "C72041" (id 4) (at 670.56 462.28 0)
+      (effects (font (size 1.27 1.27)) hide)
+    )
     (pin "1")
     (pin "2")
@@
       (effects (font (size 1.27 1.27)) hide)
     )
+    (property "LCSC" "C72041" (id 4) (at 692.15 161.29 0)
+      (effects (font (size 1.27 1.27)) hide)
+    )
     (pin "1")
     (pin "2")
@@
       (effects (font (size 1.27 1.27)) hide)
     )
+    (property "LCSC" "C72041" (id 4) (at 692.15 166.37 0)
+      (effects (font (size 1.27 1.27)) hide)
+    )
     (pin "1")
     (pin "2")
@@
       (effects (font (size 1.27 1.27)) hide)
     )
+    (property "LCSC" "C72041" (id 4) (at 703.58 163.83 0)
+      (effects (font (size 1.27 1.27)) hide)
+    )
     (pin "1")
     (pin "2")
@@
       (effects (font (size 1.27 1.27)) hide)
     )
+    (property "LCSC" "C72041" (id 4) (at 779.78 374.65 0)
+      (effects (font (size 1.27 1.27)) hide)
+    )
     (pin "1")
     (pin "2")
@@
       (effects (font (size 1.27 1.27)) hide)
     )
+    (property "LCSC" "C72041" (id 4) (at 779.78 383.54 0)
+      (effects (font (size 1.27 1.27)) hide)
+    )
     (pin "1")
     (pin "2")
@@
       (effects (font (size 1.27 1.27)) hide)
     )
+    (property "LCSC" "C72041" (id 4) (at 779.78 398.78 0)
+      (effects (font (size 1.27 1.27)) hide)
+    )
     (pin "1")
     (pin "2")
@@
     )
     (path "/371da9ee-3778-49d5-8e1a-042813c36e4b"
-      (reference "MMCU1") (unit 1) (value "MMCU1") (footprint "Connector_PinHeader_1.00mm:PinHeader_1x01_P1.00mm_Vertical")
+      (reference "MMCU1") (unit 1) (value "MMCU") (footprint "Connector_PinHeader_1.00mm:PinHeader_1x01_P1.00mm_Vertical")
     )
     (path "/5cb52594-3683-48a2-a3ac-418876fce88b"
@@
       (reference "MMCU14") (unit 1) (value "MMCU") (footprint "Connector_PinHeader_1.00mm:PinHeader_1x01_P1.00mm_Vertical")
     )
+    (path "/08c8ab9b-72e5-4e66-8440-0c7c2e37e8c8"
+      (reference "MMCU15") (unit 1) (value "MMCU") (footprint "Connector_PinHeader_1.00mm:PinHeader_1x01_P1.00mm_Vertical")
+    )
     (path "/fad97116-8017-4321-81e0-8e5306d21441"
       (reference "MMCU17") (unit 1) (value "MMCU") (footprint "Connector_PinHeader_1.00mm:PinHeader_1x01_P1.00mm_Vertical")
@@
       (reference "MMCU40") (unit 1) (value "MMCU") (footprint "Connector_PinHeader_1.00mm:PinHeader_1x01_P1.00mm_Vertical")
     )
-    (path "/08c8ab9b-72e5-4e66-8440-0c7c2e37e8c8"
-      (reference "MMCU41") (unit 1) (value "MMCU") (footprint "Connector_PinHeader_1.00mm:PinHeader_1x01_P1.00mm_Vertical")
-    )
     (path "/2517c1e8-64ff-48a7-80d6-e3cf32500647"

Commit message: Up 12/08/2021
Parts:
- D1, D10, D11, D12, D13, D14, D15, D16, D17, D18, D19, D2, D20, D21, D22, D23, D24, D25, D26, D27, D28, D29, D3, D30, D31, D4, D5, D6, D7, D8, D9: value LED -> LED-BLUE-0603
- JP14, JP16, JP17, JP2, JP20, JP21, JP22, JP23, JP24, JP25, JP26, JP27, JP29, JP3, JP31, JP32, JP33, JP35, JP4, JP41, JP42, JP43, JP44, JP46, JP47, JP49, JP5, JP50, JP51, JP52, JP54, JP56, JP59, JP7, JP73, JP77, JP78, JP85, JP86: LCSC (none) -> C17477
- Q1, Q2, Q3, Q4, Q5, Q7, Q8: LCSC (none) -> C151649
- R27: Comment (none) -> 0
- R28: LCSC C25803 -> (none)
- R29: LCSC C25804 -> (none)
- R30: value 100R -> 100; LCSC C22775 -> (none)

Commit message: Up 12/08/2021 part 2
Parts:
- M5: value Module-power5-0.1 -> Module-power5-0.2
Changed lines of the file:
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@@
     (in_bom yes) (on_board yes)
     (property "Reference" "M5" (id 0) (at 787.4 496.57 0))
-    (property "Value" "Module-power5-0.1" (id 1) (at 796.29 499.11 0))
+    (property "Value" "Module-power5-0.2" (id 1) (at 796.29 499.11 0))
     (property "Footprint" "hellen-one-power5-0.1:power5" (id 2) (at 765.81 474.98 0)
       (effects (font (size 1.27 1.27)) hide)
@@
     )
     (path "/837f573b-b69f-444b-af7b-cf02f9bc2883"
-      (reference "M5") (unit 1) (value "Module-power5-0.1") (footprint "hellen-one-power5-0.1:power5")
+      (reference "M5") (unit 1) (value "Module-power5-0.2") (footprint "hellen-one-power5-0.1:power5")
     )
     (path "/eab6451a-c287-4aeb-9352-a8447ab4d341"
